File: Trapezoid_Terminal/Processor Board/Entrex Trapezoid Processor Board v37.kicad_sch (KiCad schematic)
At the start: 194 parts, among them J1 Jumper_2_Bridged, J17 Card Edge Connector, J18 Card Edge Connector, Q1 2N3904, Q2 2N3904, Q3 2N3904

Commit message: Updated schematics during tutorial
Connections:
- net UJ5_10 renamed D0
- net UJ5_13 renamed D2
- net UJ5_6 renamed D1
- net UK3_3 renamed D4
- net UK3_7 renamed D3
- net UK5_13 renamed D6
- net UK5_3 renamed D7
- net UK5_6 renamed D5
Other:
- note added: "Mystery Section"
- note removed: "Data Bus Section?"

Commit message: Connect UD8_3
Connections:
- net R28-C65 is gone; now on net UD8_3: C65.1, R28.1
- no-connect marks 178 -> 177
Other:
- moved on the sheet: C55, C65, R17, R28, UF2A
