File: Trapezoid_Terminal/Processor Board/Entrex Trapezoid Processor Board v37.kicad_sch (KiCad schematic)
At the start: 194 parts, among them J1 Jumper_2_Bridged, J17 Card Edge Connector, J18 Card Edge Connector, Q1 2N3904, Q2 2N3904, Q3 2N3904

Commit message: notes
Changed lines of the file:
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@@
     (effects (font (size 5 5) (thickness 1) bold) (justify left bottom))
   )
+  (text "x" (at 641.35 380.365 0)
+    (effects (font (size 3 3) (thickness 1) bold (color 255 30 30 1)) (justify right bottom))
+  )
   (text "*" (at 171.45 1022.35 0)
     (effects (font (size 3 3) (thickness 1) bold (color 255 165 0 1)) (justify right bottom))
@@
       (effects (font (size 1.27 1.27)) (justify left) hide)
     )
+  )
+  (global_label "UE2_1" (shape output) (at 692.785 384.175 0) (fields_autoplaced)
+    (effects (font (size 1.27 1.27)) (justify left))
+    (property "Intersheetrefs" "${INTERSHEET_REFS}" (at 701.5569 384.175 0)
+      (effects (font (size 1.27 1.27)) (justify left) hide)
+    )
