File: Trapezoid_Terminal/Processor Board/Entrex Trapezoid Processor Board v37.kicad_sch (KiCad schematic)
At the start: 194 parts, among them J1 Jumper_2_Bridged, J17 Card Edge Connector, J18 Card Edge Connector, Q1 2N3904, Q2 2N3904, Q3 2N3904

Commit message: warnings
Other:
- note added: "WARNING: Until refined & corrected, Global Label tag arrows may not indicate the proper signal in/out direction. IN was used as default when KiCad Symbols (components) were not clear on In vs Out signals, so always check component datasheets when in doubt."
Changed lines of the file:
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@@
     (effects (font (size 3 3) (thickness 1) bold (color 255 165 0 1)) (justify right bottom))
+  )
+  (text "WARNING:  Until refined & corrected, Global Label tag arrows may not indicate the \nproper signal in/out direction.\nIN was used as default when KiCad Symbols (components) were not clear on \nIn vs Out signals, so always check component datasheets when in doubt.\n"
+    (at 1085.85 1283.97 0)
+    (effects (font (size 4 4) (thickness 0.8) bold (color 255 105 180 1)) (justify left bottom))
   )
   (text "*" (at 330.2 1183.64 0)
@@
     (effects (font (size 1.27 1.27)) (justify left bottom))
   )
+  (text "WARNING:  Until refined & corrected, Global Label tag arrows may not indicate the \nproper signal in/out direction.\nIN was used as default when KiCad Symbols (components) were not clear on \nIn vs Out signals, so always check component datasheets when in doubt.\n"
+    (at 1170.94 477.52 0)
+    (effects (font (size 4 4) (thickness 0.8) bold (color 255 105 180 1)) (justify left bottom))
+  )
   (text "x" (at 45.339 210.947 0)
     (effects (font (size 3 3) (thickness 1) bold (color 255 30 30 1)) (justify right bottom))
@@
     (effects (font (size 3 3) (thickness 1) bold (color 5 102 8 1)) (justify right bottom))
   )
+  (text "WARNING:  Until refined & corrected, Global Label tag arrows may not indicate the \nproper signal in/out direction.\nIN was used as default when KiCad Symbols (components) were not clear on \nIn vs Out signals, so always check component datasheets when in doubt.\n"
+    (at 39.37 266.7 0)
+    (effects (font (size 4 4) (thickness 0.8) bold (color 255 105 180 1)) (justify left bottom))
+  )
   (text "*" (at 435.61 1179.195 90)

Commit message: corrections
Connections:
- net R17-C55 is gone; now on net UF2_2: C55.1, R17.2
- no-connect marks 176 -> 175
Other:
- note added: "D0-D7"
- note added: "Keyboard Enable"
Changed lines of the file:
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@@
   (junction (at 391.16 781.05) (diameter 0) (color 0 0 0 0)
   )
+  (junction (at 866.14 1227.709) (diameter 0) (color 0 0 0 0)
+  )
   (junction (at 1296.67 734.06) (diameter 0) (color 0 0 0 0)
   )
@@
   (junction (at 750.57 312.42) (diameter 0) (color 0 0 0 0)
   )
+  (junction (at 866.14 1217.295) (diameter 0) (color 0 0 0 0)
+  )
   (junction (at 763.27 898.525) (diameter 0) (color 0 0 0 0)
   )
@@
   (no_connect (at 596.9 1483.995))
   (no_connect (at 982.345 816.61))
-  (no_connect (at 839.47 1217.295))
   (no_connect (at 544.195 1035.685))
   (no_connect (at 1129.665 1223.645))
@@
     (stroke (width 0) (type default))
   )
+  (bus (pts (xy 801.37 930.275) (xy 801.37 931.545))
+    (stroke (width 0) (type default))
+  )
   (bus (pts (xy 791.21 602.615) (xy 791.21 581.025))
     (stroke (width 1) (type default))
@@
     (stroke (width 0) (type default))
   )
+  (wire (pts (xy 866.14 1227.709) (xy 880.237 1227.709))
+    (stroke (width 0) (type default))
+  )
   (bus (pts (xy 563.245 720.725) (xy 563.245 734.06))
     (stroke (width 1) (type default))
@@
     (stroke (width 0) (type default))
   )
+  (wire (pts (xy 866.14 1217.2696) (xy 866.14 1217.295))
+    (stroke (width 0) (type default))
+  )
   (bus (pts (xy 1261.11 170.18) (xy 1261.11 167.64))
     (stroke (width 1) (type default))
@@
     (stroke (width 0) (type default))
   )
+  (wire (pts (xy 839.47 1217.295) (xy 866.14 1217.295))
+    (stroke (width 0) (type default))
+  )
   (bus (pts (xy 791.21 563.245) (xy 791.21 539.75))
     (stroke (width 1) (type default))
@@
     (stroke (width 0) (type default))
   )
-  (wire (pts (xy 856.742 1227.709) (xy 880.237 1227.709))
+  (wire (pts (xy 856.742 1227.709) (xy 866.14 1227.709))
     (stroke (width 0) (type default))
   )
@@
     (stroke (width 0) (type default))
   )
+  (wire (pts (xy 866.14 1217.295) (xy 866.14 1227.709))
+    (stroke (width 0) (type default))
+  )
   (wire (pts (xy 523.875 687.07) (xy 527.685 687.07))
     (stroke (width 0) (type default))
@@
     (effects (font (size 1.27 1.27)) (justify left bottom))
   )
+  (text "Keyboard Enable" (at 1153.16 1186.815 0)
+    (effects (font (size 1.27 1.27)) (justify left bottom))
+  )
   (text "*" (at 235.585 1012.19 0)
     (effects (font (size 3 3) (thickness 1) bold (color 5 102 8 1)) (justify right bottom))
@@
     (effects (font (size 3 3) (thickness 1) bold (color 29 233 22 1)) (justify right bottom))
   )
+  (text "D0-D7" (at 801.37 929.005 0)
+    (effects (font (size 1.27 1.27)) (justify left bottom))
+  )
   (text "*" (at 993.14 611.505 0)
     (effects (font (size 3 3) (thickness 1) bold (color 0 0 0 1)) (justify right bottom))
@@
     (effects (font (size 1.27 1.27)) (justify left bottom))
   )
+  (label "UF2_2" (at 867.6386 1227.709 0) (fields_autoplaced)
+    (effects (font (size 1.27 1.27)) (justify left bottom))
+  )
   (label "JPC9_16" (at 885.19 586.74 0) (fields_autoplaced)
     (effects (font (size 1.27 1.27)) (justify left bottom))
@@
     (effects (font (size 1.27 1.27)) (justify left bottom))
   )
-  (label "R17-C55" (at 856.742 1227.709 0) (fields_autoplaced)
+  (label "UF2_2" (at 856.742 1227.709 0) (fields_autoplaced)
     (effects (font (size 1.27 1.27)) (justify left bottom))
   )
@@
     (effects (font (size 1.27 1.27)) (justify left bottom))
   )
-  (label "R17-C55" (at 880.237 1227.709 180) (fields_autoplaced)
-    (effects (font (size 1.27 1.27)) (justify right bottom))
-  )
   (label "GND" (at 854.075 1751.33 180) (fields_autoplaced)
     (effects (font (size 1.27 1.27)) (justify right bottom))
@@
     (effects (font (size 1.27 1.27)) (justify left bottom))
   )
+  (label "{J17_22 J17_24 J17_26 J17_28 J17_30 J17_32 J17_34 J17_36 }"
+    (at 801.37 930.91 0) (fields_autoplaced)
+    (effects (font (size 0.125 0.125)) (justify left bottom))
+  )
   (label "UB7_11" (at 813.435 477.52 0) (fields_autoplaced)

Commit message: Update Entrex Trapezoid Processor Board v37.kicad_sch
Other:
- note added: "to UC1 pin 13 74LS138"
Changed lines of the file:
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@@
   (junction (at 166.37 654.05) (diameter 0) (color 0 0 0 0)
   )
+  (junction (at 675.64 1234.44) (diameter 0) (color 0 0 0 0)
+  )
   (junction (at 497.84 1085.85) (diameter 0) (color 0 0 0 0)
   )
@@
     (stroke (width 0) (type default))
   )
+  (wire (pts (xy 761.365 1191.26) (xy 761.365 1240.155))
+    (stroke (width 0) (type default))
+  )
   (wire (pts (xy 356.87 707.39) (xy 339.09 707.39))
     (stroke (width 0) (type default))
@@
     (stroke (width 0) (type default))
   )
+  (wire (pts (xy 744.855 1191.26) (xy 761.365 1191.26))
+    (stroke (width 0) (type default))
+  )
   (wire (pts (xy 728.98 975.995) (xy 728.98 996.95))
     (stroke (width 0) (type default))
@@
     (stroke (width 1) (type default))
   )
+  (wire (pts (xy 384.175 1181.735) (xy 384.175 1240.155))
+    (stroke (width 0) (type default))
+  )
   (wire (pts (xy 452.755 805.815) (xy 416.56 805.815))
     (stroke (width 0) (type default))
@@
     (stroke (width 1) (type default))
   )
+  (wire (pts (xy 675.64 1234.44) (xy 381.635 1234.44))
+    (stroke (width 0) (type default))
+  )
   (bus (pts (xy 1018.54 198.755) (xy 1033.78 198.755))
     (stroke (width 1) (type default))
@@
     (stroke (width 0) (type default))
   )
+  (wire (pts (xy 744.855 1188.72) (xy 744.855 1191.26))
+    (stroke (width 0) (type default))
+  )
   (bus (pts (xy 1261.11 191.77) (xy 1261.11 189.23))
     (stroke (width 1) (type default))
@@
     (stroke (width 0) (type default))
   )
+  (wire (pts (xy 384.175 1240.155) (xy 761.365 1240.155))
+    (stroke (width 0) (type default))
+  )
   (wire (pts (xy 417.195 732.79) (xy 427.99 732.79))
     (stroke (width 0) (type default))
@@
     (stroke (width 0) (type default))
   )
+  (wire (pts (xy 381.635 1181.735) (xy 381.635 1234.44))
+    (stroke (width 0) (type default))
+  )
   (wire (pts (xy 716.915 568.325) (xy 716.915 431.8))
     (stroke (width 0) (type default))
@@
     (effects (font (size 3 3) (thickness 1) bold (color 0 0 0 1)) (justify right bottom))
   )
-  (text "*" (at 856.615 1224.915 0)
+  (text "*" (at 851.535 1224.915 0)
     (effects (font (size 3 3) (thickness 1) bold (color 29 233 22 1)) (justify right bottom))
   )
@@
     (effects (font (size 3 3) (thickness 1) bold (color 255 165 0 1)) (justify right bottom))
   )
+  (text "to J25 ONLY\n" (at 372.11 1134.745 90)
+    (effects (font (size 1.27 1.27)) (justify left bottom))
+  )
   (text "*" (at 716.915 1210.31 0)
     (effects (font (size 3 3) (thickness 1) bold (color 5 102 8 1)) (justify right bottom))
@@
     (effects (font (size 3 3) (thickness 1) bold (color 5 102 8 1)) (justify right bottom))
   )
+  (text "to UC1 pin 13 74LS138" (at 791.21 375.285 0)
+    (effects (font (size 1.27 1.27)) (justify left bottom))
+  )
   (text "*" (at 241.935 800.1 0)
     (effects (font (size 3 3) (thickness 1) bold (color 255 165 0 1)) (justify right bottom))
@@
     (effects (font (size 3 3) (thickness 1) bold (color 255 165 0 1)) (justify right bottom))
   )
+  (text "Keyboard Enable" (at 852.17 1223.01 0)
+    (effects (font (size 1.27 1.27)) (justify left bottom))
+  )
   (text "3" (at 225.2101 1673.5883 0)
     (effects (font (size 5 5) bold) (justify left bottom))
@@
     (effects (font (size 3 3) (thickness 1) bold (color 255 165 0 1)) (justify right bottom))
   )
+  (text "Magic 555 Timer and other Entrex VooDoo" (at 334.645 1182.37 90)
+    (effects (font (size 1.27 1.27)) (justify right bottom))
+  )
   (text "WARNING:\nDO NOT use 'Tools -> Update PCB from Schematic'\nUse ONLY 'Tools -> Update Schematic from PCB'"

Commit message: Fix Nets
Parts:
- removed C64: C, Forgotten Machines:Disc Capacitor Entrex Trapezoid .30, symbol Device:C
- added C53: C, Forgotten Machines:Disc Capacitor Entrex Trapezoid .30, symbol Device:C
Connections:
- net GND: now also C53.2
- net JPA9_1: now also C53.1
- net JPA9_12: no longer UA1.1 (~{MR}), UA4.1 (~{MR}), UA7.12, UA7.4, UC4.2, UC4.3, UD5.1, UD5.10, UD5.3
- new net UA7_12: UA7.12, UC4.2, UC4.3, UD5.1, UD5.10, UD5.3
- new net UA7_4: UA1.1 (~{MR}), UA4.1 (~{MR}), UA7.4

Commit message: Integrate Phar's Schematics
Parts:
- removed C53: C, Forgotten Machines:Disc Capacitor Entrex Trapezoid .30, symbol Device:C
- removed C55: CAP, Forgotten Machines:Disc Capacitor Entrex Trapezoid, symbol pspice:CAP
- removed C65: CAP, Forgotten Machines:Disc Capacitor Entrex Trapezoid .10, symbol pspice:CAP
- removed CR6: 1N4148, Diode_THT:D_DO-35_SOD27_P10.16mm_Horizontal, symbol Diode:1N4148
- removed JPA9, JPB9, JPC9: 1920 vs 480, Package_DIP:DIP-16_W7.62mm, symbol Forgotten Machines:Jumper-8-P1-N.O.
- removed R24, R25, R26, R28: R, Resistor_THT:R_Axial_DIN0309_L9.0mm_D3.2mm_P12.70mm_Horizontal, symbol Device:R
- removed RND0, RNK7: R_Network07_US, Resistor_THT:R_Array_SIP8, symbol Device:R_Network07_US
- removed UA6: 74LS161, Package_DIP:DIP-16_W7.62mm, symbol 74xx:74LS161
- removed unit 2 of UA7
- removed unit 5 of UA7
- removed unit 1 of UC3
- removed unit 2 of UF3
- removed unit 3 of UF3
- removed unit 4 of UF3
- removed unit 6 of UF3
- removed UF6: 8T97, Package_DIP:DIP-16_W7.62mm, symbol Missing Parts:8T97
- removed UF9, UH9: 74LS174, Package_DIP:DIP-16_W7.62mm, symbol 74xx:74LS174
- removed unit 5 of UH4
- removed UJ5: 8T28, Package_DIP:DIP-16_W7.62mm, symbol Missing Parts:8T28
- removed UJ8, UK8: 2708_EPROM, Package_DIP:DIP-24_W15.24mm, symbol Missing Parts:2708_EPROM
- removed UK0: UA79M05, Package_TO_SOT_THT:TO-220-3_Vertical, symbol Regulator_Linear:LM7905_TO220
- removed XA8: 6.4137 MHz, Oscillator:Oscillator_DIP-14, symbol Oscillator:CXO_DIP14
- removed YJ4: Crystal CY19A 18.0Mhz, Crystal:Crystal_HC18-U_Horizontal, symbol Device:Crystal
- added C53: CAP, Forgotten Machines:Disc Capacitor Entrex Trapezoid .10, symbol pspice:CAP
- added C54: CAP, Forgotten Machines:Disc Capacitor Entrex Trapezoid, symbol pspice:CAP
- added C55: C, Forgotten Machines:Disc Capacitor Entrex Trapezoid .30, symbol Device:C
- added CR1: 1N4148, Diode_THT:D_DO-35_SOD27_P10.16mm_Horizontal, symbol Diode:1N4148
- added JPA1, JPB1, JPC1: 1920 vs 480, Package_DIP:DIP-16_W7.62mm, symbol Forgotten Machines:Jumper-8-P1-N.O.
- added R1, R11, R15, R16: R, Resistor_THT:R_Axial_DIN0309_L9.0mm_D3.2mm_P12.70mm_Horizontal, symbol Device:R
- added RND1, RNK1: R_Network07_US, Resistor_THT:R_Array_SIP8, symbol Device:R_Network07_US
- added UA6, UF1: 74LS04, Package_DIP:DIP-14_W7.62mm, symbol 74xx:74LS04
- added UA8: 74LS161, Package_DIP:DIP-16_W7.62mm, symbol 74xx:74LS161
- added UC2: 74LS107, Package_DIP:DIP-14_W7.62mm, symbol 74xx:74LS107
- added UF5: 8T97, Package_DIP:DIP-16_W7.62mm, symbol Missing Parts:8T97
- added UF6, UH6: 74LS174, Package_DIP:DIP-16_W7.62mm, symbol 74xx:74LS174
- added UJ3: 8T28, Package_DIP:DIP-16_W7.62mm, symbol Missing Parts:8T28
- added UJ4, UK7: 2708_EPROM, Package_DIP:DIP-24_W15.24mm, symbol Missing Parts:2708_EPROM
- added UK4: UA79M05, Package_TO_SOT_THT:TO-220-3_Vertical, symbol Regulator_Linear:LM7905_TO220
- added XA1: 6.4137 MHz, Oscillator:Oscillator_DIP-14, symbol Oscillator:CXO_DIP14
- added YJ1: Crystal CY19A 18.0Mhz, Crystal:Crystal_HC18-U_Horizontal, symbol Device:Crystal
Connections:
- net J18_24 is gone; now on net VIDEO_MEM_D6: J18.24 (Pin_24)
- net J18_26 is gone; now on net VIDEO_MEM_D7: J18.26 (Pin_26)
- net J18_28 is gone; now on net CPU_STATUS_INP: J18.28 (Pin_28)
- net J18_4 is gone; now on net VIDEO_MEM_D1: J18.4 (Pin_4), UE7.12 (In5), UK9.12 (Data_Out_2), UL9.12 (Data_Out_2)
- net J18_43 is gone; now on net VIDEO_MEM_WE: J18.43 (Pin_43)
- net JPA9_9 is gone; now on net SWITCH_OPTION_12: UC6.2 (CP), UC7.2 (CP), UD3.2, UE3.12 (C)
- net UA1_13 is gone; now on net UA1_12: UA1.13 (Q1), UA2.3 (A2)
- net UA7_12 is gone; now on net CLOCK_DIV4: UA7.12, UC4.2, UC4.3, UD5.1, UD5.10, UD5.3
- net UA7_4 is gone; now on net CLOCK_DIV4: UA1.1 (~{MR}), UA4.1 (~{MR})
- net -12v: no longer J1.2 (B)
- net -5V: now also CR1.2 (A), UJ4.21 (VBB_(-5v)), UK4.3 (VO), UK7.21 (VBB_(-5v)); no longer CR5.2 (A)
- net E6_12: no longer UE6.12 (E), UE6.8 (C)
- net E6_13: no longer R19.2, UE6.13 (B)
- net E6_14: no longer R22.1, R23.1, UE6.14 (C)
- net E6_2: no longer R23.2, UE6.2 (B)
- net E6_6: no longer R22.2, UE6.6 (B)
- net E6_9: no longer Q3.3 (C), R21.1, UE6.9 (B)
- net GND: now also R10.2, R19.1, UD8.10 (~{S}), C53.2, C54.2, C55.2, UA8.8 (GND), UF5.8 (GND), UF6.8 (GND), UH6.8 (GND), UJ3.8 (GND), UJ4.12 (GND), UJ4.18 (Program), UK4.1 (GND), UK7.12 (GND), UK7.18 (Program), XA1.7 (GND); no longer C59.1, R20.1, R9.2, UE6.3 (E)
- net J4_1: now also YJ1.1
- net J4_2: now also YJ1.2
- net JPA9_10: now also JPA1.10 (B)
- net JPA9_14: no longer UC6.1 (~{MR}), UC7.1 (~{MR}), UD3.10, UE3.9 (C)
- net JPA9_15: now also JPA1.15 (B)
- net JPA9_16: now also JPA1.16 (B)
- net JPB9_3: no longer UB8.4 (K)
- net JPB9_6: no longer UB8.11 (K)
- net JPB9_8: no longer UB8.8 (J)
- net JPB9_9: now also JPB1.9 (B)
- net JPC9_1: no longer UC4.9
- net JPC9_13: now also JPC1.12 (B), JPC1.13 (B)
- net JPC9_3: no longer UC4.1
- net JPC9_5: no longer UC4.4
- net JPC9_8: no longer UD5.4
- net JPC9_9: now also JPC1.9 (B)
- net Q3_2: no longer CR5.1 (K), Q3.2 (B)
- net UA1_14: now also CR2.2 (A), CR3.2 (A), UC2B1.3 (1Y)
- net UA2_12: no longer UA2.12 (O3), UB6.3
- net UA5_11: no longer UA5.11 (O4)
- net UA5_13: no longer UA5.13 (O2)
- net UA5_14: no longer UA5.14 (O1)
- net UA6_1: now also UA8.1 (~{MR})
- net UA6_11: now also UA8.11 (Q3)
- net UA6_15: now also UA8.15 (TC)
- net UA6_3: now also UA8.3 (D0)
- net UA6_4: now also UA8.4 (D1)
- net UA6_5: now also UA8.5 (D2)
- net UA6_6: now also UA8.6 (D3)
- net UA6_7: now also UA8.7 (CEP)
- net UA7_13: no longer UA7.13, UC6.12 (Q2)
- net UB2_11: no longer UB2.11 (O4), UB5.13
- net UB5_10: no longer UB2.13 (O2), UB5.10
- net UB5_11: no longer UA5.7 (O7), UB5.11, UB5.2
- net UB5_3: no longer UB5.3
- net UB5_5: no longer UA5.10 (O5), UB5.5
- net UB5_9: no longer UA2.7 (O7), UB5.9
- net UB6_1: no longer UA5.12 (O3), UB6.1, UB7.13
- net UB6_11: no longer UA2.15 (O0), UB5.4, UB6.11, UB6.2
- net UB6_13: no longer UB2.15 (O0), UB6.10, UB6.13
- net UB6_9: no longer UA5.9 (O6), UB6.9, UB7.5
- net UB7_1: no longer UA2.9 (O6), UB5.1, UB7.1, UB7.4
- net UB7_11: no longer UA5.15 (O0), UB6.4, UB7.11
- net UB7_3: no longer UB2.12 (O3), UB7.2, UB7.3
- net UB8_9: no longer UB8.12 (C), UB8.9 (C), UD4.8 (J), UD5.8
- net UC2A_3: no longer UC2A1.3 (Q), UC2B1.6 (2A)
- net UC2A_5: no longer C4.2, UC2A1.5 (CV)
- net UC2A_7: no longer C5.2, R6.1, UC2A1.6 (THR), UC2A1.7 (DIS)
- net UC2B_3: no longer CR2.2 (A), CR3.2 (A), UC2B1.3 (1Y)
- net UC3_2: now also UC2.2 (~{Q})
- net UD3_12: no longer UD3.12, UE3.4 (K)
- net UD7_10: no longer UD7.10 (In4), UD8.6 (~{Q})
- net UD8_3: now also C53.1, R11.2
- net UE2_1: no longer UB4.12 (Tc), UE2.1
- net UE2_2: no longer C3.1, R2.1, UE2.2, UE6.1 (C), UH5.2 (~{RESIN})
- net UE2_8: now also UC2.12 (C)
- net UE4_1: no longer UE4.1, UL3.1 (S), UL4.1 (S), UL8.1 (S), UM8.1 (S)
- net UE9_1: now also UH6.7 (Q2)
- net UE9_22: now also UH6.5 (Q1)
- net UE9_23: now also UH6.10 (Q3)
- net UE9_4: now also UF6.10 (Q3)
- net UF2_2: no longer R17.2
- net UF2_3: no longer UF2.3
- net UF3_5: no longer UF4.15 (DO5)
- net UF3_9: no longer UH5.7 (~{STSTB})
- net UF6_1: now also UF5.1 (DIS4)
- net UF6_10: now also UF5.10 (In4)
- net UF6_11: now also UF5.11 (Out5)
- net UF6_12: now also UF5.12 (In5)
- net UF6_9: now also UF5.9 (Out4)
- net UF9_12: now also UF6.12 (Q4)
- net UF9_13: now also UF6.13 (D4)
- net UF9_14: now also UF6.14 (D5)
- net UF9_15: now also UF6.15 (Q5)
- net UF9_2: now also UF6.2 (Q0)
- net UF9_5: now also UF6.5 (Q1)
- net UF9_7: now also UF6.7 (Q2)
- net UH1_6: now also UF5.15 (DIS2)
- net UH3_9: no longer UH2.6, UH3.9
- net UH7_1: no longer UF7.6, UH7.1 (~{MR})
- net UH8_1: no longer UH8.1
- net UH9_12: now also UH6.12 (Q4)
- net UH9_13: now also UH6.13 (D4)
- net UH9_14: now also UH6.14 (D5)
- net UH9_15: now also UH6.15 (Q5)
- net UH9_2: no longer UD8.12 (D)
- net VCC: now also CR5.1 (K), R22.1, R3.2, JPA1.13 (B), R1.1, R15.2, R16.2, RND1.1 (common), RNK1.1 (common), UA8.10 (CET), UA8.16 (VCC), UA8.9 (~{PE}), UC2.13 (~{R}), UF5.16 (VCC), UF6.16 (VCC), UH6.16 (VCC), UJ3.16 (VCC), UJ4.24 (VCC), UK7.24 (VCC), XA1.14 (Vcc); no longer CR4.1 (K), R13.2, R27.2, R3.1, UA1.9 (~{PE}), UD8.10 (~{S})
- net VDD: now also CR4.1 (K), UJ4.19 (VDD_+12v), UK7.19 (VDD_+12v)
- net XA8_1: now also XA1.1 (EN)
- net XA8_8: now also XA1.8 (OUT)
- removed net CR4_2: CR4.2 (A), R20.2, R21.2
- net D0: no longer names the net of UK3.10 (D0)
- net D0: now also UJ3.13 (B3)
- net D1: no longer names the net of UK3.9 (D1)
- net D1: now also UJ3.10 (B2)
- net D2: no longer names the net of UK3.8 (D2)
- net D2: now also UJ3.6 (B1)
- net D3: no longer names the net of UK3.7 (D3)
- net D3: now also UJ3.3 (B0)
- net D4: no longer names the net of UK3.3 (D4), UK5.10 (B2)
- net D5: no longer names the net of UK3.4 (D5), UK5.6 (B1)
- net D6: no longer names the net of UK3.5 (D6), UK5.13 (B3)
- net D7: no longer names the net of UK3.6 (D7), UK5.3 (B0)
- net J17_10 renamed D0_OUT
- net D0_OUT: now also UJ3.14 (R3)
- net J17_11 renamed read_iface_serial_buffer
- net J17_12 renamed D3_OUT
- net D3_OUT: now also UJ3.2 (R0)
- net J17_14 renamed D4_OUT
- net J17_16 renamed D5_OUT
- net J17_17 renamed read_kybd_latch
- net J17_18 renamed D6_OUT
- net J17_20 renamed D7_OUT
- net J17_21 renamed unknown_ram_read_access_1
- net J17_22 renamed D7_IN
- net D7_IN: now also RNK1.4 (R3), UF5.7 (Out3), UJ4.17 (Q8), UK7.17 (Q8)
- net J17_24 renamed D6_IN
- net D6_IN: now also RNK1.5 (R4), UF5.13 (Out6), UJ4.16 (Q7), UK7.16 (Q7)
- net J17_26 renamed D5_IN
- net D5_IN: now also RNK1.6 (R5), UF5.3 (Out1), UJ4.15 (Q6), UK7.15 (Q6)
- net J17_27 renamed write_iface_status
- net J17_28 renamed D4_IN
- net D4_IN: now also RNK1.7 (R6), UF5.5 (Out2), UJ4.14 (Q5), UK7.14 (Q5)
- net J17_29 renamed write_iface_serial_tx_1
- net J17_30 renamed D3_IN
- net D3_IN: now also RNK1.8 (R7), UJ3.4 (D0), UJ4.13 (Q4), UK7.13 (Q4)
- net J17_31 renamed write_iface_serial_tx_0
- net J17_32 renamed D0_IN
- net D0_IN: now also RNK1.3 (R2), UJ3.12 (D3), UJ4.11 (Q3), UK7.11 (Q3)
- net J17_33 renamed write_iface_prnt_tx_1
- net J17_34 renamed D2_IN
- net D2_IN: now also RNK1.2 (R1), UJ3.7 (D1), UJ4.10 (Q2), UK7.10 (Q2)
- net J17_35 renamed write_iface_prnt_tx_0
- net J17_36 renamed D1_IN
- net D1_IN: now also R3.1, UJ3.9 (D2), UJ4.9 (Q1), UK7.9 (Q1); no longer R13.1, UJ6.10 (Data_Out_1)
- net J17_38 renamed SPKR_OUT
- net J17_40 renamed kybd_ready_latch
- net kybd_ready_latch: now also R13.1; no longer R17.1
- net J17_41 renamed unknown_floppy_write_access_1
- net J17_48 renamed KYBD_D7
- net J17_5 renamed VIDEO_ENABLED
- net J17_50 renamed KYBD_D6
- net J17_51 renamed VIDEO_ENABLED1
- net J17_52 renamed KYBD_D5
- net J17_53 renamed INT_0
- net INT_0: now also RND1.8 (R7)
- net J17_54 renamed KYBD_D4
- net J17_55 renamed INT_1
- net INT_1: now also RND1.7 (R6)
- net J17_56 renamed KYBD_D3
- net J17_57 renamed INT_2
- net INT_2: now also RND1.6 (R5)
- net J17_58 renamed KYBD_D0
- net J17_59 renamed INT_3
- net INT_3: now also RND1.5 (R4)
- net J17_6 renamed D1_OUT
- net D1_OUT: now also UC2.1 (J), UJ3.11 (R2)
- net J17_60 renamed KYBD_D2
- net J17_61 renamed unused_2
- net J17_62 renamed KYBD_D1
- net J17_63 renamed INT_6
- net INT_6: now also RND1.4 (R3)
- net J17_64 renamed /read_iface_status0
- net J17_65 renamed INT_5
- net INT_5: now also RND1.3 (R2)
- net J17_66 renamed D1_OUT6
- net J17_67 renamed INT_7
- net INT_7: now also RND1.2 (R1)
- net J17_68 renamed enable_video_out
- net J17_69 renamed D1_OUT9
- net J17_7 renamed read_iface_status
- net J17_70 renamed read_iface_status0
- net J17_71 renamed read_iface_status1
- net J17_72 renamed read_iface_status2
- net J17_75 renamed unused_1
- net J17_76 renamed /PWM_OUT
- net J17_77 renamed read_iface_status7
- net J17_78 renamed RDYIN
- net RDYIN: no longer R3.2
- net J17_79 renamed read_iface_status9
- net read_iface_status9: now also UF1.8
- net J17_8 renamed D2_OUT
- net D2_OUT: now also UC2.4 (K), UJ3.5 (R1)
- net J17_80 renamed D2_OUT0
- net J17_9 renamed read_iface_prnt_status
- net J18_1 renamed VIDEO_MEM_D1
- net VIDEO_MEM_D1: now also UE7.6 (In3), UK9.10 (Data_Out_1), UL9.10 (Data_Out_1), UF6.11 (D3), UF6.6 (D2)
- net J18_10 renamed VIDEO_MEM_D4
- net VIDEO_MEM_D4: now also UF5.4 (In2), UH6.6 (D2)
- net J18_11 renamed MEM_PAGE_2
- net J18_12 renamed VIDEO_MEM_D5
- net VIDEO_MEM_D5: now also UF5.2 (In1), UH6.11 (D3)
- net J18_13 renamed MEM_PAGE_1
- net MEM_PAGE_1: now also UJ4.20 (~{CS}_(PE))
- net J18_14 renamed VIDEO_MEM_D6
- net VIDEO_MEM_D6: now also UF5.14 (In6), UH6.4 (D1)
- net J18_15 renamed MEM_PAGE_0
- net MEM_PAGE_0: now also UK7.20 (~{CS}_(PE))
- net J18_16 renamed VIDEO_MEM_D7
- net VIDEO_MEM_D7: now also UF5.6 (In3), UH6.3 (D0)
- net J18_17 renamed /CPU_STATUS_INTA
- net /CPU_STATUS_INTA: now also UF1.13; no longer J18.17 (Pin_17)
- net J18_18 renamed CPU_STATUS_INP
- removed net J18_2: J18.2 (Pin_2), UE7.6 (In3), UK9.10 (Data_Out_1), UL9.10 (Data_Out_1)
- net J18_23 renamed VIDEO_MEM_WE
- net J18_25 renamed /D01N
- net J18_27 renamed /CPU_STATUS_MEMR
- net /CPU_STATUS_MEMR: now also J18.17 (Pin_17)
- net J18_29 renamed /CPU_STATUS_M1
- net J18_3 renamed MEM_PAGE_6
- net J18_30 renamed EDGE_A0
- net J18_31 renamed COMPSITE_VIDEO_OUT
- net COMPSITE_VIDEO_OUT: now also R10.1, R9.2; no longer R10.2, R9.1
- net J18_32 renamed EDGE_A1
- net J18_33 renamed unused_3
- net J18_34 renamed EDGE_A2
- net J18_35 renamed unused_4
- net J18_36 renamed EDGE_A3
- net J18_37 renamed unused_5
- net J18_38 renamed EDGE_A4
- net J18_39 renamed unused_6
- net J18_40 renamed EDGE_A5
- net J18_41 renamed unused_7
- net J18_42 renamed EDGE_A6
- net J18_44 renamed EDGE_A7
- net J18_45 renamed /WR_bufd
- net J18_46 renamed EDGE_A8
- net J18_47 renamed VIDEO_BUS_PAGE_7
- net J18_48 renamed EDGE_A9
- net J18_49 renamed VIDEO_BUS_PAGE_6
- net J18_5 renamed MEM_PAGE_5
- net J18_50 renamed EDGE_A10
- net J18_51 renamed VIDEO_BUS_PAGE_5
- net J18_52 renamed EDGE_A11
- net J18_53 renamed VIDEO_BUS_PAGE_4
- net J18_54 renamed EDGE_A12
- net J18_55 renamed VIDEO_BUS_PAGE_3
- net J18_56 renamed EDGE_A13
- net J18_57 renamed VIDEO_BUS_PAGE_2
- net J18_58 renamed EDGE_A14
- net J18_59 renamed VIDEO_MEM_A7
- net J18_6 renamed VIDEO_MEM_D2
- net VIDEO_MEM_D2: now also UF6.4 (D1)
- net J18_60 renamed EDGE_A15
- net J18_61 renamed VIDEO_MEM_A6
- net J18_62 renamed RAMSEL_BANK_6
- net J18_63 renamed VIDEO_MEM_A5
- net J18_64 renamed RAMSEL_BANK_5
- net J18_65 renamed VIDEO_MEM_A4
- net J18_66 renamed RAMSEL_BANK_4
- net J18_67 renamed VIDEO_MEM_A0
- net J18_68 renamed RAMSEL_BANK_3
- net J18_69 renamed VIDEO_MEM_A1
- net J18_7 renamed MEM_PAGE_4
- net J18_70 renamed RAMSEL_BANK_2
- net J18_71 renamed VIDEO_MEM_A2
- net J18_72 renamed RAMSEL_BANK_1
- net J18_73 renamed VIDEO_MEM_A3
- net J18_74 renamed RAMSEL_BANK_0
- net J18_8 renamed VIDEO_MEM_D3
- net VIDEO_MEM_D3: now also UF6.3 (D0)
- net J18_9 renamed MEM_PAGE_3
- net JPA9_1 renamed SWITCH_OPTION_9
- net SWITCH_OPTION_9: now also C55.1, JPA1.1 (A), JPA1.2 (A), UA6.3
- net JPA9_12 renamed CLOCK_DIV4
- net CLOCK_DIV4: now also UC4.4, JPA1.12 (B), JPC1.5 (A), JPC1.6 (A), UA6.4, UA8.13 (Q1)
- net JPA9_4 renamed SWITCH_OPTION_10
- net SWITCH_OPTION_10: now also JPA1.3 (A), JPA1.4 (A)
- net JPA9_5 renamed SWITCH_OPTION_11
- net SWITCH_OPTION_11: now also JPA1.5 (A), JPA1.6 (A)
- net JPA9_7 renamed SWITCH_OPTION_12
- net SWITCH_OPTION_12: now also JPA1.7 (A), JPA1.8 (A), JPA1.9 (B), UF6.9 (Cp), UH6.9 (Cp); no longer UB3.3 (C)
- net JPB9_1 renamed SWITCH_OPTION_5
- net SWITCH_OPTION_5: now also JPB1.1 (A), JPB1.2 (A)
- net JPB9_10: no longer names the net of UB5.8
- net JPB9_10: now also JPB1.10 (B)
- net JPB9_11: no longer names the net of UB6.6
- net JPB9_11: now also JPB1.11 (B)
- net JPB9_12: no longer names the net of UB7.8
- net JPB9_12: now also JPB1.12 (B)
- net JPB9_13: no longer names the net of UB6.8
- net JPB9_13: now also JPB1.13 (B)
- net JPB9_14: no longer names the net of UB7.6
- net JPB9_14: now also JPB1.14 (B)
- net JPB9_15: no longer names the net of UB6.12
- net JPB9_15: now also JPB1.15 (B)
- net JPB9_16: no longer names the net of UB7.12
- net JPB9_16: now also JPB1.16 (B)
- net JPC9_10: no longer names the net of UC8.9 (O6)
- net JPC9_10: now also JPC1.10 (B)
- net JPC9_11: no longer names the net of UC8.11 (O4)
- net JPC9_11: now also JPC1.11 (B)
- net JPC9_14: no longer names the net of UC8.12 (O3)
- net JPC9_14: now also JPC1.14 (B)
- net JPC9_15: no longer names the net of UC8.13 (O2)
- net JPC9_15: now also JPC1.15 (B)
- net JPC9_16: no longer names the net of UC8.14 (O1)
- net JPC9_16: now also JPC1.16 (B)
- net Q1_2: no longer names the net of Q1.2 (B), R14.2
- net Q1_2: now also UF8.8
- net Q1_3: no longer names the net of C6.2, Q1.3 (C), Q2.2 (B), R7.2, R8.2
- net Q2_1: no longer names the net of Q2.1 (E)
- net Q2_1: now also R9.1; no longer R10.1
- net Three-Resistors: no longer names the net of R18.1
- net Three-Resistors: now also CR4.2 (A), R20.1; no longer R19.1
- net UA1_2 renamed UKNOWN_PULSE_oiewd
- net UA3_12: no longer names the net of UA3.12, UF8.13
- net UA3_5 renamed /SWITCH_OPTION_12
- net /SWITCH_OPTION_12: now also UB3.3 (C)
- net UA3_6: no longer names the net of UA3.6, UD3.3
- net UA4_15: no longer names the net of UA1.7 (CEP), UA4.15 (TC)
- net UA6_14 renamed CLOCK_DIV2
- net CLOCK_DIV2: now also UA8.14 (Q0)
- net UA7_11: no longer names the net of UA7.8
- net UA7_11: no longer UD9.9 (Clock)
- net UB3_4: no longer names the net of UB3.2 (D), UB3.4 (~{S})
- net UB3_6: no longer names the net of UB3.6 (~{Q})
- net UB3_9: no longer names the net of UB3.1 (~{R}), UB3.9 (Q)
- net UB8_6 renamed /SWITCH_OPTION_7 _8_LATCH
- net UC3_11: no longer names the net of UC3.11 (K), UC4.12
- net UC3_3 renamed PWM_OUT
- net PWM_OUT: now also UC2.3 (Q)
- net UC3_6: no longer names the net of UC3.6 (~{Q}), UD3.5
- net UC3_8: no longer names the net of UC3.8 (J), UC4.8
- net UC5_6: no longer names the net of UC5.6 (E3), UE3.3 (Q)
- net UD1_1: no longer names the net of R12.2, UD1.1 (I4)
- net UD2_14 renamed CPU_STATUS_HLTA
- net UD4_11: no longer names the net of UD4.11 (K), UD5.12
- net UD4_12: no longer names the net of UD3.4, UD9.7 (S1)
- net UD4_12: no longer UD4.12 (C)
- net UD4_2 renamed /VIDEO_ENABLE
- net UD5_13: no longer names the net of UC5.12 (O3), UD5.13
- net UE1_4: no longer names the net of UE1.4 (E1), UE4.8
- net UE1_5: no longer names the net of UE1.5 (E2), UE4.11
- net UE4_5 renamed PIXEL_GENERATOR_OUT
- net UE5_1: no longer names the net of UE5.1 (CP1..3), UE5.12 (Q0)
- net UE5_11: no longer names the net of UE5.11 (Q3), UF7.9
- net UE8_20: no longer names the net of UE8.20 (CS1/~{CS1}), UH8.8
- net UF3_12: no longer names the net of UH2.4
- net UF3_12: now also UF1.12
- net UF3_3 renamed CPU_STATUS_STACK
- net CPU_STATUS_STACK: now also UF1.3
- net UF3_6: no longer names the net of UH3.5
- net UF3_6: now also UF1.6
- net UF4_17 renamed CPU_STATUS_M1
- net UF4_6 renamed /CPU_STATUS_WO
- net UF7_3 renamed SWITCH_OPTION_7 _8_LATCH
- net UF7_5: no longer names the net of UF7.5, UF8.6
- net UF8_11: no longer names the net of UF8.11, UH4.3
- net UF8_8: no longer names the net of R14.1
- net UF8_8: no longer UF8.8
- net UH1_4: no longer names the net of UH1.4, UH3.10, UH3.11, UH3.12
- net UH1_5 renamed D0IN_bufd
- net D0IN_bufd: now also UJ3.1 (~{R/E}), UJ3.15 (B/E)
- net UH1_8: no longer names the net of UB3.12 (D), UH1.8
- net UH1_9: no longer names the net of UH1.10, UH1.9, UH3.8
- net UH3_6: no longer names the net of UH2.5, UH3.6
- net UH4_13: no longer names the net of UH4.13, UK3.17 (D0IN)
- net UH4_2 renamed A15
- net UH4_5 renamed CPU_STATUS_MEMR
- net UH5_1 renamed CPU_RESET
- net UH5_11 renamed CLOCK_PHASE_0
- net UH5_12: no longer names the net of UH5.12 (OSC)
- net UH5_13: no longer names the net of UH5.13 (TANK)
- net UH5_4 renamed READY
- net UH5_5 renamed CPU_SYNC
- net UH5_6 renamed CLOCK_PHASE_1_TTL
- net UH7_2 renamed VIDEO_ENABLE
- net UJ1_11 renamed A2
- net A2: now also UJ4.6 (A2), UK7.6 (A2)
- net UJ1_13 renamed A4
- net A4: now also UJ4.4 (A4), UK7.4 (A4)
- net UJ1_9 renamed A0
- net A0: now also UJ4.8 (A0), UK7.8 (A0)
- net UJ2_10: no longer names the net of UJ2.10 (In4), UK3.25 (A0)
- net UJ2_12: no longer names the net of UJ2.12 (In5), UK3.27 (A2)
- net UJ2_14: no longer names the net of UJ2.14 (In6), UK3.30 (A4)
- net UJ2_2: no longer names the net of UJ2.2 (In1), UK3.31 (A5)
- net UJ2_3 renamed A5
- net A5: now also UJ4.3 (A5), UK7.3 (A5)
- net UJ2_4: no longer names the net of UJ2.4 (In2), UK3.29 (A3)
- net UJ6_1 renamed A3
- net A3: now also UJ4.5 (A3), UK7.5 (A3)
- net UJ6_3 renamed A1
- net A1: now also UK7.7 (A1)
- net UJ6_7 renamed A7
- net A7: now also UJ4.1 (A7), UK7.1 (A7)
- net UK1_11 renamed A8
- net A8: now also UJ4.23 (A8), UK7.23 (A8)
- net UK1_13 renamed A10
- net UK1_9 renamed A6
- net A6: now also UJ4.2 (A6), UK7.2 (A6)
- net UK2_10: no longer names the net of UK2.10 (In4), UK3.32 (A6)
- net UK2_12: no longer names the net of UK2.12 (In5), UK3.34 (A8)
- net UK2_14: no longer names the net of UK2.14 (In6), UK3.1 (A10)
- net UK2_2: no longer names the net of UK2.2 (In1), UK3.40 (A11)
- net UK2_3 renamed A11
- net UK2_4: no longer names the net of UK2.4 (In2), UK3.35 (A9)
- net UK2_5 renamed A9
- net A9: now also UJ4.22 (A9), UK7.22 (A9)
- net UK2_6: no longer names the net of UK2.6 (In3), UK3.33 (A7)
- net UK3_15 renamed CLOCK_PHASE_1
- net UK3_16: no longer names the net of UK3.16 (INTE)
- net UK3_18: no longer names the net of UK3.18 (~{WR}), UL2.2 (In1)
- net UK3_26: no longer names the net of UJ2.6 (In3), UK3.26 (A1)
- net UK5_15: no longer names the net of UH3.4
- net UK5_15: now also UF1.4
- net UK6_19 renamed RAMSEL_BANK_7
- net UL1_11 renamed A14
- net UL1_12: no longer names the net of UL1.12, UM1.4 (E1)
- net UL1_2: no longer names the net of UL1.2, UM1.5 (E2)
- net UL1_9 renamed A12
- net UL2_10: no longer names the net of UK3.37 (A12), UL2.10 (In4)
- net UL2_12: no longer names the net of UK3.39 (A14), UL2.12 (In5)
- net UL2_4: no longer names the net of UK3.36 (A15), UL2.4 (In2)
- net UL2_6: no longer names the net of UK3.38 (A13), UL2.6 (In3)
- net UL2_7 renamed A13
- net UL3_12: no longer names the net of UL3.12 (Zd), UM3.10, UM3.11
- net UL3_5: no longer names the net of UL3.5 (I0b), UM5.6
- net UL3_7: no longer names the net of UL3.7 (Zb), UM2.2
- net UL4_11: no longer names the net of UL4.11 (I0c), UM5.12
- net UL4_12 renamed VIDEO_MEM_A10
- net UL4_7 renamed VIDEO_MEM_A11
- net UM1_6: no longer names the net of UM1.6 (E3), UM2.8
- net UM2_4: no longer names the net of UM2.3, UM2.4
- net UM2_5: no longer names the net of UL3.9 (Zc), UM2.5
- net UM2_6 renamed VIDEO_BUS_SEL_0
- net UM3_13: no longer names the net of UF2.12, UM3.13
- net UM3_13: no longer C59.2, UE6.7 (C)
- net UM3_8 renamed VIDEO_BUS_SEL_1
- net UM3_9: no longer names the net of UL3.4 (Za), UM3.9
- net UM4_1 renamed VIDEO_MEM_A9
- net UM4_14 renamed VIDEO_BUS_PAGE_1
- net UM4_15 renamed VIDEO_BUS_PAGE_0
- net UM7_10 renamed UNKNOWN_SWITCH_OPTION
- new net: UE6.12 (E), UE6.8 (C)
- new net: R20.2, UE6.13 (B)
- new net: R16.1, R17.1, R23.1, UE6.14 (C)
- new net: C5.2, R6.1, UC2A1.6 (THR), UC2A1.7 (DIS)
- new net: UD7.10 (In4), UD8.6 (~{Q})
- new net: C54.1, R13.2
- new net: Q3.3 (C), R21.1, UE6.9 (B)
- new net: R23.2, UE6.2 (B)
- new net: UH2.6, UH3.9
- new net: UB2.13 (O2), UB5.10
- new net: UA5.7 (O7), UB5.11, UB5.2
- new net: UA2.7 (O7), UB5.9
- new net: UB8.12 (C), UB8.9 (C), UD4.8 (J), UD5.8
- new net: CR5.2 (A), R19.2, R21.2
- new net: R17.2, UE6.6 (B)
- new net: UA2.12 (O3), UB6.3
- new net: UA5.15 (O0), UB6.4, UB7.11
- new net: UA5.10 (O5), UB5.5
- new net: UA5.12 (O3), UB6.1, UB7.13
- new net: UA5.9 (O6), UB6.9, UB7.5
- new net: UF1.9, UH5.7 (~{STSTB})
- new net: UF7.6, UH7.1 (~{MR})
- new net: UA2.15 (O0), UB5.4, UB6.11, UB6.2
- new net: UA2.9 (O6), UB5.1, UB7.1, UB7.4
- new net: UA7.13, UC6.12 (Q2)
- new net: UA6.10, UA8.2 (CP)
- new net: JPC1.3 (A), JPC1.4 (A)
- new net: R11.1, UF2.3
- new net: UB2.11 (O4), UB5.13
- new net: JPB1.7 (A), JPB1.8 (A)
- new net: CR1.1 (K), R22.2
- new net: UB2.12 (O3), UB7.2, UB7.3
- new net: UB2.15 (O0), UB6.10, UB6.13
- new net: UB4.12 (Tc), UE2.1
- new net: C4.2, UC2A1.5 (CV)
- new net: UD3.12, UE3.4 (K)
- new net BEEPER_OUT: UC2A1.3 (Q), UC2B1.6 (2A)
- new net CLOCK_DIV8: JPA1.11 (B), UA8.12 (Q2)
- new net CLOCK_GENERATOR_OUT: UA6.11, UD9.9 (Clock)
- new net CPU_STATUS_OUT: UF1.5, UF4.15 (DO5)
- new net DOT_GENERATOR_MODE: UD4.12 (C)
- new net J1_2: J1.2 (B), UK4.2 (VI)
- new net POWER_GOOD: C59.2, R15.1, UE6.7 (C)
- new net SWITCH_OPTION_1: JPC1.1 (A), JPC1.2 (A), UC4.9
- new net SWITCH_OPTION_2: UC4.1
- new net SWITCH_OPTION_4: JPC1.7 (A), JPC1.8 (A), UD5.4
- new net SWITCH_OPTION_6: JPB1.3 (A), JPB1.4 (A), UB8.4 (K)
- new net SWITCH_OPTION_7: JPB1.5 (A), JPB1.6 (A), UB8.11 (K)
- new net SWITCH_OPTION_8: UB8.8 (J)
- new net SYSTEM_RESET_PULSE: C3.1, R2.1, UE2.2, UE6.1 (C), UH5.2 (~{RESIN})
- new net UNKNOWN_SIGNAL_234: UD8.12 (D)
- new net VIDEO_BUS_SELECT: UE4.1, UH6.1 (~{Mr}), UL3.1 (S), UL4.1 (S), UL8.1 (S), UM8.1 (S)
- new net /UKNOWN_PULSE_oiewd: JPA1.14 (B), UC6.1 (~{MR}), UD3.10, UE3.9 (C)
- no-connect marks 175 -> 178
Other:
- note added: "/Q"
- note added: "0x50"
- note added: "0x58 interface card output register low"
- note added: "0x60 interface card output register high"
- note added: "0x78 write state to interface card"
- note added: "2MHZ"
- note added: "Analog"
- note added: "BUS DRIVERS"
- note added: "Boot ROM 0x0000"
- note added: "Bus Pullups"
- note added: "CPU Core control"
- note added: "CPU Output bus"
- note added: "CPU input bus"
- note added: "Clock Generators and Dividers"
- note added: "FIXME"
- note added: "FIXME i lost the connections here"
- note added: "FIXME two drivers"
- note added: "FIXME,two drivers?"
- note added: "FIXME?"
- note added: "FLIP FLOP"
- note added: "FONT PIXEL GENERATOR"
- note added: "Memory Mappers"
- note added: "OR"
- note added: "Options And Configuration"
- note added: "Ox40"
- note added: "PHARS WARNING: I have done a lot of feng shui here to push things into some shapes that make sense, unfortunatly every now and again a renaming mistake or wire/bus may get away from me but i try to label them with a "fixme" as i notice them"
- note added: "POWER GOOD STARTUP TIMER?"
- note added: "Port Mappers"
- note added: "Port Read Select"
- note added: "Port Write"
- note added: "Port Write Select"
- note added: "R"
- note added: "S"
- note added: "VIDEO ANALOG OUT"
- note added: "VIDEO BUS ACCESS DECODER"
- note added: "Video Memory Bus Access Decoder"
- note added: "Video Memory Bus To CPU Bus Interface"
- note added: "Voltage Regulation"
- note added: "clock divider"
- note added: "fixme"
- note added: "i CALL TWO SIGNALS HERE VIDEO OUT WHICH MEANS IM WRONG.. THIS MIGHT BE SOME ANALOG TRICKERY TO GENERATE THE NTSC CORRECTLY SO I'LL NEED TO DO MORE TO FIGURE OUT THE RIGHT NAME"
- note added: "i detached this from the group it was connected to because I suspect it belongs here"
- note added: "interrupt priority decoder"
- note added: "keyboard interface"
- note added: "port read"
- note added: "read interface card "printer status" register"
- note added: "read interface card buffer"
- note added: "read interface card register"
- note added: "read keyboard keys"
- note added: "read keyboard status latch and key modifiers"
- note added: "something to do with transmit 0x68"
- note added: "something to do with transmit 0x70"
- note removed: "1920/480 Jumper Bus"
- note removed: "All connections only go to the "Jacks" on the backplne (J17 & J18), so there are no wires to draw"
- note removed: "Composite Video"
- note removed: "D0-D7"
- note removed: "Data Bus?"
- note removed: "Interface Board"
- note removed: "Jumpers currently set to 1920 mode"
- note removed: "Keyboard Enable"
- note removed: "KiCad Bus Range Creator https://bit.ly/KiCadBRC"
- note removed: "Magic 555 Timer and other Entrex VooDoo"
- note removed: "Misc. Control Line Bus Don't know what they control yet just needed the signalas over on the other side"
- note removed: "Mystery Section"
- note removed: "Opt = Option, choice, setting, selection, etc"
- note removed: "RAM Bus"
- note removed: "This area can be moved it its own section"
- note removed: "WARNING: Until refined & corrected, Global Label tag arrows may not indicate the proper signal in/out direction. IN was used as default when KiCad Symbols (components) were not clear on In vs Out signals, so always check component datasheets when in doubt."
- note removed: "What is all this nonsense?"
- note removed: "to UC1 pin 13 74LS138"
- moved on the sheet: CR2, CR3, Q1, R14, R23, R27, UA2, UA3A, UA4, UA5, UA7C, UA7F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
