File: Trapezoid_Terminal/Interface Board/Entrex Trapezoid Interface Board v23.kicad_sch (KiCad schematic)
At the start: 103 parts, among them P15 Conn_02x40_Odd_Even_Shielded, SW1 SW_DIP_x08

Commit message: u34_13!
Connections:
- net u1_10 is gone; now on net u34_13: UA1.14 (~{CLR}), UA2.14 (~{CLR}), UA5.3 (~{R}), UA5.8 (~{R}), UA8.10 (~{S}), UB5.1 (~{R}), UB6.13, UB6.8
- net u16_15 renamed u4_3
Changed lines of the file:
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@@
   (junction (at 737.87 233.68) (diameter 0) (color 0 0 0 0)
   )
+  (junction (at 582.93 605.79) (diameter 0) (color 0 0 0 0)
+  )
   (junction (at 513.08 458.47) (diameter 0) (color 0 0 0 0)
   )
@@
   (junction (at 792.48 459.74) (diameter 0) (color 0 0 0 0)
   )
+  (junction (at 831.85 463.55) (diameter 0) (color 0 0 0 0)
+  )
   (junction (at 217.17 67.945) (diameter 0) (color 0 0 0 0)
   )
@@
   (junction (at 602.615 633.095) (diameter 0) (color 0 0 0 0)
   )
+  (junction (at 551.815 634.365) (diameter 0) (color 0 0 0 0)
+  )
   (junction (at 302.26 167.005) (diameter 0) (color 0 0 0 0)
   )
@@
     (stroke (width 0) (type default))
   )
+  (wire (pts (xy 831.85 605.79) (xy 582.93 605.79))
+    (stroke (width 0) (type default))
+  )
   (wire (pts (xy 380.365 539.115) (xy 380.365 530.225))
     (stroke (width 0) (type default))
@@
     (stroke (width 0) (type default))
   )
-  (wire (pts (xy 583.565 634.365) (xy 360.68 634.365))
+  (wire (pts (xy 583.565 634.365) (xy 551.815 634.365))
     (stroke (width 0) (type default))
   )
@@
     (stroke (width 0) (type default))
   )
-  (wire (pts (xy 551.815 605.79) (xy 551.815 691.515))
+  (wire (pts (xy 551.815 605.79) (xy 551.815 634.365))
     (stroke (width 0) (type default))
   )
@@
     (stroke (width 0) (type default))
   )
+  (wire (pts (xy 551.815 634.365) (xy 360.68 634.365))
+    (stroke (width 0) (type default))
+  )
   (wire (pts (xy 140.97 76.2) (xy 140.97 115.57))
     (stroke (width 0) (type default))
@@
     (stroke (width 0) (type default))
   )
+  (wire (pts (xy 551.815 634.365) (xy 551.815 691.515))
+    (stroke (width 0) (type default))
+  )
   (wire (pts (xy 206.375 790.575) (xy 211.455 790.575))
     (stroke (width 0) (type default))
@@
     (stroke (width 0) (type default))
   )
+  (wire (pts (xy 831.85 463.55) (xy 831.85 605.79))
+    (stroke (width 0) (type default))
+  )
   (wire (pts (xy 392.43 422.91) (xy 455.93 422.91))
     (stroke (width 0) (type default))
@@
     (effects (font (size 1.27 1.27)) (justify left bottom))
   )
-  (label "u1_10" (at 864.87 463.55 0) (fields_autoplaced)
-    (effects (font (size 1.27 1.27)) (justify left bottom))
-  )
   (label "u11_5" (at 472.44 471.17 0) (fields_autoplaced)
     (effects (font (size 1.27 1.27)) (justify left bottom))
@@
     (effects (font (size 0.25 0.25)) (justify left bottom))
   )
+  (label "u34_13" (at 864.87 463.55 0) (fields_autoplaced)
+    (effects (font (size 1.27 1.27)) (justify left bottom))
+  )
   (label "u4_12" (at 175.895 248.285 0) (fields_autoplaced)
     (effects (font (size 1.27 1.27)) (justify left bottom))
@@
     (effects (font (size 1.27 1.27)) (justify left bottom))
   )
-  (label "u1_10" (at 865.505 397.51 0) (fields_autoplaced)
-    (effects (font (size 1.27 1.27)) (justify left bottom))
-  )
   (label "P15_45" (at 164.465 260.985 0) (fields_autoplaced)
     (effects (font (size 1.27 1.27)) (justify left bottom))
@@
     (effects (font (size 1.27 1.27)) (justify left bottom))
   )
+  (label "u34_13" (at 864.87 397.51 0) (fields_autoplaced)
+    (effects (font (size 1.27 1.27)) (justify left bottom))
+  )
   (label "P15_21" (at 793.115 166.37 0) (fields_autoplaced)
     (effects (font (size 1.27 1.27)) (justify left bottom))
@@
     )
   )
-  (global_label "u1_10" (shape input) (at 624.205 691.515 270) (fields_autoplaced)
+  (global_label "u34_13" (shape input) (at 624.205 691.515 270) (fields_autoplaced)
     (effects (font (size 0.8 0.8)) (justify right))
     (property "Intersheetrefs" "${INTERSHEET_REFS}" (at 624.205 696.9643 90)
@@
     )
   )
+  (global_label "u4_3" (shape input) (at 285.75 183.515 0) (fields_autoplaced)
+    (effects (font (size 1.27 1.27)) (justify left))
+    (property "Intersheetrefs" "${INTERSHEET_REFS}" (at 293.1914 183.515 0)
+      (effects (font (size 1.27 1.27)) (justify left) hide)
+    )
+  )
   (global_label "P15_11" (shape input) (at 939.165 398.78 180) (fields_autoplaced)
     (effects (font (size 0.8 0.8)) (justify right))
@@
     )
   )
-  (global_label "u1_10" (shape input) (at 520.065 509.905 180) (fields_autoplaced)
+  (global_label "u34_13" (shape input) (at 520.065 509.905 180) (fields_autoplaced)
     (effects (font (size 0.8 0.8)) (justify right))
     (property "Intersheetrefs" "${INTERSHEET_REFS}" (at 514.6157 509.905 0)
@@
     )
   )
-  (global_label "u16_15" (shape input) (at 285.75 183.515 0) (fields_autoplaced)
-    (effects (font (size 0.8 0.8)) (justify left))
-    (property "Intersheetrefs" "${INTERSHEET_REFS}" (at 291.9612 183.515 0)
-      (effects (font (size 0.8 0.8)) (justify left) hide)
-    )
-  )
   (global_label "u4_2" (shape input) (at 409.575 164.465 180) (fields_autoplaced)
     (effects (font (size 0.8 0.8)) (justify right))
@@
     )
   )
-  (global_label "u1_10" (shape input) (at 582.93 605.79 270) (fields_autoplaced)
+  (global_label "u34_13" (shape input) (at 582.93 605.79 270) (fields_autoplaced)
     (effects (font (size 0.8 0.8)) (justify right))
     (property "Intersheetrefs" "${INTERSHEET_REFS}" (at 582.93 611.2393 90)
@@
     )
   )
-  (global_label "u1_10" (shape input) (at 520.7 536.575 180) (fields_autoplaced)
+  (global_label "u34_13" (shape input) (at 520.7 536.575 180) (fields_autoplaced)
     (effects (font (size 0.8 0.8)) (justify right))
     (property "Intersheetrefs" "${INTERSHEET_REFS}" (at 515.2507 536.575 0)
@@
     )
   )
-  (global_label "u1_10" (shape input) (at 681.355 704.215 180) (fields_autoplaced)
+  (global_label "u34_13" (shape input) (at 681.355 704.215 180) (fields_autoplaced)
     (effects (font (size 0.8 0.8)) (justify right))
     (property "Intersheetrefs" "${INTERSHEET_REFS}" (at 675.9057 704.215 0)
@@
     )
   )
-  (global_label "u1_10" (shape output) (at 668.655 704.215 0) (fields_autoplaced)
+  (global_label "u34_13" (shape output) (at 668.655 704.215 0) (fields_autoplaced)
     (effects (font (size 0.8 0.8)) (justify left))
     (property "Intersheetrefs" "${INTERSHEET_REFS}" (at 674.1043 704.215 0)
@@
     )
   )
-  (global_label "u1_10" (shape input) (at 831.85 397.51 180) (fields_autoplaced)
+  (global_label "u34_13" (shape input) (at 831.85 397.51 180) (fields_autoplaced)
     (effects (font (size 0.8 0.8)) (justify right))
     (property "Intersheetrefs" "${INTERSHEET_REFS}" (at 826.4007 397.51 0)

Commit message: IO Testing
Other:
- note added: "Clock Input"
- note added: "Data Input"
- note added: "Strobe Input"
- note removed: "Input 1"
- note removed: "Input 2"
- note removed: "Input 3"
Changed lines of the file:
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@@
     (effects (font (size 3 3) (thickness 1) bold (color 255 38 190 1)) (justify right bottom))
   )
-  (text "Input 2\n" (at 123.825 249.555 0)
+  (text "Clock Input\n" (at 123.825 249.555 0)
     (effects (font (size 1.27 1.27)) (justify left bottom))
   )
@@
     (effects (font (size 3 3) (thickness 1) bold (color 0 0 132 1)) (justify right bottom))
   )
-  (text "Input 2\n" (at 110.49 82.55 0)
+  (text "Clock Input\n" (at 107.95 82.55 0)
     (effects (font (size 1.27 1.27)) (justify left bottom))
   )
@@
     (effects (font (size 1.27 1.27)) (justify left bottom))
   )
-  (text "Input 3\n\n" (at 111.125 93.345 0)
+  (text "Strobe Input\n\n" (at 107.315 93.345 0)
     (effects (font (size 1.27 1.27)) (justify left bottom))
   )
@@
     (effects (font (size 3 3) (thickness 1) bold (color 18 244 255 1)) (justify left bottom))
   )
-  (text "Input 1" (at 92.71 73.025 0)
+  (text "Data Input" (at 92.71 73.025 0)
     (effects (font (size 1.27 1.27)) (justify left bottom))
   )
@@
     (effects (font (size 3 3) (thickness 1) bold (color 18 244 255 1)) (justify left bottom))
   )
-  (text "Input 1" (at 114.935 234.315 0)
+  (text "Data Input" (at 112.395 234.315 0)
     (effects (font (size 1.27 1.27)) (justify left bottom))
   )
@@
     (effects (font (size 3 3) (thickness 1) bold (color 0 0 132 1)) (justify right bottom))
   )
-  (text "Input 2\n" (at 132.715 237.49 0)
+  (text "Clock Input\n" (at 132.715 237.49 0)
     (effects (font (size 1.27 1.27)) (justify left bottom))
   )
@@
     (effects (font (size 3 3) (thickness 1) bold (color 5 102 8 1)) (justify right bottom))
   )
-  (text "Input 3\n\n" (at 133.35 242.57 0)
+  (text "Strobe Input\n\n" (at 132.08 241.935 0)
     (effects (font (size 1.27 1.27)) (justify left bottom))
   )
@@
     (effects (font (size 3 3) (thickness 1) bold (color 18 244 255 1)) (justify right bottom))
   )
-  (text "Input 1" (at 92.71 79.375 0)
+  (text "Data Input" (at 92.71 79.375 0)
     (effects (font (size 1.27 1.27)) (justify left bottom))
   )
@@
     (effects (font (size 3 3) (thickness 1) bold (color 255 38 190 1)) (justify right bottom))
   )
-  (text "Input 2\n" (at 100.965 95.25 0)
+  (text "Clock Input\n" (at 100.965 95.25 0)
     (effects (font (size 1.27 1.27)) (justify left bottom))
   )
@@
     (effects (font (size 3 3) (thickness 1) bold (color 5 102 8 1)) (justify right bottom))
   )
-  (text "Input 3\n\n" (at 111.125 87.63 0)
+  (text "Strobe Input\n\n" (at 107.315 87.63 0)
     (effects (font (size 1.27 1.27)) (justify left bottom))
   )
@@
     (effects (font (size 3 3) (thickness 1) bold (color 18 244 255 1)) (justify left bottom))
   )
-  (text "Input 3\n\n" (at 133.35 248.285 0)
+  (text "Strobe Input\n\n" (at 132.08 248.285 0)
     (effects (font (size 1.27 1.27)) (justify left bottom))
   )
@@
     (effects (font (size 1.27 1.27) (color 255 30 30 1)) (justify left bottom))
   )
-  (text "Input 1" (at 114.935 227.965 0)
-    (effects (font (size 1.27 1.27)) (justify left bottom))
-  )
+  (text "Data Input" (at 112.395 227.965 0)
+    (effects (font (size 1.27 1.27)) (justify left bottom))
+  )
