File: Trapezoid_Terminal/Interface Board/Entrex Trapezoid Interface Board v23.kicad_sch (KiCad schematic)
At the start: 103 parts, among them P15 Conn_02x40_Odd_Even_Shielded, SW1 SW_DIP_x08

Commit message: talkey
Changed lines of the file:
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@@
     (effects (font (size 1.27 1.27)) (justify left bottom))
   )
-  (label "{u4_10 u12_5 u4_11 u7_10 u28_4 u11_8 u10_9 u4_3 u3_8 u6-10 u12_2 u2_13 u7-13 u7_6 u34_13 P15_79 u44_14 u7_1 u7_5 u3_9 u3_10 u4_4 u3_12 P15_30 u8_11 u9_1 u10_4 u15_12 u2_10 u1_3 u29_5 u29_4 P15_32 u35_3 u11_5 P15_13 u6_13 u20_3 u27_14 P15_28 u6_12 u18_11 u33_12 P15_15 P15_12 P15_23} "
+  (label "{u4_10 u12_5 u4_11 u7_10 u28_4 u11_8 u10_9 u4_3 u3_8 u6-10 u12_2 u2_13 u7-13 u7_6 u34_13 P15_79 u44_14 u7_1 u7_5 u3_9 u3_10 u4_4 u3_12 P15_30 u8_11 u9_1 u10_4 u15_12 u2_10 u1_3 u29_5 u29_4 P15_32 u35_3 u11_5 P15_13 u6_13 u20_3 u27_14 P15_28 u6_12 u18_11 u33_12 P15_15 u44_13}"
     (at 422.91 219.71 0) (fields_autoplaced)
     (effects (font (size 0.125 0.125)) (justify left bottom))

Commit message: fix
Connections:
- net XX(UA7P3) is gone; now on net u7-13: UA7.3
- no-connect marks 89 -> 88
Changed lines of the file:
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@@
   (junction (at 781.05 475.615) (diameter 0) (color 0 0 0 0)
   )
+  (junction (at 230.505 461.645) (diameter 0) (color 0 0 0 0)
+  )
   (junction (at 317.5 400.685) (diameter 0) (color 0 0 0 0)
   )
@@
   (no_connect (at 742.315 264.795))
   (no_connect (at 616.585 686.435))
-  (no_connect (at 339.725 488.315))
   (no_connect (at 217.17 334.645))
   (no_connect (at 224.79 324.485))
@@
     (stroke (width 0) (type default))
   )
+  (wire (pts (xy 230.505 461.645) (xy 230.505 485.775))
+    (stroke (width 0) (type default))
+  )
   (bus (pts (xy 802.005 485.775) (xy 802.005 565.15))
     (stroke (width 1) (type default))
@@
     (stroke (width 0) (type default))
   )
+  (wire (pts (xy 339.725 488.315) (xy 339.725 485.775))
+    (stroke (width 0) (type default))
+  )
   (wire (pts (xy 188.595 798.195) (xy 193.675 798.195))
     (stroke (width 0) (type default))
@@
     (stroke (width 0) (type default))
   )
+  (wire (pts (xy 339.725 485.775) (xy 230.505 485.775))
+    (stroke (width 0) (type default))
+  )
   (bus (pts (xy 802.005 148.59) (xy 802.005 156.21))
     (stroke (width 1) (type default))
@@
     (effects (font (size 1.27 1.27) bold) (justify left bottom))
   )
-  (label "XX(UA7P3)" (at 339.725 488.315 180) (fields_autoplaced)
-    (effects (font (size 1.27 1.27)) (justify right bottom))
-  )
   (label "XX(UD3P9)" (at 523.24 291.465 180) (fields_autoplaced)
     (effects (font (size 1.27 1.27)) (justify right bottom))
@@
     )
   )
+  (global_label "u7-13" (shape input) (at 339.725 488.315 180) (fields_autoplaced)
+    (effects (font (size 0.8 0.8)) (justify right))
+    (property "Intersheetrefs" "${INTERSHEET_REFS}" (at 333.8947 488.315 0)
+      (effects (font (size 0.8 0.8)) (justify right) hide)
+    )
+  )

Commit message: cleanup
Other:
- moved on the sheet: R18
Changed lines of the file:
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@@
     (stroke (width 0) (type default))
   )
-  (wire (pts (xy 440.69 354.965) (xy 433.705 354.965))
-    (stroke (width 0) (type default))
-  )
   (wire (pts (xy 653.415 314.96) (xy 653.415 316.23))
     (stroke (width 0) (type default))
@@
     (stroke (width 0) (type default))
   )
+  (wire (pts (xy 433.705 357.505) (xy 445.77 357.505))
+    (stroke (width 0) (type default))
+  )
   (wire (pts (xy 408.94 253.365) (xy 408.94 256.54))
     (stroke (width 0) (type default))
@@
     (stroke (width 0) (type default))
   )
+  (wire (pts (xy 433.705 354.965) (xy 433.705 357.505))
+    (stroke (width 0) (type default))
+  )
   (wire (pts (xy 363.855 450.85) (xy 363.855 458.47))
     (stroke (width 0) (type default))
@@
     (effects (font (size 1.27 1.27)) (justify left bottom))
   )
-  (label "U44P5" (at 433.705 354.965 0) (fields_autoplaced)
-    (effects (font (size 1.27 1.27)) (justify left bottom))
-  )
   (label "P15_12" (at 791.21 192.405 0) (fields_autoplaced)
     (effects (font (size 1.27 1.27)) (justify left bottom))
@@
     )
   )
+  (global_label "U44P5" (shape input) (at 433.705 354.965 0) (fields_autoplaced)
+    (effects (font (size 0.8 0.8)) (justify left))
+    (property "Intersheetrefs" "${INTERSHEET_REFS}" (at 439.4591 354.965 0)
+      (effects (font (size 0.8 0.8)) (justify left) hide)
+    )
+  )
   (global_label "P15_8" (shape input) (at 217.805 620.395 180) (fields_autoplaced)
     (effects (font (size 0.8 0.8)) (justify right))
@@
     )
   )
-  (symbol (lib_id "SamacSys_Parts:YR1B24K9CC") (at 440.69 354.965 0) (unit 1)
+  (symbol (lib_id "SamacSys_Parts:YR1B24K9CC") (at 445.77 357.505 0) (unit 1)
     (in_bom yes) (on_board yes) (dnp no)
-    (property "Reference" "R18" (at 452.12 352.425 0)
+    (property "Reference" "R18" (at 457.2 354.965 0)
       (effects (font (size 1.27 1.27)) (justify right))
     )
-    (property "Value" "1k" (at 448.3101 357.505 90)
+    (property "Value" "1k" (at 453.3901 360.045 90)
       (effects (font (size 1.27 1.27)) (justify right) hide)
     )
-    (property "Footprint" "Resistor_THT:R_Axial_DIN0207_L6.3mm_D2.5mm_P10.16mm_Horizontal" (at 454.66 353.695 0)
+    (property "Footprint" "Resistor_THT:R_Axial_DIN0207_L6.3mm_D2.5mm_P10.16mm_Horizontal" (at 459.74 356.235 0)
       (effects (font (size 1.27 1.27)) (justify left) hide)
     )
-    (property "Datasheet" "https://datasheet.datasheetarchive.com/originals/distributors/DKDS-21/401731.pdf" (at 454.66 356.235 0)
+    (property "Datasheet" "https://datasheet.datasheetarchive.com/originals/distributors/DKDS-21/401731.pdf" (at 459.74 358.775 0)
       (effects (font (size 1.27 1.27)) (justify left) hide)
     )
-    (property "Description" "TE Connectivity R Series Axial Through Hole Fixed Resistor 24.9k +/-0.1% 0.25W +/-15ppm/C" (at 454.66 358.775 0)
+    (property "Description" "TE Connectivity R Series Axial Through Hole Fixed Resistor 24.9k +/-0.1% 0.25W +/-15ppm/C" (at 459.74 361.315 0)
       (effects (font (size 1.27 1.27)) (justify left) hide)
     )
-    (property "Height" "" (at 454.66 361.315 0)
+    (property "Height" "" (at 459.74 363.855 0)
       (effects (font (size 1.27 1.27)) (justify left) hide)
     )
-    (property "Manufacturer_Name" "TE Connectivity" (at 454.66 363.855 0)
+    (property "Manufacturer_Name" "TE Connectivity" (at 459.74 366.395 0)
       (effects (font (size 1.27 1.27)) (justify left) hide)
     )
-    (property "Manufacturer_Part_Number" "YR1B24K9CC" (at 454.66 366.395 0)
+    (property "Manufacturer_Part_Number" "YR1B24K9CC" (at 459.74 368.935 0)
       (effects (font (size 1.27 1.27)) (justify left) hide)
     )
-    (property "Mouser Part Number" "279-YR1B24K9CC" (at 454.66 368.935 0)
+    (property "Mouser Part Number" "279-YR1B24K9CC" (at 459.74 371.475 0)
       (effects (font (size 1.27 1.27)) (justify left) hide)
     )
-    (property "Mouser Price/Stock" "https://www.mouser.co.uk/ProductDetail/TE-Connectivity-Holsworthy/YR1B24K9CC?qs=VHcS2MTj4gYRZK1N8SqsaA%3D%3D" (at 454.66 371.475 0)
+    (property "Mouser Price/Stock" "https://www.mouser.co.uk/ProductDetail/TE-Connectivity-Holsworthy/YR1B24K9CC?qs=VHcS2MTj4gYRZK1N8SqsaA%3D%3D" (at 459.74 374.015 0)
       (effects (font (size 1.27 1.27)) (justify left) hide)
     )
-    (property "Arrow Part Number" "" (at 454.66 374.015 0)
+    (property "Arrow Part Number" "" (at 459.74 376.555 0)
       (effects (font (size 1.27 1.27)) (justify left) hide)
     )
-    (property "Arrow Price/Stock" "" (at 454.66 376.555 0)
+    (property "Arrow Price/Stock" "" (at 459.74 379.095 0)
       (effects (font (size 1.27 1.27)) (justify left) hide)
     )
-    (property "Mouser Testing Part Number" "" (at 454.66 379.095 0)
+    (property "Mouser Testing Part Number" "" (at 459.74 381.635 0)
       (effects (font (size 1.27 1.27)) (justify left) hide)
     )
-    (property "Mouser Testing Price/Stock" "" (at 454.66 381.635 0)
+    (property "Mouser Testing Price/Stock" "" (at 459.74 384.175 0)
       (effects (font (size 1.27 1.27)) (justify left) hide)
     )
@@
     )
   )
-  (symbol (lib_id "power:VCC") (at 458.47 354.965 270) (unit 1)
+  (symbol (lib_id "power:VCC") (at 463.55 357.505 270) (unit 1)
     (in_bom yes) (on_board yes) (dnp no)
-    (property "Reference" "#PWR028" (at 454.66 354.965 0)
+    (property "Reference" "#PWR028" (at 459.74 357.505 0)
       (effects (font (size 1.27 1.27)) hide)
     )
-    (property "Value" "VCC" (at 462.1932 355.1588 0)
+    (property "Value" "VCC" (at 467.2732 357.6988 0)
       (effects (font (size 1.27 1.27)))
     )
-    (property "Footprint" "" (at 458.47 354.965 0)
+    (property "Footprint" "" (at 463.55 357.505 0)
       (effects (font (size 1.27 1.27)) hide)
     )
-    (property "Datasheet" "" (at 458.47 354.965 0)
+    (property "Datasheet" "" (at 463.55 357.505 0)
       (effects (font (size 1.27 1.27)) hide)
     )

Commit message: UB8P12
Connections:
- net XX(UB8P12) is gone; now on net u2_10: UB8.12
- no-connect marks 88 -> 87
Changed lines of the file:
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@@
   (junction (at 294.64 165.1) (diameter 0) (color 0 0 0 0)
   )
+  (junction (at 371.475 204.47) (diameter 0) (color 0 0 0 0)
+  )
   (junction (at 802.005 617.855) (diameter 0) (color 0 0 0 0)
   )
@@
   (no_connect (at 683.895 335.28))
   (no_connect (at 528.32 531.495))
-  (no_connect (at 407.67 204.47))
   (no_connect (at 261.62 462.28))
   (no_connect (at 354.33 463.55))
@@
     (stroke (width 0) (type default))
   )
-  (wire (pts (xy 371.475 155.575) (xy 371.475 347.345))
+  (wire (pts (xy 371.475 155.575) (xy 371.475 204.47))
     (stroke (width 0) (type default))
   )
@@
     (stroke (width 0) (type default))
   )
+  (wire (pts (xy 371.475 204.47) (xy 371.475 347.345))
+    (stroke (width 0) (type default))
+  )
   (wire (pts (xy 872.49 426.72) (xy 872.49 424.815))
     (stroke (width 0) (type default))
@@
     (stroke (width 0) (type default))
   )
+  (wire (pts (xy 371.475 204.47) (xy 407.67 204.47))
+    (stroke (width 0) (type default))
+  )
   (wire (pts (xy 346.075 669.29) (xy 346.075 664.845))
     (stroke (width 0) (type default))
@@
     (effects (font (size 1.27 1.27)) (justify left bottom))
   )
-  (label "XX(UB8P12)" (at 407.67 204.47 180) (fields_autoplaced)
+  (label "u2_10" (at 407.67 204.47 180) (fields_autoplaced)
     (effects (font (size 1.27 1.27)) (justify right bottom))
   )

Commit message: u36_13
Connections:
- net u36_13 is gone; now on net VCC: UA1.13 (DS2), UA2.13 (DS2)
Changed lines of the file:
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@@
     (stroke (width 0) (type default))
   )
-  (wire (pts (xy 824.865 452.12) (xy 872.49 452.12))
-    (stroke (width 0) (type default))
-  )
   (polyline (pts (xy 217.932 806.45) (xy 246.38 806.45))
     (stroke (width 0) (type default))
@@
     (stroke (width 0) (type default))
   )
-  (wire (pts (xy 824.865 386.08) (xy 872.49 386.08))
-    (stroke (width 0) (type default))
-  )
   (wire (pts (xy 709.93 175.26) (xy 698.5 175.26))
     (stroke (width 0) (type default))
@@
     (stroke (width 0) (type default))
   )
-  (wire (pts (xy 824.865 386.08) (xy 824.865 452.12))
-    (stroke (width 0) (type default))
-  )
   (wire (pts (xy 602.615 633.095) (xy 616.585 633.095))
     (stroke (width 0) (type default))
@@
     (effects (font (size 1.27 1.27)) (justify left bottom))
   )
-  (label "u36_13" (at 864.87 452.12 0) (fields_autoplaced)
-    (effects (font (size 1.27 1.27)) (justify left bottom))
-  )
   (label "P15_23" (at 793.115 162.56 0) (fields_autoplaced)
     (effects (font (size 1.27 1.27)) (justify left bottom))
@@
     (effects (font (size 1.27 1.27)) (justify left bottom))
   )
-  (label "u36_13" (at 864.87 386.08 0) (fields_autoplaced)
-    (effects (font (size 1.27 1.27)) (justify left bottom))
-  )
   (label "{P15_14 P15_16 P15_18 P15_20 P15_22 P15_24 P15_26 P15_59 P15_60 P15_61 P15_62 P15_63 P15_64 P15_65 P15_66 P15_67 P15_68 P15_69 P15_70 P15_71 P15_72 P15_73 P15_74 P15_75 P15_76 P15_77 P15_78}"
     (at 139.7 848.36 0) (fields_autoplaced)
@@
     )
   )
-  (global_label "u36_13" (shape input) (at 824.865 386.08 180) (fields_autoplaced)
-    (effects (font (size 0.8 0.8)) (justify right))
-    (property "Intersheetrefs" "${INTERSHEET_REFS}" (at 818.6538 386.08 0)
-      (effects (font (size 0.8 0.8)) (justify right) hide)
-    )
-  )
   (global_label "P15_13" (shape input) (at 188.595 777.875 180) (fields_autoplaced)
     (effects (font (size 0.8 0.8)) (justify right))
@@
     )
   )
-  (symbol (lib_id "power:VCC") (at 872.49 389.89 90) (unit 1)
+  (symbol (lib_id "power:VCC") (at 872.49 386.08 90) (unit 1)
     (in_bom yes) (on_board yes) (dnp no) (fields_autoplaced)
-    (property "Reference" "#PWR024" (at 876.3 389.89 0)
+    (property "Reference" "#PWR024" (at 876.3 386.08 0)
       (effects (font (size 1.27 1.27)) hide)
     )
-    (property "Value" "VCC" (at 867.41 389.89 0)
-      (effects (font (size 1.27 1.27)))
+    (property "Value" "VCC" (at 869.95 386.715 90)
+      (effects (font (size 1.27 1.27)) (justify left))
     )
-    (property "Footprint" "" (at 872.49 389.89 0)
+    (property "Footprint" "" (at 872.49 386.08 0)
       (effects (font (size 1.27 1.27)) hide)
     )
-    (property "Datasheet" "" (at 872.49 389.89 0)
+    (property "Datasheet" "" (at 872.49 386.08 0)
       (effects (font (size 1.27 1.27)) hide)
     )
@@
     )
   )
+  (symbol (lib_id "power:VCC") (at 872.49 389.89 90) (unit 1)
+    (in_bom yes) (on_board yes) (dnp no) (fields_autoplaced)
+    (property "Reference" "#PWR0121" (at 876.3 389.89 0)
+      (effects (font (size 1.27 1.27)) hide)
+    )
+    (property "Value" "VCC" (at 869.95 390.525 90)
+      (effects (font (size 1.27 1.27)) (justify left))
+    )
+    (property "Footprint" "" (at 872.49 389.89 0)
+      (effects (font (size 1.27 1.27)) hide)
+    )
+    (property "Datasheet" "" (at 872.49 389.89 0)
+      (effects (font (size 1.27 1.27)) hide)
+    )
+    (pin "1")
+    (instances
+      (project "Entrex Trapezoid Interface Board v23"
+        (path "/2743c6c7-b9b4-4894-8f09-402edf838239"
+          (reference "#PWR0121") (unit 1)
+        )
+      )
+    )
+  )
   (symbol (lib_id "power:GND") (at 1232.535 489.585 0) (unit 1)
     (in_bom yes) (on_board yes) (dnp no)
@@
         )
       )
+    )
+  )
+  (symbol (lib_id "power:VCC") (at 872.49 452.12 90) (unit 1)
+    (in_bom yes) (on_board yes) (dnp no) (fields_autoplaced)
+    (property "Reference" "#PWR0122" (at 876.3 452.12 0)
+      (effects (font (size 1.27 1.27)) hide)
+    )
+    (property "Value" "VCC" (at 869.95 452.755 90)
+      (effects (font (size 1.27 1.27)) (justify left))
+    )
+    (property "Footprint" "" (at 872.49 452.12 0)
+      (effects (font (size 1.27 1.27)) hide)
+    )
+    (property "Datasheet" "" (at 872.49 452.12 0)
+      (effects (font (size 1.27 1.27)) hide)
+    )
+    (pin "1")
+    (instances
+      (project "Entrex Trapezoid Interface Board v23"
+        (path "/2743c6c7-b9b4-4894-8f09-402edf838239"
+          (reference "#PWR0122") (unit 1)
+        )
+      )

Commit message: UB5B Pin 11
Connections:
- net XX(UB5P11) is gone; now on net u20_3: UB5.11 (C)
- no-connect marks 87 -> 86
Changed lines of the file:
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@@
   (junction (at 170.815 248.285) (diameter 0) (color 0 0 0 0)
   )
+  (junction (at 556.26 585.47) (diameter 0) (color 0 0 0 0)
+  )
   (junction (at 726.44 205.74) (diameter 0) (color 0 0 0 0)
   )
@@
   (no_connect (at 338.455 554.355))
   (no_connect (at 590.55 595.63))
-  (no_connect (at 335.915 539.115))
   (no_connect (at 582.93 590.55))
   (no_connect (at 711.2 173.99))
@@
     (stroke (width 0) (type default))
   )
+  (wire (pts (xy 509.905 552.45) (xy 509.905 585.47))
+    (stroke (width 0) (type default))
+  )
   (wire (pts (xy 400.05 567.055) (xy 530.86 567.055))
     (stroke (width 0) (type default))
@@
     (stroke (width 0) (type default))
   )
+  (wire (pts (xy 497.205 525.145) (xy 497.205 552.45))
+    (stroke (width 0) (type default))
+  )
   (wire (pts (xy 134.62 234.315) (xy 143.51 234.315))
     (stroke (width 0) (type default))
@@
     (stroke (width 0) (type default))
   )
+  (wire (pts (xy 334.01 539.115) (xy 334.01 532.13))
+    (stroke (width 0) (type default))
+  )
   (wire (pts (xy 561.975 615.95) (xy 615.315 615.95))
     (stroke (width 0) (type default))
@@
     (stroke (width 0) (type default))
   )
+  (wire (pts (xy 497.205 552.45) (xy 509.905 552.45))
+    (stroke (width 0) (type default))
+  )
   (wire (pts (xy 217.805 489.585) (xy 217.805 391.16))
     (stroke (width 0) (type default))
@@
     (stroke (width 0) (type default))
   )
+  (wire (pts (xy 334.01 532.13) (xy 366.395 532.13))
+    (stroke (width 0) (type default))
+  )
   (wire (pts (xy 1114.425 674.37) (xy 1110.615 674.37))
     (stroke (width 0) (type default))
@@
     (stroke (width 0) (type default))
   )
+  (wire (pts (xy 366.395 532.13) (xy 366.395 525.145))
+    (stroke (width 0) (type default))
+  )
   (wire (pts (xy 855.345 483.235) (xy 855.345 432.435))
     (stroke (width 0) (type default))
@@
     (stroke (width 0) (type default))
   )
+  (wire (pts (xy 509.905 585.47) (xy 556.26 585.47))
+    (stroke (width 0) (type default))
+  )
   (wire (pts (xy 317.5 160.02) (xy 363.22 160.02))
     (stroke (width 0) (type default))
@@
     (stroke (width 0) (type default))
   )
-  (wire (pts (xy 556.26 600.075) (xy 556.26 565.785))
+  (wire (pts (xy 556.26 600.075) (xy 556.26 585.47))
     (stroke (width 0) (type default))
   )
@@
     (stroke (width 0) (type default))
   )
+  (wire (pts (xy 366.395 525.145) (xy 497.205 525.145))
+    (stroke (width 0) (type default))
+  )
   (wire (pts (xy 387.985 450.85) (xy 363.855 450.85))
     (stroke (width 0) (type default))
@@
     (stroke (width 0) (type default))
   )
+  (wire (pts (xy 556.26 585.47) (xy 556.26 565.785))
+    (stroke (width 0) (type default))
+  )
   (wire (pts (xy 158.75 231.14) (xy 166.37 231.14))
     (stroke (width 0) (type default))
@@
     (stroke (width 0) (type default))
   )
+  (wire (pts (xy 335.915 539.115) (xy 334.01 539.115))
+    (stroke (width 0) (type default))
+  )
   (wire (pts (xy 407.67 222.25) (xy 407.67 220.345))
     (stroke (width 0) (type default))
@@
     (effects (font (size 1.27 1.27)) (justify left bottom))
   )
-  (label "XX(UB5P11)" (at 335.915 539.115 90) (fields_autoplaced)
-    (effects (font (size 1.27 1.27)) (justify left bottom))
-  )
   (label "XX(UC7P12)" (at 579.12 488.95 270) (fields_autoplaced)
     (effects (font (size 1.27 1.27)) (justify right bottom))
@@
     )
   )
+  (global_label "u20_3" (shape input) (at 335.915 539.115 90) (fields_autoplaced)
+    (effects (font (size 0.8 0.8)) (justify left))
+    (property "Intersheetrefs" "${INTERSHEET_REFS}" (at 335.915 533.6657 90)
+      (effects (font (size 1.27 1.27)) (justify left) hide)
+    )
+  )

Commit message: Corrections & Testing
Connections:
- net XX(UD7P2) is gone; now on net u10_8: UD7.2
- no-connect marks 86 -> 85
Changed lines of the file:
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@@
   (junction (at 423.545 392.43) (diameter 0) (color 0 0 0 0)
   )
+  (junction (at 174.625 333.375) (diameter 0) (color 0 0 0 0)
+  )
   (junction (at 201.93 60.96) (diameter 0) (color 0 0 0 0)
   )
@@
   (no_connect (at 584.2 473.71))
   (no_connect (at 424.18 250.825))
-  (no_connect (at 408.305 178.435))
   (no_connect (at 739.775 264.795))
   (bus_entry (at 467.36 494.665) (size 2.54 2.54)
@@
     (stroke (width 0) (type default))
   )
+  (wire (pts (xy 361.95 180.975) (xy 408.305 180.975))
+    (stroke (width 0) (type default))
+  )
   (wire (pts (xy 169.545 657.86) (xy 169.545 659.13))
     (stroke (width 0) (type default))
@@
     (stroke (width 1) (type default))
   )
+  (wire (pts (xy 408.305 178.435) (xy 408.305 180.975))
+    (stroke (width 0) (type default))
+  )
   (wire (pts (xy 123.825 217.805) (xy 123.825 220.98))
     (stroke (width 0) (type default))
@@
     (stroke (width 0) (type default))
   )
+  (wire (pts (xy 174.625 317.5) (xy 216.535 317.5))
+    (stroke (width 0) (type default))
+  )
   (wire (pts (xy 748.665 463.55) (xy 788.035 463.55))
     (stroke (width 0) (type default))
@@
     (stroke (width 0) (type default))
   )
+  (wire (pts (xy 174.625 333.375) (xy 180.34 333.375))
+    (stroke (width 0) (type default))
+  )
   (wire (pts (xy 313.055 424.18) (xy 313.055 427.355))
     (stroke (width 0) (type default))
@@
     (stroke (width 0) (type default))
   )
+  (wire (pts (xy 216.535 317.5) (xy 216.535 311.785))
+    (stroke (width 0) (type default))
+  )
   (wire (pts (xy 225.425 135.255) (xy 225.425 184.15))
     (stroke (width 0) (type default))
@@
     (stroke (width 0) (type default))
   )
-  (wire (pts (xy 168.275 333.375) (xy 180.34 333.375))
+  (wire (pts (xy 168.275 333.375) (xy 174.625 333.375))
     (stroke (width 0) (type default))
   )
@@
     (stroke (width 1) (type default))
   )
+  (wire (pts (xy 174.625 333.375) (xy 174.625 317.5))
+    (stroke (width 0) (type default))
+  )
   (wire (pts (xy 156.845 66.04) (xy 156.845 67.31))
     (stroke (width 0) (type default))
@@
     (stroke (width 0) (type default))
   )
+  (wire (pts (xy 361.95 311.785) (xy 361.95 180.975))
+    (stroke (width 0) (type default))
+  )
   (wire (pts (xy 201.93 184.15) (xy 225.425 184.15))
     (stroke (width 0) (type default))
@@
     (stroke (width 1) (type default))
   )
+  (wire (pts (xy 216.535 311.785) (xy 361.95 311.785))
+    (stroke (width 0) (type default))
+  )
   (polyline (pts (xy 182.245 835.66) (xy 160.655 835.66))
     (stroke (width 0) (type default))
@@
     (effects (font (size 1.27 1.27)) (justify right bottom))
   )
-  (label "XX(UD7P2)" (at 408.305 178.435 180) (fields_autoplaced)
-    (effects (font (size 1.27 1.27)) (justify right bottom))
-  )
   (label "P15_40" (at 163.83 198.12 0) (fields_autoplaced)
     (effects (font (size 1.27 1.27)) (justify left bottom))
@@
     )
   )
+  (global_label "u10_8" (shape input) (at 408.305 178.435 180) (fields_autoplaced)
+    (effects (font (size 0.8 0.8)) (justify right))
+    (property "Intersheetrefs" "${INTERSHEET_REFS}" (at 402.8557 178.435 0)
+      (effects (font (size 1.27 1.27)) (justify right) hide)
+    )
+  )

Commit message: fixes
Connections:
- net XX(UC7P11) is gone; now on net GND: UC7.11 (C)
- no-connect marks 85 -> 84
Changed lines of the file:
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@@
   (no_connect (at 405.765 333.375))
   (no_connect (at 416.56 245.745))
-  (no_connect (at 581.66 488.95))
   (no_connect (at 579.12 488.95))
   (no_connect (at 584.2 473.71))
@@
     (effects (font (size 1.27 1.27)) (justify right bottom))
   )
-  (label "XX(UC7P11)" (at 581.66 488.95 270) (fields_autoplaced)
-    (effects (font (size 1.27 1.27)) (justify right bottom))
-  )
   (label "u14_3" (at 693.42 34.925 0) (fields_autoplaced)
     (effects (font (size 1.27 1.27)) (justify left bottom))
@@
         )
       )
+    )
+  )
+  (symbol (lib_id "power:GND") (at 581.66 488.95 0) (unit 1)
+    (in_bom yes) (on_board yes) (dnp no) (fields_autoplaced)
+    (property "Reference" "#PWR0124" (at 581.66 495.3 0)
+      (effects (font (size 1.27 1.27)) hide)
+    )
+    (property "Value" "GND" (at 581.66 494.03 0)
+      (effects (font (size 1.27 1.27)))
+    )
+    (property "Footprint" "" (at 581.66 488.95 0)
+      (effects (font (size 1.27 1.27)) hide)
+    )
+    (property "Datasheet" "" (at 581.66 488.95 0)
+      (effects (font (size 1.27 1.27)) hide)
+    )
+    (pin "1")
+    (instances
+      (project "Entrex Trapezoid Interface Board v23"
+        (path "/2743c6c7-b9b4-4894-8f09-402edf838239"
+          (reference "#PWR0124") (unit 1)
+        )
+      )
