File: Trapezoid_Terminal/Interface Board/Entrex Trapezoid Interface Board v23.kicad_sch (KiCad schematic)
At the start: 103 parts, among them P15 Conn_02x40_Odd_Even_Shielded, SW1 SW_DIP_x08

Commit message: fixes
Connections:
- net XX(UB5P4) is gone; now on net VCC: UB5.4 (~{S})
- net XX(UB5P9) is gone; now on net u20_10: UB5.9 (Q)
- net VCC: now also UB5.10 (~{S})
- net u20_10: no longer UB5.10 (~{S})
- no-connect marks 84 -> 82
Changed lines of the file:
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@@
   (no_connect (at 1069.34 784.225))
   (no_connect (at 1094.74 784.225))
-  (no_connect (at 338.455 554.355))
   (no_connect (at 590.55 595.63))
-  (no_connect (at 582.93 590.55))
   (no_connect (at 711.2 173.99))
   (no_connect (at 208.915 270.51))
@@
     (stroke (width 0) (type default))
   )
-  (wire (pts (xy 343.535 544.83) (xy 400.05 544.83))
-    (stroke (width 0) (type default))
-  )
   (wire (pts (xy 598.805 563.88) (xy 657.225 563.88))
     (stroke (width 0) (type default))
@@
     (stroke (width 1) (type default))
   )
-  (wire (pts (xy 400.05 544.83) (xy 400.05 547.37))
-    (stroke (width 0) (type default))
-  )
   (wire (pts (xy 448.945 403.86) (xy 448.945 401.955))
     (stroke (width 0) (type default))
@@
     (stroke (width 0) (type default))
   )
+  (wire (pts (xy 338.455 554.355) (xy 400.05 554.355))
+    (stroke (width 0) (type default))
+  )
   (wire (pts (xy 302.26 165.1) (xy 302.26 167.005))
     (stroke (width 0) (type default))
@@
     (stroke (width 0) (type default))
   )
+  (wire (pts (xy 400.05 554.355) (xy 400.05 547.37))
+    (stroke (width 0) (type default))
+  )
   (wire (pts (xy 348.615 212.09) (xy 348.615 232.41))
     (stroke (width 0) (type default))
@@
     (stroke (width 0) (type default))
   )
-  (wire (pts (xy 343.535 544.83) (xy 343.535 546.735))
-    (stroke (width 0) (type default))
-  )
   (wire (pts (xy 256.54 588.01) (xy 262.89 588.01))
     (stroke (width 0) (type default))
@@
     (effects (font (size 1.27 1.27)) (justify right bottom))
   )
-  (label "XX(UB5P9)" (at 338.455 554.355 270) (fields_autoplaced)
-    (effects (font (size 1.27 1.27)) (justify right bottom))
-  )
   (label "XX(UE4P10)" (at 217.805 602.615 180) (fields_autoplaced)
     (effects (font (size 1.27 1.27)) (justify right bottom))
@@
     (effects (font (size 1.27 1.27)) (justify right bottom))
   )
+  (label "u20_10" (at 339.09 554.355 0) (fields_autoplaced)
+    (effects (font (size 1.27 1.27)) (justify left bottom))
+  )
   (label "u18_8" (at 330.835 666.75 180) (fields_autoplaced)
     (effects (font (size 1.27 1.27)) (justify right bottom))
@@
     (effects (font (size 1.27 1.27)) (justify left bottom))
   )
-  (label "XX(UB5P4)" (at 582.93 590.55 90) (fields_autoplaced)
+  (label "VCC" (at 582.93 590.55 90) (fields_autoplaced)
     (effects (font (size 1.27 1.27)) (justify left bottom))
   )
@@
     )
   )
-  (global_label "u20_10" (shape input) (at 343.535 546.735 0) (fields_autoplaced)
+  (global_label "VCC" (shape input) (at 343.535 546.735 0) (fields_autoplaced)
     (effects (font (size 0.8 0.8)) (justify left))
     (property "Intersheetrefs" "${INTERSHEET_REFS}" (at 349.7462 546.735 0)

Commit message: fixes
Connections:
- net XX(UC7P4) is gone; now on net u8_11: UC7.4 (~{S})
- net XX(UE3P10) is gone; now on net VCC: UE3.10 (~{S})
- net XX(UE3P4) is gone; now on net VCC: UE3.4 (~{S})
- no-connect marks 82 -> 79
Changed lines of the file:
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@@
   (junction (at 169.545 657.86) (diameter 0) (color 0 0 0 0)
   )
+  (junction (at 499.11 427.355) (diameter 0) (color 0 0 0 0)
+  )
   (junction (at 556.26 600.075) (diameter 0) (color 0 0 0 0)
   )
@@
   (no_connect (at 333.375 596.265))
   (no_connect (at 333.375 638.175))
-  (no_connect (at 343.535 630.555))
   (no_connect (at 544.83 314.325))
   (no_connect (at 544.83 310.515))
-  (no_connect (at 343.535 588.645))
   (no_connect (at 178.435 270.51))
   (no_connect (at 178.435 298.45))
@@
   (no_connect (at 405.765 335.915))
   (no_connect (at 405.765 333.375))
-  (no_connect (at 416.56 245.745))
   (no_connect (at 579.12 488.95))
   (no_connect (at 584.2 473.71))
@@
     (stroke (width 0) (type default))
   )
-  (wire (pts (xy 411.48 427.355) (xy 699.77 427.355))
+  (wire (pts (xy 411.48 427.355) (xy 499.11 427.355))
     (stroke (width 0) (type default))
   )
@@
     (stroke (width 0) (type default))
   )
+  (wire (pts (xy 499.11 245.745) (xy 499.11 427.355))
+    (stroke (width 0) (type default))
+  )
   (wire (pts (xy 174.625 317.5) (xy 216.535 317.5))
     (stroke (width 0) (type default))
@@
     (stroke (width 0) (type default))
   )
+  (wire (pts (xy 499.11 427.355) (xy 699.77 427.355))
+    (stroke (width 0) (type default))
+  )
   (wire (pts (xy 630.555 205.105) (xy 422.91 205.105))
     (stroke (width 0) (type default))
@@
     (stroke (width 0) (type default))
   )
+  (wire (pts (xy 499.11 245.745) (xy 416.56 245.745))
+    (stroke (width 0) (type default))
+  )
   (wire (pts (xy 149.86 240.03) (xy 163.83 240.03))
     (stroke (width 0) (type default))
@@
     (effects (font (size 3 3) (thickness 1) bold (color 255 38 190 1)) (justify right bottom))
   )
-  (label "XX(UC7P4)" (at 416.56 245.745 90) (fields_autoplaced)
-    (effects (font (size 1.27 1.27)) (justify left bottom))
-  )
   (label "XX(UC3P10)" (at 683.895 325.12 0) (fields_autoplaced)
     (effects (font (size 1.27 1.27)) (justify left bottom))
@@
     (effects (font (size 1.27 1.27)) (justify left bottom))
   )
-  (label "XX(UE3P4)" (at 343.535 630.555 0) (fields_autoplaced)
-    (effects (font (size 1.27 1.27)) (justify left bottom))
-  )
   (label "P15_5" (at 469.9 497.205 0) (fields_autoplaced)
     (effects (font (size 1.27 1.27)) (justify left bottom))
@@
     (effects (font (size 1.27 1.27)) (justify right bottom))
   )
-  (label "XX(UE3P10)" (at 343.535 588.645 0) (fields_autoplaced)
-    (effects (font (size 1.27 1.27)) (justify left bottom))
-  )
   (label "P15_38" (at 161.925 191.77 0) (fields_autoplaced)
     (effects (font (size 1.27 1.27)) (justify left bottom))
@@
     (effects (font (size 1.27 1.27)) (justify left bottom))
   )
+  (label "u8_11" (at 417.195 245.745 0) (fields_autoplaced)
+    (effects (font (size 1.27 1.27)) (justify left bottom))
+  )
   (label "XX(UF3P10)" (at 1123.315 786.765 180) (fields_autoplaced)
     (effects (font (size 1.27 1.27)) (justify right bottom))
@@
     )
   )
+  (symbol (lib_id "power:VCC") (at 343.535 630.555 270) (unit 1)
+    (in_bom yes) (on_board yes) (dnp no) (fields_autoplaced)
+    (property "Reference" "#PWR0156" (at 339.725 630.555 0)
+      (effects (font (size 1.27 1.27)) hide)
+    )
+    (property "Value" "VCC" (at 346.71 631.19 90)
+      (effects (font (size 1.27 1.27)) (justify left))
+    )
+    (property "Footprint" "" (at 343.535 630.555 0)
+      (effects (font (size 1.27 1.27)) hide)
+    )
+    (property "Datasheet" "" (at 343.535 630.555 0)
+      (effects (font (size 1.27 1.27)) hide)
+    )
+    (pin "1")
+    (instances
+      (project "Entrex Trapezoid Interface Board v23"
+        (path "/2743c6c7-b9b4-4894-8f09-402edf838239"
+          (reference "#PWR0156") (unit 1)
+        )
+      )
+    )
+  )
   (symbol (lib_id "74xx:74LS00") (at 254.635 436.88 0) (unit 4)
     (in_bom yes) (on_board yes) (dnp no)
@@
         )
       )
+    )
+  )
+  (symbol (lib_id "power:VCC") (at 343.535 588.645 270) (unit 1)
+    (in_bom yes) (on_board yes) (dnp no) (fields_autoplaced)
+    (property "Reference" "#PWR0139" (at 339.725 588.645 0)
+      (effects (font (size 1.27 1.27)) hide)
+    )
+    (property "Value" "VCC" (at 346.71 589.28 90)
+      (effects (font (size 1.27 1.27)) (justify left))
+    )
+    (property "Footprint" "" (at 343.535 588.645 0)
+      (effects (font (size 1.27 1.27)) hide)
+    )
+    (property "Datasheet" "" (at 343.535 588.645 0)
+      (effects (font (size 1.27 1.27)) hide)
+    )
+    (pin "1")
+    (instances
+      (project "Entrex Trapezoid Interface Board v23"
+        (path "/2743c6c7-b9b4-4894-8f09-402edf838239"
+          (reference "#PWR0139") (unit 1)
+        )
+      )

Commit message: fixes
Connections:
- net VCC: now also UA8.1 (~{R})
- net UA8_4: now reaches UA8.9 (Q)
- net UA8_4: now also UA8.4 (~{S})
- no-connect marks 79 -> 76
Changed lines of the file:
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@@
   (no_connect (at 120.396 88.265))
   (no_connect (at 742.315 264.795))
-  (no_connect (at 616.585 686.435))
   (no_connect (at 217.17 334.645))
-  (no_connect (at 224.79 324.485))
-  (no_connect (at 224.79 339.725))
   (no_connect (at 433.705 349.885))
   (no_connect (at 433.705 347.345))
@@
     (stroke (width 0) (type default))
   )
+  (wire (pts (xy 246.38 341.63) (xy 224.79 341.63))
+    (stroke (width 0) (type default))
+  )
   (wire (pts (xy 690.88 671.83) (xy 690.88 674.37))
     (stroke (width 0) (type default))
@@
     (stroke (width 0) (type default))
   )
+  (wire (pts (xy 616.585 686.435) (xy 616.585 688.975))
+    (stroke (width 0) (type default))
+  )
   (wire (pts (xy 361.95 473.71) (xy 387.35 473.71))
     (stroke (width 0) (type default))
@@
     (stroke (width 0) (type default))
   )
+  (wire (pts (xy 599.44 686.435) (xy 283.845 686.435))
+    (stroke (width 0) (type default))
+  )
   (bus (pts (xy 802.005 462.28) (xy 802.005 466.09))
     (stroke (width 1) (type default))
@@
     (stroke (width 0) (type default))
   )
+  (wire (pts (xy 246.38 356.87) (xy 246.38 341.63))
+    (stroke (width 0) (type default))
+  )
   (wire (pts (xy 393.7 175.26) (xy 393.7 190.5))
     (stroke (width 0) (type default))
@@
     (stroke (width 0) (type default))
   )
+  (wire (pts (xy 224.79 341.63) (xy 224.79 339.725))
+    (stroke (width 0) (type default))
+  )
   (wire (pts (xy 346.075 664.845) (xy 466.09 664.845))
     (stroke (width 0) (type default))
@@
     (stroke (width 0) (type default))
   )
+  (wire (pts (xy 283.845 356.87) (xy 246.38 356.87))
+    (stroke (width 0) (type default))
+  )
   (wire (pts (xy 129.54 231.14) (xy 143.51 231.14))
     (stroke (width 0) (type default))
@@
     (stroke (width 0) (type default))
   )
+  (wire (pts (xy 599.44 688.975) (xy 599.44 686.435))
+    (stroke (width 0) (type default))
+  )
   (wire (pts (xy 392.43 422.91) (xy 455.93 422.91))
     (stroke (width 0) (type default))
@@
     (stroke (width 0) (type default))
   )
+  (wire (pts (xy 616.585 688.975) (xy 599.44 688.975))
+    (stroke (width 0) (type default))
+  )
   (wire (pts (xy 111.76 234.315) (xy 121.285 234.315))
     (stroke (width 0) (type default))
@@
     (stroke (width 0) (type default))
   )
+  (wire (pts (xy 283.845 686.435) (xy 283.845 356.87))
+    (stroke (width 0) (type default))
+  )
   (wire (pts (xy 304.165 240.03) (xy 304.165 319.405))
     (stroke (width 0) (type default))
@@
     (effects (font (size 1.27 1.27)) (justify left bottom))
   )
+  (label "UA8_4" (at 225.425 341.63 0) (fields_autoplaced)
+    (effects (font (size 1.27 1.27)) (justify left bottom))
+  )
   (label "{P15_14 P15_16 P15_18 P15_20 P15_22 P15_24 P15_26 P15_59 P15_60 P15_61 P15_62 P15_63 P15_64 P15_65 P15_66 P15_67 P15_68 P15_69 P15_70 P15_71 P15_72 P15_73 P15_74 P15_75 P15_76 P15_77 P15_78}"
     (at 139.7 848.36 0) (fields_autoplaced)
@@
     )
   )
+  (global_label "UA8_4" (shape output) (at 616.585 686.435 180) (fields_autoplaced)
+    (effects (font (size 0.8 0.8)) (justify right))
+    (property "Intersheetrefs" "${INTERSHEET_REFS}" (at 611.0976 686.435 0)
+      (effects (font (size 1.27 1.27)) (justify right) hide)
+    )
+  )
   (global_label "P15_7" (shape input) (at 748.665 406.4 0) (fields_autoplaced)
     (effects (font (size 0.8 0.8)) (justify left))
@@
         )
       )
+    )
+  )
+  (symbol (lib_id "power:VCC") (at 224.79 324.485 270) (unit 1)
+    (in_bom yes) (on_board yes) (dnp no)
+    (property "Reference" "#PWR0173" (at 220.98 324.485 0)
+      (effects (font (size 1.27 1.27)) hide)
+    )
+    (property "Value" "VCC" (at 223.52 323.215 90)
+      (effects (font (size 1.27 1.27)))
+    )
+    (property "Footprint" "" (at 224.79 324.485 0)
+      (effects (font (size 1.27 1.27)) hide)
+    )
+    (property "Datasheet" "" (at 224.79 324.485 0)
+      (effects (font (size 1.27 1.27)) hide)
+    )
+    (pin "1")
+    (instances
+      (project "Entrex Trapezoid Interface Board v23"
+        (path "/2743c6c7-b9b4-4894-8f09-402edf838239"
+          (reference "#PWR0173") (unit 1)
+        )
+      )

Commit message: Integrate Phar's Schematics
Parts:
- removed C101: 0.1UF-0603-25V-5%, Capacitor_THT:C_Disc_D4.7mm_W2.5mm_P5.00mm, symbol SparkFun-Capacitors:0.1UF-0603-25V-5%
- removed DPLX_sw_SG1, DPLX_sw_SG2: SW_SPDT, symbol Switch:SW_SPDT
- removed R0, R1000: 330R, Resistor_THT:R_Axial_DIN0207_L6.3mm_D2.5mm_P10.16mm_Horizontal, symbol SamacSys_Parts:YR1B24K9CC
- removed R101: 150R, Resistor_THT:R_Axial_DIN0207_L6.3mm_D2.5mm_P10.16mm_Horizontal, symbol SamacSys_Parts:YR1B24K9CC
- removed unit 1 of UB6
- removed unit 3 of UB6
- removed unit 4 of UB6
- removed unit 3 of UB8
- removed unit 2 of UB8
- removed unit 1 of UB8
- removed unit 2 of UD7
- removed unit 3 of UD7
- removed unit 4 of UD7
- removed unit 1 of UD7
- removed unit 1 of UD8
- removed unit 2 of UD8
- removed unit 5 of UD8
- removed unit 3 of UD8
- removed unit 6 of UD8
- added C29: 0.1UF-0603-25V-5%, Capacitor_THT:C_Disc_D4.7mm_W2.5mm_P5.00mm, symbol SparkFun-Capacitors:0.1UF-0603-25V-5%
- added R1, R24: 330R, Resistor_THT:R_Axial_DIN0207_L6.3mm_D2.5mm_P10.16mm_Horizontal, symbol SamacSys_Parts:YR1B24K9CC
- added R25: 150R, Resistor_THT:R_Axial_DIN0207_L6.3mm_D2.5mm_P10.16mm_Horizontal, symbol SamacSys_Parts:YR1B24K9CC
- added R26: 1K, Resistor_THT:R_Axial_DIN0207_L6.3mm_D2.5mm_P10.16mm_Horizontal, symbol SamacSys_Parts:YR1B24K9CC
- added UB1, UD4: SN74LS08N, Package_DIP:DIP-14_W7.62mm, symbol 74xx:74LS08
- added UB2: SN74LS00N, Package_DIP:DIP-14_W7.62mm, symbol 74xx:74LS00
- added UD2: SN74LS04N, Package_DIP:DIP-14_W7.62mm, symbol 74xx:74LS04
- R19: value 10K -> 330R
- R23: value 330R -> 10K
Connections:
- net u2_6 is gone; now on an unnamed net: UA8.13 (~{R})
- net u4_12 is gone; now on net CG1_PORT_SELECTED: UC5.9 (CC), UD5.3 (1STRB), UD6.13 (2STRB), UF1.1 (C)
- net GND: now also UE3.10 (~{S}), UE3.4 (~{S}), C29.2
- net P15_14: no longer R3.2, UC1.6 (In3)
- net P15_16: no longer R2.2, UC1.10 (In4)
- net P15_18: no longer R4.2, UC1.12 (In5)
- net P15_20: no longer R5.2, UC1.4 (In2)
- net P15_22: no longer R6.1, UC1.14 (In6)
- net P15_24: no longer R7.1, UC1.2 (In1)
- net VCC: now also R23.2, R26.2; no longer R16.2, R19.2, UB5.10 (~{S}), UB5.4 (~{S}), UE3.10 (~{S}), UE3.4 (~{S})
- net XX(UC7P8): no longer UC7.8 (~{Q})
- net u27_3: now also R12.1, UC4.7 (B4); no longer R8.1, UC4.3 (B0)
- net u27_4: now also R11.1, UC4.6 (B3); no longer R9.1, UC4.4 (B1)
- net u27_6: now also R9.1, UC4.4 (B1); no longer R11.1, UC4.6 (B3)
- net u27_7: now also R8.1, UC4.3 (B0); no longer R12.1, UC4.7 (B4)
- net u4_2: now also UD2.2, UD4.1
- net D1P1: no longer names the net of UC2.6, UC6.4
- net P15_10 renamed read_iface_prnt_status
- net P15_11 renamed D4_in
- net D4_in: no longer UA2.16 (DI5)
- net P15_12 renamed read_iface_serial_buffer
- net read_iface_serial_buffer: now also UB1.12; no longer UC3.1 (M), UC3.2 (N)
- net P15_13 renamed D3_in
- net P15_15 renamed D2_in
- net P15_17 renamed D1_in
- net P15_19 renamed D0_in
- net P15_21 renamed D0_out
- net P15_23 renamed D1_out
- net P15_25 renamed D2_out
- net P15_27 renamed D3_out
- net P15_28 renamed CPU_OUT_0x78
- net P15_29 renamed D4_out
- net P15_31 renamed D5_out
- net P15_32 renamed write_iface_serial_tx_0
- net P15_33 renamed D6_out
- net P15_35 renamed D7_out
- net P15_37 renamed CG1_PIN_C
- net CG1_PIN_C: no longer P15.37 (Pin_37)
- net P15_38 renamed CG1_PIN_B
- net P15_39 renamed CG1_PIN_A
- net P15_40 renamed CG1_PIN_F
- net P15_41 renamed CG1_PIN_J
- net P15_42 renamed CG1_PIN_P
- net P15_43 renamed CG1_PIN_R
- net P15_44 renamed CG1_PIN_H
- net P15_45 renamed CG1_PIN_N
- net CG1_PIN_N: now also P15.37 (Pin_37)
- net P15_46 renamed CG1_PIN_D
- net P15_47 renamed CG_SEL2
- net CG_SEL2: now also UD2.13
- net P15_48 renamed CG_SEL1
- net CG_SEL1: now also UD2.1
- net P15_49 renamed CG2_PIN_H
- net P15_5 renamed D7_in
- net P15_50 renamed CG2_PIN_D
- net P15_51 renamed CG2_PIN_R
- net P15_52 renamed CG2_PIN_P
- net P15_53 renamed CG2_PIN_J
- net P15_54 renamed CG2_PIN_N
- net P15_55 renamed CG2_PIN_C
- net P15_56 renamed CG2_PIN_B
- net P15_57 renamed CG2_PIN_A
- net P15_58 renamed CG2_PIN_F
- net P15_59 renamed D7_in9
- net P15_64: no longer names the net of UC2.13, UE7.12
- net P15_64: no longer P15.64 (Pin_64)
- net P15_66: no longer names the net of UC2.11, UF6.3
- net P15_66: no longer P15.66 (Pin_66)
- net P15_68 renamed term_selectd_and_S2_INT7
- net P15_7 renamed D6_in
- net P15_70 renamed D6_in0
- net P15_71 renamed D6_in1
- net P15_72 renamed D6_in2
- net P15_75 renamed D6_in5
- net P15_76 renamed D6_in6
- net P15_77 renamed D6_in7
- net P15_78 renamed D6_in8
- net P15_79 renamed PERIPHERAL_RESET
- net PERIPHERAL_RESET: now also UB1.9
- net P15_8 renamed read_iface_status
- net P15_9 renamed D5_in
- net U44P12: no longer names the net of UC6.6
- net U44P12: now also UB1.1
- net UA1_17: no longer names the net of UA1.17 (DO6), UD1.11
- net UA1_8: no longer names the net of UA1.8 (DO3), UD1.1
- net UA8_4: no longer names the net of UA8.4 (~{S}), UA8.9 (Q)
- net UA8_4: now also UB2.6
- net XX(UA2P11): no longer names the net of UA2.11 (Strobe)
- net XX(UC4P1): no longer names the net of UC4.1 (~{E})
- net XX(UC7P5): no longer names the net of UC7.5 (Q)
- net XX(UD5P14): no longer names the net of UD5.14 (2YP_(Sink))
- net XX(UD5P2): no longer names the net of UD5.2 (1YP_(Sink))
- net XX(UD6P14): no longer names the net of UD6.14 (2YP_(Sink))
- net XX(UD6P2): no longer names the net of UD6.2 (1YP_(Sink))
- net XX(UF4P6): no longer names the net of UF4.6 (~{Q})
- net XXUE6P14: no longer names the net of UE6.14 (2YP_(Sink))
- net XXUE6P2: no longer names the net of UE6.2 (1YP_(Sink))
- net u10_11 renamed ENABLE_CG1_RX
- net ENABLE_CG1_RX: now also UD4.11
- net u10_3: no longer names the net of UD6.3 (1STRB)
- net u10_3: now also UD4.3
- net u10_4: no longer names the net of UC6.11
- net u10_4: now also UD4.4
- net u10_9 renamed CG1_PORT_SELECTED
- net CG1_PORT_SELECTED: now also UD2.12, UD4.12
- net u11_1: no longer names the net of UE7.1, UF8.15 (Q3)
- net u11_13: no longer names the net of UE7.13, UF5.3
- net u11_2: no longer names the net of UE7.2, UF8.11 (~{Q2})
- net u11_5 renamed /CPU_OUT_0x78
- net u11_8: no longer names the net of UD3.7 (Clock_2), UE7.8
- net u12_2: no longer names the net of UC7.6 (~{Q}), UF7.2
- net u12_5 renamed terminal_address_selected
- net terminal_address_selected: no longer UC5.7 (1C)
- net u13_1: no longer names the net of UA6.1, UB6.6
- net u13_12 renamed status_d1
- net u14_3 renamed 8_bits_from_serial_ready
- net 8_bits_from_serial_ready: now also UB1.3
- net u14_4: no longer names the net of UB5.8 (~{Q}), UB6.4
- net u14_5 renamed was_selected_and_S1
- net u15_10: no longer names the net of UA6.3, UC6.10
- net u15_12 renamed /terminal_address_selected
- net u15_8 renamed serial_handshake_cts
- net u15_9: no longer names the net of UA6.11, UC6.9
- net u16_12: no longer names the net of C25.1, UD6.12 (2RTC)
- net u16_4: no longer names the net of C22.2, UD6.4 (1RTC)
- net u17_12: no longer names the net of C24.2, UE6.12 (2RTC)
- net u17_4: no longer names the net of C23.2, UE6.4 (1RTC)
- net u18_11: no longer names the net of UF6.11, UF8.1 (~{Mr})
- net u18_8: no longer names the net of UF5.9, UF6.8
- net u1_3 renamed single_ended_rts
- net single_ended_rts: now also R15.1
- net u1_6: no longer names the net of UA8.6 (~{Q})
- net u1_6: now also UD4.10
- net u1_8: no longer names the net of UA8.8 (~{Q}), UC6.5
- net u20_10: no longer names the net of UA6.13
- net u20_10: now also UB5.10 (~{S}); no longer UB5.9 (Q)
- net u20_2 renamed serial_reg_Q1
- net u20_3 renamed advance_state_machine
- net advance_state_machine: now also UB2.8; no longer UB5.11 (C)
- net u22_4: no longer names the net of C26.2, UD5.4 (1RTC)
- net u24_8: no longer names the net of UF2.13 (~{R}), UF5.8
- net u25_6: no longer names the net of UA4.6 (Serial_Out), UB4.5
- net u25_9: no longer names the net of UA4.9 (Clock)
- net u25_9: no longer UA6.6
- net u27_10 renamed serial_reg_Q7
- net u27_11 renamed serial_reg_Q6
- net u27_12 renamed serial_reg_Q5
- net u27_13 renamed serial_reg_Q4
- net u27_14: no longer names the net of UC4.14 (A=B), UF5.4, UF5.5
- net u27_9 renamed serial_reg_Q8
- net u28_14 renamed status_d0
- net u28_2 renamed 8_bits_ready_on_latch
- net u28_4 renamed terminal_has_output_data_waiting
- net u29_4: no longer names the net of UF4.4 (~{S})
- net u29_4: now also C29.1, R25.2
- net u29_5 renamed terminal_has_data_waiting
- net u2_1: no longer names the net of UC8.6 (~{Q})
- net u2_1: now also UB2.1
- net u2_10 renamed bit_counter_overflow
- net bit_counter_overflow: now also UB2.10
- net u2_13 renamed /single_ended_rts
- net /single_ended_rts: now also UD2.6
- net u2_2: no longer names the net of UC2.4
- net u2_2: now also UB2.2, UB2.4
- net u2_5: no longer names the net of UC8.5 (Q)
- net u2_5: now also UB2.5
- net u30_11: no longer names the net of UB7.8
- net u30_11: now also UA4.11 (D1); no longer UA3.11 (D1)
- net u30_6 renamed serial_register_out
- net u30_9: no longer names the net of UA3.9 (Clock), UA6.8
- net u31_12 renamed serial_reg_Q3
- net u33_12 renamed serial_reg_Q2
- net u34_11 renamed term_selectd_and_S0
- net u34_12: no longer names the net of UA5.15 (Q), UE3.12 (D)
- net u34_13 renamed reset_state_machine
- net reset_state_machine: now also UB1.13, UB1.8; no longer UF2.1 (~{R})
- net u34_2: no longer names the net of UA5.11 (Q), UE3.2 (D)
- net u34_3 renamed term_selectd_and_S1
- net u35_3: no longer names the net of UF3.3
- net u35_3: now also R25.1
- net u35_6: no longer names the net of UC7.10 (~{S}), UF3.6
- net u36_15: no longer names the net of UA2.15 (DO5), UE2.9
- net u36_17: no longer names the net of UA2.17 (DO6), UE2.11
- net u36_19: no longer names the net of UA2.19 (DO7), UE1.1
- net u36_8: no longer names the net of UA2.8 (DO3), UE2.1
- net u37_8: no longer names the net of UC2.8, UE7.3
- net u3_1: no longer names the net of UC8.1 (~{R})
- net u3_1: now also UB1.11
- net u3_10: no longer names the net of UC8.10 (~{S}), UD8.8
- net u3_12 renamed single_ended_data
- net single_ended_data: now also R26.1; no longer R15.1
- net u3_2: no longer names the net of UC8.2 (D), UC8.4 (~{S})
- net u3_3 renamed N_HAS_RXD_8_BITS
- net u3_8: no longer names the net of UC8.8 (~{Q}), UE7.9, UE8.9 (~{Pe})
- net u3_9: no longer names the net of UC8.13 (~{R}), UC8.9 (Q)
- net u40_10: no longer names the net of UA1.10 (DO4), UE1.5
- net u40_15: no longer names the net of UA1.15 (DO5), UD1.9
- net u40_19: no longer names the net of UA1.19 (DO7), UD1.13
- net u40_4: no longer names the net of UA1.4 (DO1), UD1.5
- net u40_6: no longer names the net of UA1.6 (DO2), UD1.3
- net u44_13: no longer names the net of UF1.13 (B)
- net u44_13: now also R1.1; no longer R23.2
- net u44_14 renamed POWER_GOOD
- net POWER_GOOD: now also R23.1, UB1.10; no longer R19.1
- net u44_2: no longer names the net of UF1.2 (B)
- net u44_2: now also R24.2
- net u44_6: no longer names the net of UF1.6 (B)
- net u44_6: now also R19.1
- net u44_8 renamed POWER_ENABLE
- net POWER_ENABLE: now also R1.2, R24.1; no longer R23.1
- net u44_9: no longer names the net of R20.1, R21.1, UF1.9 (B)
- net u4_10 renamed differntial_transmit_enable
- net differntial_transmit_enable: now also UD2.10
- net u4_11: no longer names the net of UC6.3
- net u4_11: now also UD2.11
- net u4_3 renamed single_ended_clock
- net single_ended_clock: now also UD2.3; no longer UA7.9, UE7.10
- net u4_4: no longer names the net of UC8.11 (C), UE8.2 (CK)
- net u4_4: now also UE7.10, UD2.4
- net u6-10: no longer names the net of UF7.4, UF8.10 (Q2)
- net u6-2: no longer names the net of UF6.1, UF8.2 (Q0)
- net u6_12: no longer names the net of UF7.8, UF8.12 (D2)
- net u6_13 renamed address_match_bufd
- net u6_3: no longer names the net of UF5.2, UF8.3 (~{Q0})
- net u6_6: no longer names the net of UF5.1, UF8.6 (~{Q1})
- net u6_7: no longer names the net of UF6.4, UF8.7 (Q1)
- net u7-13 renamed protocol_request_data
- net protocol_request_data: now also UD4.5; no longer UA7.13
- net u7-2: no longer names the net of UA7.2, UB7.4
- net u7_1: no longer names the net of UA7.1, UA7.4, UB4.1, UB4.3, UB7.10
- net u7_10 renamed /protocol_request_data
- net u7_12: no longer names the net of UA6.4, UA7.12
- net u7_5: no longer names the net of UA7.5, UB7.2
- net u7_6: no longer names the net of UA6.10, UA7.6, UF4.10 (~{S})
- net u7_8: no longer names the net of UA6.5, UA6.9, UA7.8
- net u8_11 renamed /term_has_data_when_requested
- net u8_5: no longer names the net of UB4.8, UB7.5
- net u8_6: no longer names the net of UB7.6
- net u8_6: now also UA3.11 (D1); no longer UA4.11 (D1)
- net u8_9: no longer names the net of UB4.6, UB7.9
- net u9_1 renamed reset_state_machine_bufd
- net u9_13: no longer names the net of UC7.13 (~{R}), UE7.6
- net u9_9 renamed serial_out_unknown_flag_2
- new net: UD4.6, UD4.9
- new net: R4.2, UC1.12 (In5)
- new net: R5.2, UC1.4 (In2)
- new net: UB2.9, UD2.5
- new net: R6.1, UC1.14 (In6)
- new net: R7.1, UC1.2 (In1)
- new net: UB1.2, UB2.3
- new net: R2.2, UC1.10 (In4)
- new net: UD4.13, UD4.8
- new net: R3.2, UC1.6 (In3)
- new net: UC3.1 (M), UC3.2 (N)
- new net .8: R19.2
- new net INT_5: P15.66 (Pin_66)
- new net INT_6: P15.64 (Pin_64)
- new net XX(UB5P4): UB5.4 (~{S})
- new net XX(UD7P2): UD4.2
- no-connect marks 76 -> 77
Other:
- note added: ""CG1""
- note added: ""CG2""
- note added: "0b0000"
- note added: "0b1000 NAND term_select"
- note added: "0bxx00"
- note added: "0bxxx1 NAND term_seler"
- note added: "0x02 0b00000010 0x04 0b00001000 0x05 0b00001001 0x06 0b00000110 0x08 0b00001000 0x61 0b01100001 0x40 0b01000000 0x64 0b01100100 0x90 0b10010000"
- note added: "3 input AND (2 inverted inputs)"
- note added: "AND"
- note added: "Clock"
- note added: "Data"
- note added: "FIXME"
- note added: "I think this is how we set terminal status of ready"
- note added: "INP Port Access"
- note added: "OUT Port Access"
- note added: "Output shift register buffer"
- note added: "Printer port acess high reg"
- note added: "Printer port acess low reg"
- note added: "Q1 is last bit in"
- note added: "Request to send"
- note added: "any command with this bit as a zero when we have data waiting during a terminal selection, this command alsoo uses the was_single_ended_rts latch"
- note added: "any command with this bit set will INT"
- note added: "bit counter"
- note added: "causes the terminal to stop blinking- makes sense this just sets a flag for the terminal to read"
- note added: "fixme"
- note added: "i believe this sets the required initial state of the CTS an enable are contingent on the state machine being in a receptive state"
- note added: "interface and printer status port access"
- note added: "is this a start bit?"
- note added: "is wire this right?"
- note added: "latch that terminal has data in the serial tx_buffer"
- note added: "ok, i understand this latch now.. it simply waits for the bit overflow then reloads from parallel after seeing the first data bit so i think this is a start bit"
- note added: "pulse generator"
- note added: "this disables CTS if there is no data waiting"
- note added: "this disables the differential RX reciever if we're sending data but only kicks in after a reset"
- note added: "this gate suggests that RTS has to be held LOW? inj order for the 8 bit register latch signal to be recognizd"
- note added: "this just sets a flag for the terminal to read, but no other bits can be set when sending this command"
- note added: "this latches some state _when_ the terminal is selected with address and S=0x4"
- note added: "this latchis stat wen the terminal is selected with address and S|=0x1"
- note added: "was_single_ended_rts"
- note added: "well shit.. didnt see this"
- note removed: "/\"
- note removed: "= Data Bus? = Keyboard = Processor Board = Floppy Disk Controller Board (FDC) = RAM Bus = I/O (Duplexer) Board = Printer"
- note removed: "All Points Start and End with Backplane Connector (P15)"
- note removed: "Backplane pins that are not connected to any other pins other than the backplane connector are not connected to the Backplane BUS. Neither are backplane pins whose multi-pin connections are otherwise represented with regular wires"
- note removed: "How to make u4_10 and u12_5 both go high?"
- note removed: "KiCad Bus Range Creator https://bit.ly/KiCadBRC"
- note removed: "Other Trans"
- note removed: "Strobe Input"
- note removed: "Terminal Back I/O Plug "CG1""
- note removed: "Terminal Back I/O Plug "CG2""
- note removed: "UC7A Pin 6 inverse-Q latch"
- note removed: "UF2A pin 5 Q latch"
- note removed: "UF4A Q latch"
- note removed: "UF7A four conditions"
- note removed: "UF8 Pin 10 Q2"
- note removed: "Unused"
- note removed: "WARNING: Until refined & corrected, Global Label tag arrows may not indicate the proper signal in/out direction. IN was used as default when KiCad Symbols (components) were not clear on In vs Out signals, so always check component datasheets when in doubt."
- note removed: "x"
- moved on the sheet: C10, C11, C12, C13, C14, C15, C16, C17, C18, C19, C2, C20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
