File: Trapezoid_Terminal/Interface Board/Entrex Trapezoid Interface Board v23.kicad_pcb (KiCad board)
At the start: 2 copper layers, 169.1 x 191 mm, 101 parts, among them P15 Conn_02x40_Odd_Even_Shielded, SW1 SW_DIP_x08

Commit message: Corrections & Testing
Connections:
- UD7 pad 2: /XX(UD7P2) -> u10_8
Routing:
- net u10_8: track 14.0 -> 21.6 mm

Commit message: fixes
Connections:
- UC7 pad 11: /XX(UC7P11) -> GND
Routing:
- net GND: track 1625.1 -> 1636.1 mm
