File: Trapezoid_Terminal/Interface Board/Entrex Trapezoid Interface Board v23.kicad_pcb (KiCad board)
At the start: 2 copper layers, 169.1 x 191 mm, 101 parts, among them P15 Conn_02x40_Odd_Even_Shielded, SW1 SW_DIP_x08

Commit message: fixes
Connections:
- UB5 pad 10: u20_10 -> VCC
- UB5 pad 4: /XX(UB5P4) -> VCC
- UB5 pad 9: /XX(UB5P9) -> u20_10
Routing:
- net VCC: track 1895.0 -> 1905.8 mm

Commit message: fixes
Connections:
- UC7 pad 4: /XX(UC7P4) -> u8_11
- UE3 pad 10: /XX(UE3P10) -> VCC
- UE3 pad 4: /XX(UE3P4) -> VCC
Routing:
- net VCC: track 1905.8 -> 1916.4 mm
- net u8_11: track 387.7 -> 389.3 mm

Commit message: fixes
Connections:
- UA8 pad 1: unconnected-(UA8A-~{R}-Pad1) -> VCC
- UA8 pad 4: unconnected-(UA8A-~{S}-Pad4) -> UA8_4
- UA8 pad 9: unconnected-(UA8B-Q-Pad9) -> UA8_4
Routing:
- net UA8_4: track 0.00 -> 9.72 mm
- net VCC: track 1916.4 -> 1924.0 mm
