File: Trapezoid_Terminal/Interface Board/_autosave-Entrex Trapezoid Interface Board v23.kicad_sch (KiCad schematic)
At the start: 106 parts, among them P15 Conn_02x40_Odd_Even_Shielded, SW1 SW_DIP_x08

Commit message: JoeZ Fixes the Trapezoid!!!!!
Connections:
- net u27_3: now also SW1.1
Changed lines of the file:
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@@
   (junction (at 178.562 123.7587) (diameter 0) (color 0 0 0 0)
   )
+  (junction (at 593.471 332.74) (diameter 0) (color 0 0 0 0)
+  )
   (junction (at 326.0965 377.5496) (diameter 0) (color 0 0 0 0)
   )
@@
     (stroke (width 0) (type default))
   )
-  (wire (pts (xy 613.41 332.74) (xy 593.471 332.74))
+  (wire (pts (xy 582.676 332.74) (xy 593.471 332.74))
     (stroke (width 0) (type default))
   )
@@
     (stroke (width 0) (type default))
   )
-  (wire (pts (xy 593.344 332.74) (xy 582.676 332.74))
-    (stroke (width 0) (type default))
-  )
   (wire (pts (xy 68.58 467.995) (xy 73.66 467.995))
     (stroke (width 0) (type default))
@@
     (stroke (width 0) (type default))
   )
+  (wire (pts (xy 593.471 332.74) (xy 613.41 332.74))
+    (stroke (width 0) (type default))
+  )
