File: Trapezoid_Terminal/Interface Board/Talk To Me/Talk To Me.kicad_sch (KiCad schematic)
At the start: 86 parts, among them P15 Conn_02x40_Odd_Even_Shielded, SW1 SW_DIP_x08

Commit message: Update Talk To Me.kicad_sch
Other:
- note added: "u28_4 & u7_10"
Changed lines of the file:
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@@
     (stroke (width 0) (type default))
   )
+  (wire (pts (xy 307.975 467.36) (xy 307.975 691.515))
+    (stroke (width 0) (type default))
+  )
   (wire (pts (xy 188.595 785.495) (xy 193.675 785.495))
     (stroke (width 0) (type default))
@@
     (stroke (width 0) (type default))
   )
-  (wire (pts (xy 314.96 250.19) (xy 384.81 250.19))
+  (wire (pts (xy 314.96 250.19) (xy 383.54 250.19))
     (stroke (width 0) (type default))
   )
@@
     (stroke (width 0) (type default))
   )
-  (wire (pts (xy 384.81 250.19) (xy 384.81 280.67))
+  (wire (pts (xy 383.54 250.19) (xy 383.54 280.67))
     (stroke (width 0) (type default))
   )
@@
     (stroke (width 0) (type default))
   )
-  (wire (pts (xy 384.81 280.67) (xy 408.94 280.67))
+  (wire (pts (xy 383.54 280.67) (xy 408.94 280.67))
     (stroke (width 0) (type default))
   )
@@
     (stroke (width 0) (type default))
   )
+  (wire (pts (xy 378.46 255.27) (xy 341.63 255.27))
+    (stroke (width 0) (type default))
+  )
   (wire (pts (xy 260.35 220.345) (xy 260.35 222.25))
     (stroke (width 0) (type default))
@@
     (stroke (width 0) (type default))
   )
+  (wire (pts (xy 307.975 691.515) (xy 581.66 691.515))
+    (stroke (width 0) (type default))
+  )
   (wire (pts (xy 188.595 808.355) (xy 193.675 808.355))
     (stroke (width 0) (type default))
@@
     (stroke (width 0) (type default))
   )
-  (wire (pts (xy 382.27 255.27) (xy 341.63 255.27))
-    (stroke (width 0) (type default))
-  )
   (wire (pts (xy 1192.53 725.805) (xy 1192.4891 730.7604))
     (stroke (width 0) (type default))
@@
     (stroke (width 0) (type default))
   )
-  (wire (pts (xy 551.815 691.515) (xy 581.66 691.515))
-    (stroke (width 0) (type default))
-  )
   (polyline (pts (xy 246.38 776.605) (xy 217.678 776.605))
     (stroke (width 0) (type default))
@@
     (stroke (width 0) (type default))
   )
-  (wire (pts (xy 530.86 567.055) (xy 530.86 612.775))
-    (stroke (width 0) (type default))
-  )
   (wire (pts (xy 598.805 561.975) (xy 598.805 563.88))
     (stroke (width 0) (type default))
@@
     (stroke (width 0) (type default))
   )
-  (wire (pts (xy 551.815 634.365) (xy 360.68 634.365))
-    (stroke (width 0) (type default))
-  )
   (wire (pts (xy 140.97 76.2) (xy 140.97 115.57))
     (stroke (width 0) (type default))
@@
     (stroke (width 0) (type default))
   )
-  (wire (pts (xy 382.27 255.27) (xy 382.27 295.275))
-    (stroke (width 0) (type default))
-  )
   (wire (pts (xy 188.595 803.275) (xy 193.675 803.275))
     (stroke (width 0) (type default))
@@
     (stroke (width 0) (type default))
   )
-  (wire (pts (xy 382.27 295.275) (xy 410.845 295.275))
-    (stroke (width 0) (type default))
-  )
   (wire (pts (xy 499.745 356.235) (xy 499.745 351.155))
     (stroke (width 0) (type default))
@@
     (stroke (width 0) (type default))
   )
+  (wire (pts (xy 378.46 255.27) (xy 378.46 295.275))
+    (stroke (width 0) (type default))
+  )
   (wire (pts (xy 598.805 545.465) (xy 608.965 545.465))
     (stroke (width 0) (type default))
@@
     (stroke (width 0) (type default))
   )
+  (bus (pts (xy 148.59 645.795) (xy 148.59 647.065))
+    (stroke (width 0) (type default))
+  )
   (wire (pts (xy 699.77 314.96) (xy 725.805 314.96))
     (stroke (width 0) (type default))
@@
     (stroke (width 0) (type default))
   )
+  (wire (pts (xy 378.46 295.275) (xy 410.845 295.275))
+    (stroke (width 0) (type default))
+  )
   (bus (pts (xy 211.455 29.845) (xy 360.68 29.845))
     (stroke (width 0.5) (type default))
@@
     (stroke (width 0) (type default))
   )
-  (wire (pts (xy 307.975 467.36) (xy 307.975 654.05))
-    (stroke (width 0) (type default))
-  )
   (wire (pts (xy 264.16 245.745) (xy 264.16 243.84))
     (stroke (width 0) (type default))
@@
     (stroke (width 0) (type default))
   )
-  (wire (pts (xy 551.815 634.365) (xy 551.815 691.515))
-    (stroke (width 0) (type default))
-  )
   (wire (pts (xy 206.375 790.575) (xy 211.455 790.575))
     (stroke (width 0) (type default))
@@
     (stroke (width 0) (type default))
   )
-  (wire (pts (xy 360.68 634.365) (xy 360.68 654.05))
-    (stroke (width 0) (type default))
-  )
   (polyline (pts (xy 217.805 794.385) (xy 246.38 794.385))
     (stroke (width 0) (type default))
@@
     (stroke (width 0) (type default))
   )
-  (wire (pts (xy 334.645 141.605) (xy 160.655 141.605))
-    (stroke (width 0) (type default))
-  )
   (wire (pts (xy 398.145 223.52) (xy 398.145 241.3))
     (stroke (width 0) (type default))
@@
     (stroke (width 0) (type default))
   )
-  (wire (pts (xy 360.68 654.05) (xy 307.975 654.05))
-    (stroke (width 0) (type default))
-  )
   (wire (pts (xy 158.75 126.365) (xy 174.625 126.365))
     (stroke (width 0) (type default))
@@
     (stroke (width 0) (type default))
   )
-  (wire (pts (xy 334.645 141.605) (xy 334.645 186.055))
-    (stroke (width 0) (type default))
-  )
   (wire (pts (xy 392.43 422.91) (xy 455.93 422.91))
     (stroke (width 0) (type default))
@@
     (effects (font (size 3 3) (thickness 1) bold (color 18 244 255 1)) (justify left bottom))
   )
+  (text "u28_4 & u7_10" (at 147.955 645.16 0)
+    (effects (font (size 1.27 1.27) (thickness 0.254) bold) (justify left bottom))
+  )
   (text "Clock Input\n" (at 107.95 82.55 0)
     (effects (font (size 1.27 1.27)) (justify left bottom))
@@
     (effects (font (size 1.27 1.27)) (justify left bottom))
   )
+  (label "{u28_4 u7_10}" (at 148.59 647.065 0) (fields_autoplaced)
+    (effects (font (size 0.5 0.5)) (justify left bottom))
+  )
   (label "{P15_14 P15_16 P15_18 P15_20 P15_22 P15_24 P15_26 P15_59 P15_60 P15_61 P15_62 P15_63 P15_64 P15_65 P15_66 P15_67 P15_68 P15_69 P15_70 P15_71 P15_72 P15_73 P15_74 P15_75 P15_76 P15_77 P15_78}"

Commit message: Update Talk To Me.kicad_sch
Other:
- note added: "{u34_13 u7_6 u7-13}"
Changed lines of the file:
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@@
     (stroke (width 0) (type default))
   )
-  (wire (pts (xy 339.09 482.6) (xy 370.205 482.6))
-    (stroke (width 0) (type default))
-  )
   (wire (pts (xy 99.06 234.315) (xy 105.41 234.315))
     (stroke (width 0) (type default))
@@
     (stroke (width 0) (type default))
   )
+  (bus (pts (xy 226.695 471.17) (xy 226.695 472.44))
+    (stroke (width 0) (type default))
+  )
   (wire (pts (xy 302.26 165.1) (xy 302.26 167.005))
     (stroke (width 0) (type default))
@@
     (effects (font (size 3 3) (thickness 1) bold (color 18 244 255 1)) (justify left bottom))
   )
+  (text "{u34_13 u7_6 u7-13}" (at 226.06 470.535 0)
+    (effects (font (size 1.27 1.27) (thickness 0.254) bold) (justify left bottom))
+  )
   (text "*" (at 220.345 811.53 0)
     (effects (font (size 3 3) (thickness 1) bold (color 18 244 255 1)) (justify right bottom))
@@
     (effects (font (size 1.27 1.27)) (justify left bottom))
   )
+  (label "{u34_13 u7_6 u7-13}" (at 226.695 472.44 0) (fields_autoplaced)
+    (effects (font (size 0.5 0.5)) (justify left bottom))
+  )
   (label "XX(UD6P10)" (at 264.16 266.065 180) (fields_autoplaced)

Commit message: talkey
Other:
- note added: "{P15_79 u44_14}"
Changed lines of the file:
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@@
     (stroke (width 0.5) (type default))
   )
-  (wire (pts (xy 344.805 432.435) (xy 355.6 432.435))
-    (stroke (width 0) (type default))
-  )
   (wire (pts (xy 156.845 73.66) (xy 144.78 73.66))
     (stroke (width 0) (type default))
@@
     (stroke (width 0) (type default))
   )
+  (bus (pts (xy 643.89 687.07) (xy 643.89 688.34))
+    (stroke (width 0) (type default))
+  )
   (wire (pts (xy 188.595 788.035) (xy 193.675 788.035))
     (stroke (width 0) (type default))
@@
     (effects (font (size 3 3) (thickness 1) bold (color 18 244 255 1)) (justify left bottom))
   )
+  (text "{P15_79 u44_14}" (at 643.255 686.435 0)
+    (effects (font (size 1.27 1.27) (thickness 0.254) bold) (justify left bottom))
+  )
   (text "Other Trans\n\n" (at 179.07 78.74 0)
     (effects (font (size 1.27 1.27)) (justify left bottom))
@@
     (effects (font (size 1.27 1.27)) (justify left bottom))
   )
+  (label "{P15_79 u44_14}" (at 643.89 688.34 0) (fields_autoplaced)
+    (effects (font (size 0.5 0.5)) (justify left bottom))
+  )
   (label "{u28_4 u7_10}" (at 148.59 647.065 0) (fields_autoplaced)
