File: Trapezoid_Terminal/Interface Board/Talk To Me/Talk To Me.kicad_sch (KiCad schematic)
At the start: 86 parts, among them P15 Conn_02x40_Odd_Even_Shielded, SW1 SW_DIP_x08

Commit message: hunt
Other:
- note added: "8.55kHz 500ns except after 2 keystrokes"
- note added: "Default High blips LOW every 2 keystrokes"
- note added: "UC7A Pin 6 inverse-Q latch - High on PowerUp"
- note added: "UF8 Pin 10 Q2 - High on PowerUp"
- note added: "u28_4 & u7_10 must go high"
- note removed: "UC7A Pin 6 inverse-Q latch"
- note removed: "UF8 Pin 10 Q2"
- note removed: "u28_4 & u7_10"
Changed lines of the file:
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@@
     (effects (font (size 3 3) (thickness 1) bold (color 0 0 132 1)) (justify right bottom))
   )
-  (text "UC7A Pin 6 inverse-Q latch" (at 375.92 225.425 0)
+  (text "UC7A Pin 6 inverse-Q latch - High on PowerUp\n" (at 356.235 225.425 0)
     (effects (font (size 1.27 1.27)) (justify left bottom))
   )
@@
     (effects (font (size 3 3) (thickness 1) bold (color 18 244 255 1)) (justify left bottom))
   )
-  (text "u28_4 & u7_10" (at 147.955 645.16 0)
+  (text "u28_4 & u7_10 must go high" (at 147.955 645.16 0)
     (effects (font (size 1.27 1.27) (thickness 0.254) bold) (justify left bottom))
   )
@@
     (effects (font (size 3 3) (thickness 1) bold (color 18 244 255 1)) (justify left bottom))
   )
+  (text "Default High\nblips LOW every \n2 keystrokes" (at 640.08 700.405 0)
+    (effects (font (size 1.27 1.27)) (justify left bottom))
+  )
   (text "*" (at 105.41 234.95 0)
     (effects (font (size 3 3) (thickness 1) bold (color 18 244 255 1)) (justify left bottom))
@@
     (effects (font (size 2 2) (thickness 0.6) bold) (justify left bottom))
   )
-  (text "UF2A pin 5 Q latch\n" (at 384.175 230.505 0)
+  (text "UF2A pin 5 Q latch\n\n" (at 384.175 232.41 0)
     (effects (font (size 1.27 1.27)) (justify left bottom))
   )
@@
     (effects (font (size 3 3) (thickness 1) bold (color 5 102 8 1)) (justify right bottom))
   )
-  (text "UF8 Pin 10 Q2" (at 387.985 227.965 0)
+  (text "UF8 Pin 10 Q2 - High on PowerUp" (at 368.3 227.965 0)
     (effects (font (size 1.27 1.27)) (justify left bottom))
   )
@@
     (effects (font (size 3 3) (thickness 1) bold (color 18 244 255 1)) (justify left bottom))
   )
+  (text "8.55kHz 500ns \nexcept after \n2 keystrokes" (at 477.52 486.41 0)
+    (effects (font (size 1.27 1.27)) (justify left bottom))
+  )
   (text "Clock Input\n" (at 100.965 95.25 0)
     (effects (font (size 1.27 1.27)) (justify left bottom))
@@
     (effects (font (size 1.27 1.27) (color 255 30 30 1)) (justify left bottom))
   )
+  (text "Default High\nblips LOW every \n2 keystrokes" (at 177.8 869.315 0)
+    (effects (font (size 1.27 1.27)) (justify left bottom))
+  )
   (text "Data Input" (at 112.395 227.965 0)

Commit message: Talk To Me
Other:
- note added: "High with Data riples"
- note added: "High with slight data riples"
- note added: "Solid Data Continuous"
Changed lines of the file:
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@@
   (no_connect (at 424.18 250.825))
   (no_connect (at 739.775 264.795))
-  (bus_entry (at 467.36 494.665) (size 2.54 2.54)
-    (stroke (width 0) (type default))
-  )
   (bus_entry (at 103.505 715.01) (size 2.54 -2.54)
     (stroke (width 0) (type default))
@@
     (stroke (width 0) (type default))
   )
-  (bus_entry (at 467.36 484.505) (size 2.54 2.54)
-    (stroke (width 0) (type default))
-  )
   (bus_entry (at 467.36 459.74) (size 2.54 2.54)
     (stroke (width 0) (type default))
@@
     (stroke (width 0) (type default))
   )
-  (bus (pts (xy 467.36 494.665) (xy 467.36 738.505))
+  (bus (pts (xy 467.36 480.695) (xy 467.36 738.505))
     (stroke (width 1) (type default))
   )
@@
     (stroke (width 0) (type default))
   )
-  (wire (pts (xy 369.57 466.09) (xy 369.57 462.915))
-    (stroke (width 0) (type default))
-  )
   (polyline (pts (xy 217.932 806.45) (xy 246.38 806.45))
     (stroke (width 0) (type default))
@@
     (stroke (width 0) (type default))
   )
-  (bus (pts (xy 467.36 484.505) (xy 467.36 494.665))
-    (stroke (width 1) (type default))
-  )
   (wire (pts (xy 433.07 304.8) (xy 433.07 306.07))
     (stroke (width 0) (type default))
@@
     (stroke (width 0) (type default))
   )
-  (bus (pts (xy 467.36 480.695) (xy 467.36 484.505))
-    (stroke (width 1) (type default))
-  )
   (wire (pts (xy 206.375 798.195) (xy 211.455 798.195))
     (stroke (width 0) (type default))
@@
     (effects (font (size 3 3) (thickness 1) bold (color 18 244 255 1)) (justify left bottom))
   )
+  (text "High with\nData riples" (at 353.695 511.81 0)
+    (effects (font (size 1.27 1.27)) (justify left bottom))
+  )
   (text "Unused" (at 144.145 234.95 0)
     (effects (font (size 1.27 1.27)) (justify left bottom))
@@
     (effects (font (size 3 3) (thickness 1) bold (color 18 244 255 1)) (justify left bottom))
   )
+  (text "High with \nslight data riples" (at 370.205 464.185 0)
+    (effects (font (size 1.27 1.27)) (justify left bottom))
+  )
   (text "*" (at 127 84.455 0)
     (effects (font (size 3 3) (thickness 1) bold (color 18 244 255 1)) (justify left bottom))
@@
     (effects (font (size 1.27 1.27)) (justify left bottom))
   )
+  (text "Solid Data \nContinuous\n" (at 502.285 464.185 0)
+    (effects (font (size 1.27 1.27)) (justify left bottom))
+  )
   (text "*" (at 121.92 43.942 0)
     (effects (font (size 3 3) (thickness 1) bold (color 18 244 255 1)) (justify left bottom))
@@
     (effects (font (size 3 3) (thickness 1) bold (color 18 244 255 1)) (justify right bottom))
   )
+  (text "Solid Data \nContinuous\n" (at 431.165 485.14 0)
+    (effects (font (size 1.27 1.27)) (justify left bottom))
+  )
   (text "Data Input" (at 92.71 79.375 0)
     (effects (font (size 1.27 1.27)) (justify left bottom))
@@
     (effects (font (size 1.27 1.27)) (justify left bottom))
   )
-  (label "P15_5" (at 469.9 497.205 0) (fields_autoplaced)
-    (effects (font (size 1.27 1.27)) (justify left bottom))
-  )
   (label "P15_47" (at 161.29 112.395 0) (fields_autoplaced)
     (effects (font (size 1.27 1.27) bold) (justify left bottom))
@@
     (effects (font (size 1.27 1.27)) (justify left bottom))
   )
-  (label "P15_19" (at 469.9 487.045 0) (fields_autoplaced)
-    (effects (font (size 1.27 1.27)) (justify left bottom))
-  )

Commit message: Talk To Me
Other:
- note added: "↑1"
- note added: "↓1"
Changed lines of the file:
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@@
     (effects (font (size 3 3) (thickness 1) bold (color 18 244 255 1)) (justify left bottom))
+  )
+  (text "↑1" (at 184.15 55.88 0)
+    (effects (font (size 2 2) (thickness 0.4) bold (color 2 138 15 1)) (justify left bottom))
   )
   (text "Processor\n" (at 222.885 802.005 0)
@@
     (effects (font (size 3 3) (thickness 1) bold (color 5 102 8 1)) (justify right bottom))
   )
+  (text "↓1" (at 184.15 42.545 0)
+    (effects (font (size 2 2) (thickness 0.6) bold (color 203 17 29 1)) (justify left bottom))
+  )
   (text "*" (at 146.05 194.945 0)
     (effects (font (size 3 3) (thickness 1) bold (color 18 244 255 1)) (justify left bottom))
@@
     (effects (font (size 1.27 1.27)) (justify left bottom))
   )
+  (text "↑1" (at 184.15 63.5 0)
+    (effects (font (size 2 2) (thickness 0.4) bold (color 2 138 15 1)) (justify left bottom))
+  )
   (text "Data Input" (at 112.395 227.965 0)

Commit message: fix
Connections:
- net XX(UA7P3) is gone; now on net u7-13: UA7.3
- no-connect marks 54 -> 53
Other:
- note added: "HIGH on power up"
- note added: "LOW on power up"

Commit message: cleanup
Parts:
- removed R18: 1k, Resistor_THT:R_Axial_DIN0207_L6.3mm_D2.5mm_P10.16mm_Horizontal, symbol SamacSys_Parts:YR1B24K9CC
- added R1: 1k, Resistor_THT:R_Axial_DIN0207_L6.3mm_D2.5mm_P10.16mm_Horizontal, symbol SamacSys_Parts:YR1B24K9CC
Connections:
- net U44P5: now also R1.1
- net VCC: now also R1.2

Commit message: tweaks
Other:
- note added: "Goes low every 9th & 10th clock cycle"
Changed lines of the file:
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@@
     (effects (font (size 3 3) (thickness 1) bold (color 18 244 255 1)) (justify left bottom))
+  )
+  (text "Goes low every 9th & 10th clock cycle" (at 373.38 374.015 0)
+    (effects (font (size 0.5 0.5)) (justify left bottom))
   )
   (text "*" (at 26.67 42.545 0)
@@
     (effects (font (size 3 3) (thickness 1) bold (color 18 244 255 1)) (justify left bottom))
   )
+  (text "Goes low every 9th & 10th clock cycle" (at 542.925 349.885 0)
+    (effects (font (size 0.5 0.5)) (justify left bottom))
+  )
   (text "↓1" (at 334.645 505.46 0)
