File: Trapezoid_Terminal/Keyboard/Entrex Trapezoid Keyboard Typewriter.kicad_sch (KiCad schematic)
At the start: 58 parts, among them J1 Conn_02x12_Top_Bottom, U1 74LS00, U2 8748, U3 SN75453, U4 74LS04, U5 74LS04, U6 7442, U7 LM319, U8 74LS145

Commit message: kbd
Parts:
- J1: footprint (none) -> Forgotten Machines:Card_Edge_Entrex_Trapezoid Keyboard
- R16: footprint (none) -> Forgotten Machines:Disc Capacitor Entrex Trapezoid .25
- U1: footprint (none) -> Package_DIP:DIP-14_W7.62mm
Changed lines of the file:
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@@
       (effects (font (size 1.27 1.27)))
     )
-    (property "Footprint" "" (at 538.48 224.79 0)
+    (property "Footprint" "Package_DIP:DIP-14_W7.62mm" (at 538.48 224.79 0)
       (effects (font (size 1.27 1.27)) hide)
     )
@@
       (effects (font (size 1.27 1.27)))
     )
-    (property "Footprint" "" (at 506.095 205.105 0)
+    (property "Footprint" "Package_DIP:DIP-14_W7.62mm" (at 506.095 205.105 0)
       (effects (font (size 1.27 1.27)) hide)
     )
@@
       (effects (font (size 1.27 1.27)))
     )
-    (property "Footprint" "" (at 505.46 221.615 0)
+    (property "Footprint" "Package_DIP:DIP-14_W7.62mm" (at 505.46 221.615 0)
       (effects (font (size 1.27 1.27)) hide)
     )
@@
       (effects (font (size 1.27 1.27)) (justify left))
     )
-    (property "Footprint" "" (at 405.892 137.16 90)
+    (property "Footprint" "Forgotten Machines:Disc Capacitor Entrex Trapezoid .25" (at 405.892 137.16 90)
       (effects (font (size 1.27 1.27)) hide)
     )
@@
       (effects (font (size 1.27 1.27)) (justify left) hide)
     )
-    (property "Footprint" "" (at 501.015 111.76 0)
+    (property "Footprint" "Forgotten Machines:Card_Edge_Entrex_Trapezoid Keyboard" (at 501.015 111.76 0)
       (effects (font (size 1.27 1.27)) hide)
     )
@@
       (effects (font (size 1.27 1.27)))
     )
-    (property "Footprint" "" (at 525.78 165.1 0)
+    (property "Footprint" "Package_DIP:DIP-14_W7.62mm" (at 525.78 165.1 0)
       (effects (font (size 1.27 1.27)) hide)
     )
@@
       (effects (font (size 1.27 1.27)))
     )
-    (property "Footprint" "" (at 538.48 204.47 0)
-      (effects (font (size 1.27 1.27)) hide)
-    )
+    (property "Footprint" "Package_DIP:DIP-14_W7.62mm" (at 538.48 204.47 0)
+      (effects (font (size 1.27 1.27)) hide)
+    )

Commit message: keyboard
Parts:
- C1, C10, C11, C12, C13, C14, C2, C3, C4, C6, C7, C8, R1, R10, R11, R12, R13, R14, R15, R17, R18, R19, R2, R20, R3, R4, R5, R6, R7, R8, R9: footprint (none) -> Forgotten Machines:Resistor-Cap-P10.16mm_Horizontal
- C5: footprint (none) -> Forgotten Machines:Disc Capacitor Entrex Trapezoid .125
- C9: footprint (none) -> Forgotten Machines:CAP Medium Polarized
- JP1, JP3: footprint (none) -> Forgotten Machines:Wire Jumper 0.325in
- R16: footprint Forgotten Machines:Disc Capacitor Entrex Trapezoid .25 -> Forgotten Machines:Resistor-Cap-P10.16mm_Horizontal
Connections:
- net U8_1: now reaches U8.1 (Q0)
- net U8_10: now reaches U8.10 (Q8)
- net U8_11: now reaches U8.11 (Q9)
- net U8_12: now reaches U8.12 (P3)
- net U8_13: now reaches U8.13 (P2)
- net U8_14: now reaches U8.14 (P1)
- net U8_15: now reaches U8.15 (P0)
- net U8_2: now reaches U8.2 (Q1)
- net U8_3: now reaches U8.3 (Q2)
- net U8_4: now reaches U8.4 (Q3)
- net U8_5: now reaches U8.5 (Q4)
- net U8_6: now reaches U8.6 (Q5)
- net U8_7: now reaches U8.7 (Q6)
- net U8_9: now reaches U8.9 (Q7)
Other:
- moved on the sheet: C1, C10, C11, C12, C2, C3, C7, C8, C9, D1, D2, D3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

Commit message: Keyboard
Connections:
- net J1_1 is gone; now on net VCC: J1.1 (Pin_1)
- net J1_2 is gone; now on net GND: J1.2 (Pin_2)
- net J1_A is gone; now on net VCC: J1.13 (Pin_13)
- net J1_B is gone; now on net GND: J1.14 (Pin_14)
- net J1_N is gone; now on net J1_12: J1.24 (Pin_24)
- net U1_10 is gone; now on net P1.2: U1.10
- net U1_12 is gone; now on net P2.0: U1.12
- net U1_13 is gone; now on net P1.3: U1.13
- net U1_2 is gone; now on net T1: U1.2
- net U1_4 is gone; now on net U1_3: U1.4
- net U1_5 is gone; now on net P2.1: U1.5
- net U1_6 is gone; now on net T1: U1.6
- net U1_9 is gone; now on net P2.0: U1.9
- net U3_6 is gone; now on net EA: U3.6 (2A)
- net U4_10 is gone; now on net J1_H: U4.10
- net U4_12 is gone; now on net J1_L: U4.12
- net U4_13 is gone; now on net DB.2: U4.13
- net U4_2 is gone; now on net J1_11: U4.2
- net U4_4 is gone; now on net J1_10: U4.4
- net U4_5 is gone; now on net DB.3: U4.5
- net U4_6 is gone; now on net J1_9: U4.6
- net U4_8 is gone; now on net J1_8: U4.8
- net U4_9 is gone; now on net DB.4: U4.9
- net U5_10 is gone; now on net J1_J: U5.10
- net U5_11 is gone; now on net DB.0: U5.11
- net U5_12 is gone; now on net J1_K: U5.12
- net U5_13 is gone; now on net DB.1: U5.13
- net U5_2 is gone; now on net J1_5: U5.2
- net U5_4 is gone; now on net J1_4: U5.4
- net U5_6 is gone; now on net J1_3: U5.6
- net U5_8 is gone; now on net U1_1: U5.8
- net U7_12 is gone; now on net U5_9: U7.12
- net VDD is gone; now on net GND: U7.6 (V-)
- net Vpp/VDD is gone; now on net VCC: U2.26 (Vpp/VDD)
- net ~{SS} is gone; now on net ~{INT}: U2.5 (~{SS})
- net GND: now also C12.1, C5.2, C6.1, C7.1, D1.1 (K), JP1.1 (A)
- net J1_10: now also J1.22 (Pin_22); no longer J1.10 (Pin_10)
- net J1_11: now also J1.23 (Pin_23); no longer J1.11 (Pin_11)
- net J1_12: no longer J1.12 (Pin_12)
- net J1_3: now also J1.15 (Pin_15); no longer J1.3 (Pin_3)
- net J1_4: now also J1.16 (Pin_16); no longer J1.4 (Pin_4)
- net J1_5: now also J1.17 (Pin_17); no longer J1.5 (Pin_5)
- net J1_6: now also J1.18 (Pin_18), R4.2; no longer J1.6 (Pin_6)
- net J1_7: now also J1.19 (Pin_19); no longer J1.7 (Pin_7)
- net J1_8: now also J1.20 (Pin_20); no longer J1.8 (Pin_8)
- net J1_9: now also J1.21 (Pin_21); no longer J1.9 (Pin_9)
- net J1_C: now also J1.3 (Pin_3); no longer J1.15 (Pin_15)
- net J1_D: now also J1.4 (Pin_4); no longer J1.16 (Pin_16)
- net J1_E: now also J1.5 (Pin_5), R3.2; no longer J1.17 (Pin_17)
- net J1_F: now also J1.6 (Pin_6); no longer J1.18 (Pin_18)
- net J1_H: now also J1.7 (Pin_7); no longer J1.19 (Pin_19)
- net J1_J: now also J1.8 (Pin_8); no longer J1.20 (Pin_20)
- net J1_K: now also J1.9 (Pin_9); no longer J1.21 (Pin_21)
- net J1_L: now also J1.10 (Pin_10); no longer J1.22 (Pin_22)
- net J1_M: now also J1.11 (Pin_11), JP1.2 (B); no longer J1.23 (Pin_23)
- net T0: now also JP3.1 (A), R2.2
- net U5_9: now also R5.2
- net U7_10: now also D2.2 (A), R6.2
- net U7_4: now also C11.2, R18.2
- net U7_5: now also R13.2
- net U7_7: now also C8.2, R8.2, R9.2
- net U7_9: now also R7.2
- net VCC: now also C5.1, C6.2, C7.2
- net X1: now also C1.2, YJ1.2
- net X2: now also C3.2, YJ1.1
- net ~{INT}: now also R1.1
- net Ax: now reaches C11.1
- net Ax: now also C12.2, R19.2
- net Net-(D3-K): now reaches R10.2
- net D1-D2: now reaches D1.2 (A)
- net D1-D2: now also D2.1 (K)
- new net -12v(J1_N): J1.12 (Pin_12)

Commit message: keyboard
Connections:
- net EA is gone; now on net GND: U2.7 (EA), U3.6 (2A)
- net U3_7 is gone; now on net P2.4: U3.7 (2B)
- net U8_12 is gone; now on net U1_11: U8.12 (P3)
- net U8_13 is gone; now on net U1_8: U8.13 (P2)
Other:
- note added: "= NC on Backplane/Board/Cable"
- note added: "x"
- moved on the sheet: C1, C10, C11, C12, C13, C14, C2, C3, C5, C6, C7, C8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
