File: Trapezoid_Terminal/Interface Board/Phar's Versions/Entrex Trapezoid Interface Board v23.kicad_pcb (KiCad board)
At the start: 2 copper layers, 169.1 x 191 mm, 101 parts, among them P15 Conn_02x40_Odd_Even_Shielded, SW1 SW_DIP_x08

Commit message: UB5B Pin 11
Connections:
- UA1 pad 13: VCC -> u36_13
- UA2 pad 13: VCC -> u36_13
- UA7 pad 3: u7-13 -> /XX(UA7P3)
- UB5 pad 11: u20_3 -> /XX(UB5P11)
- UB8 pad 12: u2_10 -> /XX(UB8P12)
Routing:
- net VCC: track 1895.0 -> 1871.5 mm, vias 8 -> 7
- net u36_13: track 0.00 -> 23.4 mm
- net u20_3: track 372.5 -> 363.8 mm
- net u7-13: track 280.8 -> 272.1 mm
- net u2_10: track 93.9 -> 92.4 mm
