File: Trapezoid_Terminal/Interface Board/Phar's Versions/Entrex Trapezoid Interface Board v23.kicad_sch (KiCad schematic)
At the start: 108 parts, among them P15 Conn_02x40_Odd_Even_Shielded, SW1 SW_DIP_x08

Commit message: Testing x2
Parts:
- removed unit 1 of UA6
- removed unit 4 of UA6
- removed unit 2 of UB1
- removed unit 2 of UB5
- removed unit 3 of UC6
- renumbered UB2 to UB8, UD4 to UD7, UD2 to UD8
Connections:
- net at UE7.5, UF3.2, UF3.4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: no longer UA5.1 (C), UA5.6 (C), UC2.2, UF6.13
- net at C26.2: now also UD5.4 (1RTC)
- net bit_counter_overflow: now reaches UB8.10, UD8.9, UE8.15 (Tc)
- net bit_counter_overflow: now also UB8.12
- net latch_status_d0 renamed term_selectd_and_S0
- net set_unknown_status_1 renamed n_has_RX'd_16_bits
- new net: UA5.1 (C), UA5.6 (C), UF6.13
- no-connect marks 83 -> 80
Other:
- note added: "0b0000"
- note added: "0b1000 NAND term_select"
- note added: "0bxx00"
- note added: "0bxx1x &term_select &single_ended_rts &_not_was_single_ended_rts"
- note added: "0bxx1x NAND term_selet"
- note added: "0bxxx1 NAND term_seler"
- note added: "AND"
- note added: "seems to be part of enabling serial transmitter"
- note added: "was_single_ended_rts"
- moved on the sheet: UC2E, UF6A, UF6B, UF7A
