File: DataScope/Power Supply/Power Supply - Entrex DataScope.kicad_sch (KiCad schematic)
At the start: 128 parts, among them J2 Conn_02x04_Odd_Even, Q1 MPS3638, Q10 PN3569, Q11 PS3638, Q12 2N4918, Q13 2N3055, Q14 PN3569, Q15 PS3638, Q16 PN3569, Q17 PN3569, Q18 PS3638, Q19 JE520, Q2 PN3569, Q20 PN3569, Q3 PN3569, Q4 PS3638, Q5 2N4918, Q6 2N3055, Q7 PN3569, Q8 PS3638, Q9 PN3569

Commit message: build
Parts:
- J2: value Conn_02x04_Odd_Even -> Power Port
Connections:
- net SCR2P2: now also R48.2
Other:
- moved on the sheet: C1, C10, C11, C12, C4, C9, CR1, CR18, CR19, CR20, CR21, CR22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

Commit message: build
Other:
- moved on the sheet: C4, R10, R17, R18, R7, R8, SCR1

Commit message: build
Other:
- moved on the sheet: CR7, Q3, Q7, R13, R15, R8

Commit message: Build
Connections:
- net Q13P2: now also R32.1
- net Q14P2: now also R30.2
Other:
- moved on the sheet: C1, C10, C11, C12, C3, C4, C5, C6, C7, C8, C9, CR1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

Commit message: Add Images
Parts:
- removed CR1, CR2, CR3, CR4: 1N4001, Diode_THT:D_DO-41_SOD81_P12.70mm_Horizontal, symbol ForgottenMachines:1N4001_Entrex_PSU
- added CR1, CR2, CR3, CR4: 1N4001, Diode_THT:D_DO-41_SOD81_P12.70mm_Horizontal, symbol ForgottenMachines:Diagonal Diode for Full Wave Bridge Lower
- R33: value R -> 0.22Ω
Connections:
- net 5vGND: now also CR1., CR3.
- net C1+: now also CR2., CR4.
- net E1: now also CR1., CR2.
- net E2: now also CR3., CR4.
Other:
- note added: "+14v DC"
- moved on the sheet: C1, CR5, CR6, E1, E2, R1

Commit message: Update Power Supply - Entrex DataScope.kicad_sch
Other:
- note added: "+23v DC"
Changed lines of the file:
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@@
     (effects (font (size 5 5) (thickness 1) bold) (justify left bottom))
+  )
+  (text "+23v DC" (at 401.955 380.365 0)
+    (effects (font (size 2 2) (thickness 0.4) bold) (justify left bottom))
   )
   (label "Q7P2" (at 486.41 320.675 270) (fields_autoplaced)

Commit message: resistors
Parts:
- R1, R6, R8: value R -> 1kΩ
- R10, R13, R28: value R -> 270Ω
- R11, R3, R49: value R -> 390Ω
- R12, R27, R46, R9: value R -> 470Ω
- R14, R18, R29, R32: value R -> 100Ω
- R15: value R -> 0.1Ω
- R16: value R -> 120Ω
- R17: value R -> ∞Ω
- R19, R24, R35, R40, R7: value R -> 1KΩ
- R2: value R -> 2.2kΩ
- R20: value R -> 3.4KΩ
- R21, R25, R37, R41, R44, R45: value R -> 1.5KΩ
- R22: value R -> 1.8KΩ
- R23: value R -> 3KΩ
- R26, R34, R42: value R -> 680Ω
- R30, R31: value R -> 1.5kΩ
- R38: value R -> 81KΩ
- R39, R4: value R -> 3kΩ
- R43: value R -> 91Ω
- R47: value R -> 1.2Ω
- R48: value R -> 1.2KΩ
- R5: value R -> 2.4kΩ
- R51: value R -> 68Ω

Commit message: mpre
Other:
- note added: "+0.68v"
- note added: "+0.7v"
- note added: "+18.5v"
- note added: "+3.3v"
- note added: "+4.0v"
- note added: "+4.6v"
- note added: "+6.2v"
- note added: "0v"
- note added: "v AC"
- moved on the sheet: C1, C3, C4, CR1, CR2, CR3, CR4, CR5, CR6, CR7, E1, E2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
