File: Front Panel (Entrex)/Tester - Entrex Front Panel/Tester - Entrex Front Panel.kicad_pcb (KiCad board)
At the start: 2 copper layers, 114 x 99 mm, 11 parts, among them J1 Slot_02x26, J2 Conn_01x04, J3 Conn_01x08, J4 Conn_01x08, J5 Conn_01x06, J6 Conn_01x04, J7 Conn_01x02, J8 Conn_01x19

Commit message: Front Panel Tester
Parts:
- moved G*** 13.8 mm to (103.4, 86.1)
Routing:
- net +5V: track 259.9 -> 0.00 mm
- net D2: track 209.2 -> 0.00 mm, vias 1 -> 0
- net ~{CON DATA}: track 204.7 -> 0.00 mm, vias 1 -> 0
- net ~{CONT+ISTP+MSTP}: track 202.4 -> 0.00 mm, vias 1 -> 0
- net ~{STOP}: track 194.3 -> 0.00 mm, vias 2 -> 0
- net ~{ISTP}: track 183.2 -> 0.00 mm, vias 2 -> 0
- net ~{PL}: track 181.9 -> 0.00 mm, vias 2 -> 0
- net ~{CON INST}: track 178.7 -> 0.00 mm, vias 2 -> 0
- net ~{CON RQ}: track 177.6 -> 0.00 mm, vias 2 -> 0
- net ~{RST}: track 174.7 -> 0.00 mm, vias 2 -> 0
- net RESTART ENABLE: track 170.5 -> 0.00 mm, vias 2 -> 0
- net D48: track 139.7 -> 0.00 mm, vias 1 -> 0
- net D47: track 138.1 -> 0.00 mm, vias 1 -> 0
- net D46: track 137.6 -> 0.00 mm, vias 2 -> 0
- net D44: track 129.4 -> 0.00 mm, vias 2 -> 0
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Other:
- board text added: "Entrex 480 / Nixdorf 620 Front Panel Tester"
- board text removed: "DG Nova / DCC D116"
- board text removed: "Entrex 480 / Nixdorf 620"
- board text removed: "Forgotten Machines"
- board text removed: "Front Panel Tester"
