File: Front Panel (Entrex)/Tester - Entrex Front Panel/Tester - Entrex Front Panel.kicad_pcb (KiCad board)
At the start: 2 copper layers, 114 x 99 mm, 15 parts, among them J1 Logic 8 CH, J10 Conn_02x26_Top_Bottom, J11 Logic 8 CH, J12 Logic 8 CH, J2 Conn_01x04, J3 Conn_01x08, J4 Conn_01x08, J5 Conn_01x06, J6 Conn_01x04, J7 Conn_01x02, J8 Conn_01x19, J9 Logic 8 CH, SW1 Reset

Commit message: build
Changed lines of the file:
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@@
     (effects (font (size 0.7 0.7) (thickness 0.15)))
   )
-  (gr_text "Front Panel" (at 93.35 47.9) (layer "F.SilkS")
+  (gr_text "Front Panel" (at 94.234 47.625) (layer "F.SilkS")
     (effects (font (size 1.2 1.2) (thickness 0.15)))
   )

Commit message: build
Connections:
- J11 pad 9: unconnected-(J11-Pin_9-Pad9) -> GND
- J12 pad 9: unconnected-(J12-Pin_9-Pad9) -> GND
- J9 pad 9: unconnected-(J9-Pin_9-Pad9) -> GND
Routing:
- net GND: track 32.6 -> 40.7 mm, vias 7 -> 8

Commit message: front panel tester DRC
Routing:
- net ~{64K}: track 62.1 -> 58.6 mm
- net GND: track 40.7 -> 44.2 mm, vias 8 -> 10
- net ~{MEM5}: track 147.8 -> 145.1 mm
- net +V LAMP: track 73.4 -> 70.7 mm
- net +5V: track 127.5 -> 125.0 mm
- net ~{MEM10}: track 141.0 -> 138.9 mm
- net ~{MEM0}: track 159.1 -> 157.1 mm
- net Logic6: track 61.3 -> 59.6 mm
- net Net-(J7-Pin_1): track 25.4 -> 24.2 mm
- net ~{MEM12}: track 95.2 -> 94.0 mm
- net ~{DISK RDY}: track 120.4 -> 119.2 mm
- net ~{CON RQ}: track 98.6 -> 97.5 mm
- net D9: track 74.1 -> 73.0 mm
- net D13: track 71.5 -> 70.8 mm
- net Net-(J8-Pin_3): track 76.7 -> 76.1 mm
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
Commit message: mmm
Changed lines of the file:
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@@
     (solder_mask_min_width 0.25)
     (pcbplotparams
-      (layerselection 0x00010fc_ffffffff)
+      (layerselection 0x00310fc_ffffffff)
       (plot_on_all_layers_selection 0x0000000_00000000)
       (disableapertmacros false)
@@
   (segment (start 81.788 56.644) (end 83.176 55.256) (width 0.254) (layer "F.Cu") (net 45))
   (segment (start 52.705 44.704) (end 53.467 43.942) (width 0.25) (layer "F.Cu") (net 46))
-  (segment (start 44.718 52.691) (end 51.816 45.593) (width 0.25) (layer "F.Cu") (net 46))
+  (segment (start 45.085 112.623) (end 45.606 113.144) (width 0.25) (layer "F.Cu") (net 46))
   (segment (start 52.705 44.704) (end 53.34 44.069) (width 0.25) (layer "F.Cu") (net 46))
-  (segment (start 51.816 45.593) (end 52.705 44.704) (width 0.25) (layer "F.Cu") (net 46))
-  (segment (start 61.875 129.413) (end 44.718 112.256) (width 0.25) (layer "F.Cu") (net 46))
+  (segment (start 61.875 129.413) (end 45.606 113.144) (width 0.25) (layer "F.Cu") (net 46))
+  (segment (start 45.085 52.324) (end 45.085 112.623) (width 0.25) (layer "F.Cu") (net 46))
+  (segment (start 52.705 44.704) (end 45.085 52.324) (width 0.25) (layer "F.Cu") (net 46))
   (segment (start 61.875 136.22) (end 61.875 129.413) (width 0.25) (layer "F.Cu") (net 46))
-  (segment (start 44.718 112.256) (end 44.718 52.691) (width 0.25) (layer "F.Cu") (net 46))
   (via (at 53.34 44.069) (size 0.6) (drill 0.3) (layers "F.Cu" "B.Cu") (net 46))
   (segment (start 57.404 42.686) (end 54.723 42.686) (width 0.254) (layer "B.Cu") (net 46))
