File: Front Panel (Entrex)/Tester - Entrex Front Panel/Tester - Entrex Front Panel.kicad_sch (KiCad schematic)
At the start: 11 parts, among them J1 Conn_02x26_Top_Bottom, J1 Slot_02x26, J2 Conn_01x04, J3 Conn_01x08, J4 Conn_01x08, J5 Conn_01x06, J6 Conn_01x04, J7 Conn_01x02, J8 Conn_01x19, SW1 SW_Push

Commit message: Front Panel Tester
Parts:
- removed J1: Slot_02x26, port_nova:port_Nova_52pin, symbol port_nova:Slot_02x26
- added J1: Logic 8 CH, Connector_PinHeader_2.54mm:PinHeader_1x08_P2.54mm_Vertical, symbol Connector_Generic:Conn_01x08
- added J11, J12, J9: Logic 8 CH, Forgotten Machines:PinHeader_2x05_P2.54mm_Vertical - Backside, symbol Connector_Generic:Conn_02x05_Odd_Even
- J1: footprint Forgotten Machines:DG NOVA Front Pannel Connector -> Forgotten Machines:DG Nova Front Panel Card Edge
- J2: footprint port_nova:PinHeader_1x04_P2.54mm_Vertical -> Connector_PinHeader_2.54mm:PinHeader_1x05_P2.54mm_Vertical; symbol Connector_Generic:Conn_01x04 -> Connector_Generic:Conn_01x05
Connections:
- net D15 is gone; now on net ~{CON RQ}: XA1.D15 (D15_RX3)
- net D16 is gone; now on net ~{M CON DATA}: XA1.D16 (D16_TX2)
- net D17 is gone; now on net ~{CON DATA}: XA1.D17 (D17_RX2)
- net D18 is gone; now on net ~{M CON INST}: XA1.D18 (D18_TX1)
- net D19 is gone; now on net ~{CON INST}: XA1.D19 (D19_RX1)
- net D20 is gone; now on net 64K: XA1.D20 (D20_SDA)
- net D21 is gone; now on net ~{64K}: XA1.D21 (D21_SCL)
- net D22 is gone; now on net ~{MBO0}: XA1.D22
- net D23 is gone; now on net ~{MEM0}: XA1.D23
- net D24 is gone; now on net ~{MEM1}: XA1.D24
- net D25 is gone; now on net ~{MEM2}: XA1.D25
- net D26 is gone; now on net ~{MEM3}: XA1.D26
- net D27 is gone; now on net ~{MEM4}: XA1.D27
- net D28 is gone; now on net ~{MEM5}: XA1.D28
- net D29 is gone; now on net ~{MEM6}: XA1.D29
- net D30 is gone; now on net ~{MEM7}: XA1.D30
- net D31 is gone; now on net 52: XA1.D31
- net D32 is gone; now on net ~{MEM9}: XA1.D32
- net D33 is gone; now on net ~{MEM10}: XA1.D33
- net D34 is gone; now on net ~{MEM11}: XA1.D34
- net D35 is gone; now on net ~{MEM12}: XA1.D35
- net D36 is gone; now on net ~{MEM13}: XA1.D36
- net D37 is gone; now on net ~{MEM14}: XA1.D37
- net D38 is gone; now on net ~{MEM15}: XA1.D38
- net D39 is gone; now on net ~{RUN}: XA1.D39
- net D40 is gone; now on net ~{RST}: XA1.D40
- net D42 is gone; now on net ~{MA LOAD}: XA1.D42
- net D43 is gone; now on net ~{DCHP OUT}: XA1.D43
- net D44 is gone; now on net ~{POWER FAIL}: XA1.D44
- net D45 is gone; now on net ~{SCNR BUSY}: XA1.D45
- net D46 is gone; now on net ~{DISK RDY}: XA1.D46
- net D47 is gone; now on net DISK CS: XA1.D47
- net D48 is gone; now on net TAPE CS: XA1.D48
- net D49 is gone; now on net EXT CS: XA1.D49
- net D50 is gone; now on net SWITCHOVER POWER: XA1.D50
- net D51 is gone; now on net ~{NORMAL}: XA1.D51
- net +5V: now also J6.3 (Pin_3), J6.4 (Pin_4)
- net -5V: now also J2.5 (Pin_5)
- net D DEFER AGAIN: now also J3.4 (Pin_4), XA1.A11
- net GND: now also J6.1 (Pin_1), J6.2 (Pin_2), J11.10 (Pin_10), J12.10 (Pin_10), J9.10 (Pin_10)
- net S10: now also J7.1 (Pin_1), XA1.D52
- net S2: now also J3.8 (Pin_8), XA1.A15
- net S3: now also J3.7 (Pin_7), XA1.A14
- net S4: now also J3.6 (Pin_6), XA1.A13
- net S5: now also J3.5 (Pin_5), XA1.A12
- net ~{CON DATA}: no longer J6.3 (Pin_3), J8.2 (Pin_2), XA1.D0 (D0_RX0)
- net ~{CON INST}: no longer J4.5 (Pin_5), J5.3 (Pin_3), XA1.A4
- net ~{CON RQ}: now also J11.3 (Pin_3); no longer J4.6 (Pin_6), J5.4 (Pin_4), XA1.A5
- net ~{M CON DATA}: now also J11.2 (Pin_2), J9.8 (Pin_8)
- net ~{M CON INST}: now also J11.1 (Pin_1)
- net ~{MEM0}: now also J11.8 (Pin_8), J9.5 (Pin_5)
- net ~{MEM10}: now also J9.7 (Pin_7)
- net ~{MEM2}: now also J11.5 (Pin_5), J9.2 (Pin_2)
- net ~{MEM5}: now also J11.6 (Pin_6), J9.3 (Pin_3)
- net ~{MEM6}: now also J11.4 (Pin_4), J9.1 (Pin_1)
- net ~{MEM9}: now also J9.6 (Pin_6)
- net ~{RST}: now also J11.7 (Pin_7), J9.4 (Pin_4); no longer J4.7 (Pin_7), J5.5 (Pin_5), XA1.A6
- net at J1.23 (Pin_23): now also J5.3 (Pin_3)
- net at J1.25 (Pin_25): now also J5.2 (Pin_2)
- net at J1.26 (Pin_26): now also J5.1 (Pin_1)
- net D2: no longer names the net of XA1.D2 (D2_INT0)
- net D2: now also J8.1 (Pin_1)
- net D41: no longer names the net of XA1.D41
- net RESTART ENABLE: no longer names the net of J4.8 (Pin_8), XA1.A7
- net RESTART ENABLE: no longer J5.6 (Pin_6)
- removed net ~{CONT+ISTP+MSTP}: J6.2 (Pin_2), J8.3 (Pin_3), XA1.D1 (D1_TX0)
- net ~{ISTP}: no longer names the net of J4.3 (Pin_3), XA1.A2
- net ~{ISTP}: no longer J5.1 (Pin_1)
- net ~{MSTP}: no longer names the net of J8.4 (Pin_4)
- net ~{MSTP}: now also XA1.D14 (D14_TX3); no longer J6.1 (Pin_1)
- net ~{PL}: no longer names the net of J4.4 (Pin_4), XA1.A3
- net ~{PL}: no longer J5.2 (Pin_2)
- removed net ~{STOP}: J6.4 (Pin_4), J8.1 (Pin_1), XA1.D14 (D14_TX3)
- new net: J4.5 (Pin_5), XA1.A4
- new net: J4.6 (Pin_6), XA1.A5
- new net: J4.7 (Pin_7), XA1.A6
- new net: J8.3 (Pin_3), XA1.D0 (D0_RX0)
- new net: J8.2 (Pin_2), XA1.D1 (D1_TX0)
- new net Logic1: J1.1 (Pin_1), J12.1 (Pin_1)
- new net Logic2: J1.2 (Pin_2), J12.2 (Pin_2)
- new net Logic3: J1.3 (Pin_3), J12.3 (Pin_3)
- new net Logic4: J1.4 (Pin_4), J12.4 (Pin_4)
- new net Logic5: J1.5 (Pin_5), J12.5 (Pin_5)
- new net Logic6: J1.6 (Pin_6), J12.6 (Pin_6)
- new net Logic7: J1.7 (Pin_7), J12.7 (Pin_7)
- new net Logic8: J1.8 (Pin_8), J12.8 (Pin_8)
Other:
- note removed: "Address 15 light"
- note removed: "Data Light 15"
- note removed: "NOT used??!!!"
- note removed: "RESTART_ENAB = A7; // input from the CPU... connected to center/common of Reset & Stop switches, so must be low to test those RST = A6; // RESET CON_RQ = A5; //used by multiple switches???? CON_INST = A4; // input from the CPU..."the twin of CON_DATA - nevets01" PL = A3; // PROG LOAD - Has it's own wire to p1-23 ISTP = A2; // INST STEP - Has it's own wire to p1-24 STOP = 14; // STOP CON_DATA = 0;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"
- note removed: "to +V LAMP trace at bottom- right corner of backplane PCB"
- moved on the sheet: J1, J5, J6, J7, J8
