File: Front Panel (Entrex)/Tester - Entrex Front Panel/Status Board - Tester - Entrex front Panel.kicad_pcb (KiCad board)
At the start: 2 copper layers, 114 x 44.9 mm, 5 parts, among them J3 Conn_01x08, J4 Conn_01x08, J7 Conn_01x02, J8 Conn_01x19

Commit message: DRC Checks p1
Changed lines of the file:
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@@
     (polygon
       (pts
-        (xy 42.799 36.576)
-        (xy 42.418 144.399)
-        (xy 164.465 144.272)
-        (xy 164.592 36.322)
+        (xy 44.5 41.25)
+        (xy 44.65 86.4)
+        (xy 158.45 86.2)
+        (xy 158.65 41.25)
       )
     )
@@
     (polygon
       (pts
-        (xy 161.798 145.923)
-        (xy 44.069 143.637)
-        (xy 44.568 37.663)
-        (xy 162.251 38.171)
+        (xy 158.45 86.2)
+        (xy 44.65 86.4)
+        (xy 44.5 41.25)
+        (xy 158.65 41.25)
       )
     )
