File: Mystery Test Board/AMLDC-2044B.kicad_sch (KiCad schematic)
At the start: 321 parts, among them J1 Port A, J2 Port B, Q1 PNP MPS6533, Y1 Crystal

Commit message: Chips Placed First Wave
Parts:
- C6: footprint FM-editable:Capacitor non-polarized P25.00mm -> Forgotten Machines:CAP non-polarized P25.00mm
- UL5, UN0, UU5: footprint (none) -> Package_DIP:DIP-14_W7.62mm
- UM8: footprint (none) -> Package_DIP:DIP-16_W7.62mm
- US2: footprint Package_DIP:DIP-16_W7.62mm -> Package_DIP:DIP-14_W7.62mm
- Y1: footprint (none) -> Crystal:Crystal_HC49-U_Horizontal_1EP_style1
- renumbered UD2 to UD3, UH1 to UH2
Connections:
- net D2p10: no longer UD2.11
- net K5p11: now also UK5.11
- net L5p1: now also UL5.1
- net L5p2: now also UL5.2
- net L5p4: now also UL5.4
- net L5p5: now also UL5.5
- net L5p6: now also UL5.6
- net M8p1: now also UM8.1 (C)
- net M8p14: now also UM8.14 (~{Q})
- net M8p15: now also UM8.15 (Q)
- net M8p16: now also UM8.16 (K)
- net M8p2: now also UM8.2 (~{S})
- net M8p3: now also UM8.3 (~{R})
- net M8p4: now also UM8.4 (J)
- new net D2p11: UD2.11
Other:
- moved on the sheet: UL5A, UM8A

Commit message: Place Missing Chips
Parts:
- added U1, UF3: 9328, Package_DIP:DIP-16_W7.62mm, symbol ForgottenMachines:DM9328
- added UB3: DM958, symbol ForgottenMachines:DM958
Connections:
- new net B3p1: UB3.1
- new net B3p10: UB3.10
- new net B3p11: UB3.11
- new net B3p12: UB3.12
- new net B3p13: UB3.13
- new net B3p2: UB3.2
- new net B3p3: UB3.3
- new net B3p4: UB3.4
- new net B3p5: UB3.5
- new net B3p6: UB3.6
- new net B3p8: UB3.8
- new net B3p9: UB3.9
- new net F3p1: UF3.1
- new net F3p10: UF3.10
- new net F3p11: UF3.11 (D0)
- new net F3p12: UF3.12 (D1)
- new net F3p13: UF3.13 (S)
- new net F3p14: UF3.14 (Q7)
- new net F3p15: UF3.15 (Q7)
- new net F3p2: UF3.2 (Q7)
- new net F3p3: UF3.3 (Q7)
- new net F3p4: UF3.4 (S)
- new net F3p5: UF3.5 (D0)
- new net F3p6: UF3.6 (D1)
- new net F3p7: UF3.7
- new net F3p9: UF3.9

Commit message: Right before 1st board tracing picture removal and addition of second
Parts:
- added JP1, JP2, JP3, JP4, JP5, JP6: Vipass Ammeter, Forgotten Machines:DG Nova Board Jumper 5mm, symbol Jumper:Jumper_2_Open
- added JP7, JP8: Vipass Ammeter, Forgotten Machines:DG Nova Board Jumper 3.8mm, symbol Jumper:Jumper_2_Open
- CR1: footprint Forgotten Machines:Diode for Entrex-AMLDC Board -> Diode_THT:D_DO-41_SOD81_P12.70mm_Horizontal
- R1: value R_US -> ~; footprint Forgotten Machines:Resistor for Entrex-AMLDC Board -> Resistor_THT:R_Axial_DIN0411_L9.9mm_D3.6mm_P12.70mm_Horizontal
- R2, R4: value R_US -> ~
- UB3: footprint (none) -> Package_DIP:DIP-14_W7.62mm
- renumbered U1 to UF3
Connections:
- net B2p3 is gone; now on net B2p13: UB2.3
- net B2p9 is gone; now on net B2p13: UB2.9
- net B3p11 is gone; now on net B3p10: UB3.11
- net B3p12 is gone; now on net B3p8: UB3.12
- net B3p13 is gone; now on net B3p8: UB3.13
- net B3p3 is gone; now on net B3p6: UB3.3
- net B3p5 is gone; now on net B3p6: UB3.5
- net B3p9 is gone; now on net B3p8: UB3.9
- net B4p5 is gone; now on net B4p1: UB4.5 (Q)
- net B4p9 is gone; now on net GND: UB4.9 (A)
- net C2p9 is gone; now on net C2p13: UC2.9 (A)
- net C3p11 is gone; now on net GND: UC3.11 (C)
- net C3p2 is gone; now on net C3p9: UC3.2 (D)
- net C4p2 is gone; now on net C4p13: UC4.2
- net C4p9 is gone; now on net B4p1: UC4.9
- net D0p13 is gone; now on net D0p9: UD0.13
- net D0p5 is gone; now on net D0p9: UD0.5
- net D1p12 is gone; now on net B1p13: UD1.12
- net D1p4 is gone; now on net B1p3: UD1.4
- net D1p5 is gone; now on net D1p9: UD1.5
- net D1p8 is gone; now on net B1p12: UD1.8
- net D2p13 is gone; now on net B2p13: UD2.13
- net D3p4 is gone; now on net D3p10: UD3.4 (~{Q})
- net D3p9 is gone; now on net GND: UD3.9 (A)
- net D4p11 is gone; now on net C4p5: UD4.11 (C)
- net D4p2 is gone; now on net C4p3: UD4.2 (D)
- net D4p9 is gone; now on net B4p10: UD4.9 (Q)
- net E0p13 is gone; now on net D0p9: UE0.13
- net E0p9 is gone; now on net D0p9: UE0.9
- net E1p2 is gone; now on net D1p3: UE1.2 (D)
- net E1p3 is gone; now on net B1p3: UE1.3 (C)
- net E1p5 is gone; now on net D1p9: UE1.5 (Q)
- net E3p12 is gone; now on net C3p5: UE3.12 (D)
- net F0p9 is gone; now on net E0p6: UF0.9
- net F1p4 is gone; now on net D1p3: UF1.4
- net F2p12 is gone; now on net F2p3: UF2.12
- net F3p11 is gone; now on net G3p11: UF3.11 (D0)
- net F3p13 is gone; now on net GND: UF3.13 (S)
- net F3p14 is gone; now on net J3p3: UF3.14 (Q7)
- net F3p3 is gone; now on net G3p12: UF3.3 (Q7)
- net F3p4 is gone; now on net GND: UF3.4 (S)
- net F3p6 is gone; now on net G3p8: UF3.6 (D1)
- net F3p7 is gone; now on net F3p10: UF3.7
- net F3p9 is gone; now on net GND: UF3.9
- net F4p2 is gone; now on net F4p12: UF4.2 (D)
- net G0p11 is gone; now on net F0p4: UG0.11
- net G0p12 is gone; now on net F0p2: UG0.12
- net G0p3 is gone; now on net F0p2: UG0.3
- net G1p10 is gone; now on net F1p2: UG1.10
- net G1p12 is gone; now on net F1p2: UG1.12
- net G1p13 is gone; now on net G1p2: UG1.13
- net G1p4 is gone; now on net D1p9: UG1.4
- net G1p5 is gone; now on net F1p6: UG1.5
- net G1p9 is gone; now on net E1p8: UG1.9
- net G2p11 is gone; now on net D2p5: UG2.11
- net G2p3 is gone; now on net G2p2: UG2.3
- net G2p5 is gone; now on net G2p2: UG2.5
- net G3p1 is gone; now on net J3p3: UG3.1
- net G3p13 is gone; now on net J3p3: UG3.13
- net G3p3 is gone; now on net E3p2: UG3.3
- net H1p2 is gone; now on net H1p10: UH1.2
- net H1p4 is gone; now on net H1p11: UH1.4
- net H2p3 is gone; now on net H2p12: UH2.3
- net H2p5 is gone; now on net H2p12: UH2.5
- net H2p8 is gone; now on net G2p6: UH2.8
- net H3p13 is gone; now on net G3p2: UH3.13
- net H3p6 is gone; now on net H3p9: UH3.6
- net H3p8 is gone; now on net G3p9: UH3.8
- net H4p9 is gone; now on net GND: UH4.9 (A)
- net J0p1 is gone; now on net H0p2: UJ0.1
- net J1p8 is gone; now on net H1p5: UJ1.8 (~{Q})
- net J2p1 is gone; now on net G2p1: UJ2.1 (~{R})
- net J2p5 is gone; now on net J2p12: UJ2.5 (Q)
- net J3p13 is gone; now on net H3p12: UJ3.13
- net K1p1 is gone; now on net J1p1: UK1.1 (~{R})
- net K1p2 is gone; now on net K1p9: UK1.2 (D)
- net K2p12 is gone; now on net J2p4: UK2.12
- net K2p13 is gone; now on net G2p1: UK2.13
- net K2p8 is gone; now on net G2p2: UK2.8
- net L0p2 is gone; now on net L0p13: UL0.2
- net L0p5 is gone; now on net L0p10: UL0.5
- net L1p13 is gone; now on net J1p13: UL1.13 (Mr)
- net L1p14 is gone; now on net +5V: UL1.14 (VCC)
- net L1p7 is gone; now on net GND: UL1.7 (GND)
- net L2p12 is gone; now on net K2p11: UL2.12
- net L3p2 is gone; now on net L3p13: UL3.2
- net L3p5 is gone; now on net L3p10: UL3.5
- net L4p14 is gone; now on net +5V: UL4.14 (VCC)
- net L4p7 is gone; now on net GND: UL4.7 (GND)
- net M0p11 is gone; now on net L0p11: UM0.11
- net M0p2 is gone; now on net M0p13: UM0.2
- net M0p3 is gone; now on net L0p3: UM0.3
- net M0p5 is gone; now on net M0p10: UM0.5
- net M0p6 is gone; now on net L0p6: UM0.6
- net M0p8 is gone; now on net L0p8: UM0.8
- net M1p10 is gone; now on net L1p10: UM1.10 (P1)
- net M1p11 is gone; now on net L1p4: UM1.11 (P3)
- net M1p13 is gone; now on net J1p13: UM1.13 (Mr)
- net M1p14 is gone; now on net +5V: UM1.14 (VCC)
- net M1p3 is gone; now on net L1p3: UM1.3 (P2)
- net M1p4 is gone; now on net N1p7: UM1.4 (P0)
- net M1p7 is gone; now on net GND: UM1.7 (GND)
- net M2p1 is gone; now on net L2p3: UM2.1 (~{PL})
- net M2p15 is gone; now on net GND: UM2.15 (~{CE})
- net M2p16 is gone; now on net +5V: UM2.16 (VCC)
- net M2p8 is gone; now on net GND: UM2.8 (GND)
- net M3p11 is gone; now on net L3p11: UM3.11
- net M3p2 is gone; now on net M3p13: UM3.2
- net M3p3 is gone; now on net L3p3: UM3.3
- net M3p5 is gone; now on net M3p10: UM3.5
- net M3p6 is gone; now on net L3p6: UM3.6
- net M3p8 is gone; now on net L3p8: UM3.8
- net M4p10 is gone; now on net L4p10: UM4.10 (P1)
- net M4p11 is gone; now on net L4p11: UM4.11 (P3)
- net M4p13 is gone; now on net L4p13: UM4.13 (Mr)
- net M4p14 is gone; now on net +5V: UM4.14 (VCC)
- net M4p3 is gone; now on net L4p3: UM4.3 (P2)
- net M4p4 is gone; now on net L4p4: UM4.4 (P0)
- net M4p7 is gone; now on net GND: UM4.7 (GND)
- net N0p11 is gone; now on net L0p11: UN0.11
- net N0p13 is gone; now on net L0p3: UN0.13
- net N0p5 is gone; now on net L0p6: UN0.5
- net N0p9 is gone; now on net L0p8: UN0.9
- net N1p13 is gone; now on net N1p4: UN1.13 (E01)
- net N1p2 is gone; now on net L1p3: UN1.2 (D0)
- net N1p3 is gone; now on net L1p11: UN1.3 (D1)
- net N1p5 is gone; now on net +5V: UN1.5 (VCC)
- net N1p6 is gone; now on net L1p10: UN1.6 (D2)
- net N2p12 is gone; now on net GND: UN2.12 (GND)
- net N2p4 is gone; now on net N2p13: UN2.4 (E23)
- net N3p11 is gone; now on net L3p11: UN3.11
- net N3p13 is gone; now on net L3p3: UN3.13
- net N3p5 is gone; now on net L3p6: UN3.5
- net N3p9 is gone; now on net L3p8: UN3.9
- net N4p2 is gone; now on net L4p3: UN4.2 (D0)
- net N4p3 is gone; now on net L4p11: UN4.3 (D1)
- net N4p4 is gone; now on net N4p13: UN4.4 (E23)
- net N4p6 is gone; now on net L4p10: UN4.6 (D2)
- net N4p7 is gone; now on net L4p4: UN4.7 (D3)
- net P0p10 is gone; now on net N0p4: UP0.10
- net P0p11 is gone; now on net L0p11: UP0.11
- net P0p2 is gone; now on net P0p13: UP0.2
- net P0p3 is gone; now on net L0p3: UP0.3
- net P0p5 is gone; now on net N0p4: UP0.5
- net P0p6 is gone; now on net L0p6: UP0.6
- net P0p8 is gone; now on net L0p8: UP0.8
- net P1p1 is gone; now on net P1p13: UP1.1
- net P1p2 is gone; now on net P1p12: UP1.2
- net P1p4 is gone; now on net P1p12: UP1.4
- net P3p11 is gone; now on net L3p11: UP3.11
- net P3p2 is gone; now on net P3p13: UP3.2
- net P3p3 is gone; now on net L3p3: UP3.3
- net P3p5 is gone; now on net P3p10: UP3.5
- net P3p6 is gone; now on net L3p6: UP3.6
- net P3p8 is gone; now on net L3p8: UP3.8
- net R0p10 is gone; now on net R0p13: UR0.10
- net R0p11 is gone; now on net L0p11: UR0.11
- net R0p2 is gone; now on net R0p13: UR0.2
- net R0p3 is gone; now on net L0p3: UR0.3
- net R0p5 is gone; now on net R0p13: UR0.5
- net R0p6 is gone; now on net L0p6: UR0.6
- net R0p8 is gone; now on net L0p8: UR0.8
- net R1p12 is gone; now on net GND: UR1.12 (GND)
- net R1p13 is gone; now on net R1p4: UR1.13 (E01)
- net R2p10 is gone; now on net P2p5: UR2.10 (Q2)
- net R2p2 is gone; now on net N2p16: UR2.2 (D0)
- net R2p3 is gone; now on net N2p15: UR2.3 (D1)
- net R2p5 is gone; now on net +5V: UR2.5 (VCC)
- net R2p6 is gone; now on net N2p10: UR2.6 (D2)
- net R2p7 is gone; now on net N2p9: UR2.7 (D3)
- net R3p11 is gone; now on net L3p11: UR3.11
- net R3p2 is gone; now on net R3p13: UR3.2
- net R3p3 is gone; now on net L3p3: UR3.3
- net R3p5 is gone; now on net R3p10: UR3.5
- net R3p6 is gone; now on net L3p6: UR3.6
- net R3p8 is gone; now on net L3p8: UR3.8
- net R4p12 is gone; now on net GND: UR4.12 (GND)
- net R4p4 is gone; now on net R4p13: UR4.4 (E23)
- net S0p10 is gone; now on net R0p13: US0.10
- net S0p13 is gone; now on net R0p13: US0.13
- net S0p2 is gone; now on net R0p13: US0.2
- net S0p5 is gone; now on net R0p13: US0.5
- net S1p12 is gone; now on net GND: US1.12 (GND)
- net S1p13 is gone; now on net R1p4: US1.13 (E01)
- net S1p4 is gone; now on net R1p4: US1.4 (E23)
- net S1p5 is gone; now on net R1p5: US1.5 (VCC)
- net S3p10 is gone; now on net R3p10: US3.10
- net S3p13 is gone; now on net R3p13: US3.13
- net S3p2 is gone; now on net R3p13: US3.2
- net S3p5 is gone; now on net R3p10: US3.5
- net S4p12 is gone; now on net GND: US4.12 (GND)
- net S4p13 is gone; now on net R4p13: US4.13 (E01)
- net S4p4 is gone; now on net R4p13: US4.4 (E23)
- net +5V: now also C26.1, C46.1, C55.1, C65.1, C66.2, C67.1, C68.2, C70.1, R1.1, R12.2, R13.1, R18.2, R2.1, R27.2, R29.2, R30.2, R32.2, R37.2, R47.1, R50.1, R54.1, R55.2, R68.1, R73.1, R85.2, R87.2, R88.2, R93.1, R93.2, UB1.14 (VCC), UB2.14 (VCC), UB3.14 (VCC), UB4.16 (VCC), UC1.14 (VCC), UC2.16 (VCC), UC3.14 (VCC), UC4.14 (VCC), UD0.14 (VCC), UD1.14 (VCC), UD2.14 (VCC), UD3.16 (VCC), UD4.14 (VCC), UE0.14 (VCC), UE1.14 (VCC), UE2.14 (VCC), UE3.14 (VCC), UE4.14 (VCC), UF1.14 (VCC), UF2.14 (VCC), UF3.16 (VCC), UF4.14 (VCC), UG0.14 (VCC), UG1.14 (VCC), UG2.14 (VCC), UG3.14 (VCC), UG4.16 (VCC), UH0.14 (VCC), UH1.14 (VCC), UH2.14 (VCC), UH3.14 (VCC), UH4.16 (VCC), UJ0.14 (VCC), UJ1.14 (VCC), UJ2.14 (VCC), UJ3.14 (VCC), UK0.14 (VCC), UK1.14 (VCC), UK2.14 (VCC), UL0.14 (VCC), UL2.14 (VCC), UL3.14 (VCC), UM0.14 (VCC), UM3.14 (VCC), UN0.14 (VCC), UN3.14 (VCC), UP0.14 (VCC), UP1.14 (VCC), UP3.14 (VCC), UP4.16 (VCC), UR0.14 (VCC), UR3.14 (VCC), US0.14 (VCC), US2.14 (VDD), US3.14 (VCC)
- net B1p10: now also R77.1
- net B1p2: now also C45.2, R38.2
- net B1p9: now also C16.1, R77.2
- net B2p10: now also C30.1, R91.2
- net B2p11: now also R91.1
- net B2p4: now also R70.1
- net B2p5: now also C13.1, R70.2
- net B4p14: now also C41.2
- net B4p15: now also C41.1
- net B4p6: now also C42.1
- net B4p7: now also C42.2
- net C0p5: now also R19.1
- net C0p9: now also CR1.1 (K), R49.1
- net C2p14: now also C29.2
- net C2p6: now also C15.2
- net D0p3: now also R71.2
- net D2p2: now also C44.1
- net D3p14: now also C25.2
- net D3p15: now also C25.1
- net D3p6: now also C27.1
- net D3p7: now also C27.2
- net DISK2: now also R16.2
- net DSK ~{RST}: now also R17.1
- net E0p11: now also R51.2
- net E0p3: now also R53.2
- net E4p4: now also UF4.13 (~{R})
- net E4p6: now also UG4.5 (Q)
- net F4p11: now also UG4.4 (~{Q})
- net F4p3: now also UG4.12 (~{Q}), UG4.2 (B)
- net G0p2: now also JP6.1 (A)
- net G0p5: now also JP3.1 (A)
- net G0p6: now also JP2.1 (A)
- net GND: now also C13.2, C16.2, C26.2, C30.2, C31.1, C43.2, C45.1, C62.2, C64.2, C65.2, C66.1, C67.2, C68.1, C71.2, C72.2, CR1.2 (A), CR3.2 (A), R19.2, R49.2, R7.2, R72.2, UB1.7 (GND), UB2.7 (GND), UB3.7 (GND), UB4.8 (GND), UC0.7 (GND), UC1.7 (GND), UC2.8 (GND), UC3.7 (GND), UC4.7 (GND), UD0.7 (GND), UD1.7 (GND), UD2.7 (GND), UD3.8 (GND), UD4.7 (GND), UE0.7 (GND), UE1.7 (GND), UE2.7 (GND), UE3.7 (GND), UE4.7 (GND), UF0.7 (GND), UF1.7 (GND), UF2.7 (GND), UF3.8 (GND), UF4.7 (GND), UG0.7 (GND), UG1.7 (GND), UG2.7 (GND), UG3.7 (GND), UG4.8 (GND), UG4.9 (A), UH0.7 (GND), UH1.7 (GND), UH2.7 (GND), UH3.7 (GND), UH4.8 (GND), UJ0.7 (GND), UJ1.7 (GND), UJ2.7 (GND), UJ3.7 (GND), UK0.7 (GND), UK1.7 (GND), UK2.7 (GND), UL0.7 (GND), UL2.7 (GND), UL3.7 (GND), UM0.7 (GND), UM3.7 (GND), UN0.7 (GND), UN3.7 (GND), UP0.7 (GND), UP1.7 (GND), UP3.7 (GND), UP4.8 (GND), UR0.7 (GND), UR3.7 (GND), US0.7 (GND), US2.7 (VSS), US3.7 (GND)
- net H0p10: now also JP3.2 (B)
- net H0p11: now also JP4.2 (B)
- net H0p12: now also JP5.2 (B)
- net H0p13: now also JP6.2 (B)
- net H0p8: now also JP1.2 (B)
- net H0p9: now also JP2.2 (B)
- net H4p12: now also UG4.10 (B)
- net H4p14: now also C56.2
- net H4p15: now also C56.1
- net H4p6: now also C11.1
- net H4p7: now also C11.2, R67.1
- net J0p10: now also UJ0.13
- net K0p1: now also C57.1
- net K0p10: now also C72.1
- net K0p5: now also C64.1
- net L1p4: no longer UL1.4 (P0)
- net L4p10: now also UP4.10 (A2)
- net L4p3: now also UP4.15 (A3)
- net L4p4: now also UP4.6 (A1)
- net N1p7: now also UL1.4 (P0)
- net N2p5: now also C69.1, UP2.14 (VCC)
- net N4p12: now also C55.2, UP4.11 (B2), UP4.14 (D3), UP4.2 (B0), UP4.5 (B1)
- net SPARE: now also R56.1
- net R9p2: now reaches C43.1
- net R9p2: now also R9.2
- net C14p2: now reaches R29.1
- net C14p2: now also C14.2
- net R10p2: now reaches R10.2
- net Pad15p15: now reaches C12.1
- net Pad15p15: now also UG4.15 (RCext)
- net Pad14p14: now reaches C12.2
- net Pad14p14: now also UG4.14 (Cext)
- net C60p1: now reaches R53.1
- net C60p1: now also C60.1
- net R34P1: now reaches R16.1
- net R34P1: now also R15.1, R34.1, R35.1
- net B49: now reaches J2.49 (Pin_49)
- net Pad6p6: now reaches UG4.6 (Cext)
- net Net-(UG4A-Q): now reaches UG4.13 (Q)
- net Net-(UG4A-Q): no longer UG4.7 (RCext)
- net C59p1: now reaches C59.1
- net C59p1: now also R51.1
- net C58p2: now reaches C59.2
- net C58p2: now also C58.2, C60.2, C61.2
- net C58p1: now reaches R71.1
- net C58p1: now also C58.1
- net R50P2: now reaches CR3.1 (K)
- net R50P2: now also C28.2
- net R56P2: now reaches R56.2
- net R56P2: now also R17.2, R36.2, R92.2
- net R13p2: now reaches R13.2
- net R13p2: now also C15.1
- net A77: now reaches R36.1
- net A77: now also J1.77 (Pin_77)
- net C61p1: now reaches R33.1
- net C61p1: now also C61.1
- net C31p2: now reaches R94.2
- net C31p2: now also C31.2
- net unconnected-(UV4-D-Pad14): now reaches UV4.14 (D)
- net Pad77: now reaches R35.2
- new net UG4A: UG4.7 (RCext)
Other:
- moved on the sheet: C47, UG4A

Commit message: ready for AMLDC Front Board Tracing part 2
Parts:
- removed UL5: 74LS21, Package_DIP:DIP-14_W7.62mm, symbol 74xx:74LS21
- added UL5: 9321, Package_DIP:DIP-16_W7.62mm, symbol ForgottenMachines:9321
- UR5: footprint Package_DIP:DIP-16_W7.62mm -> Package_DIP:DIP-14_W7.62mm
Connections:
- net B8p11 is gone; now on net C8p10: UB8.11 (Q3)
- net +5V: now also C39.2
- net GND: now also C39.1, C8.1, R25.2
- net L5p1: now also UL5.1 (E)
- net L5p10: now also UL5.10 (02)
- net L5p12: now also UL5.12 (00)
- net L5p13: now also UL5.13 (A0)
- net L5p2: now also UL5.2 (A0)
- net L5p4: now also UL5.4 (00)
- net L5p5: now also UL5.5 (01)
- net L5p6: now also UL5.6 (02)
- net L5p9: now also UL5.9 (03)
- net Q1p1: now reaches Q1.1 (C)
- net Q1p1: now also Q1.2 (B)
- net Q1p3: now reaches Q1.3 (E)
- net unconnected-(UV4-GND-Pad7): now reaches UV4.7 (Qb)
- new net L5p11: UL5.11 (01)
- new net L5p14: UL5.14 (A0)
- new net L5p15: UL5.15 (E)
- new net L5p3: UL5.3 (A0)
- new net L5p7: UL5.7 (03)
Other:
- note added: "Rework Wire Here"

Commit message: Trace Part 3
Parts:
- UU4, UV4: footprint Package_DIP:DIP-16_W7.62mm -> Package_DIP:DIP-14_W7.62mm
Connections:
- net unconnected-(UV4-D-Pad14) is gone; now on net V4p14: UV4.14 (D)
- net unconnected-(UV4-GND-Pad7) is gone; now on net V4p7: UV4.7 (Qb)
- net V4p1: now also UV4.1 (Mr)
- net V4p10: now also UV4.10 (Ld)
- net V4p11: now also UV4.11 (Qd)
- net V4p12: now also UV4.12 (~{Qd})
- net V4p13: now also UV4.13 (Sh)
- net V4p15: now also UV4.15 (C)
- net V4p2: now also UV4.2 (B)
- net V4p3: now also UV4.3 (A)
- net V4p4: now also UV4.4 (Ds)
- net V4p5: now also UV4.5 (Qa)
- net V4p6: now also UV4.6 (CLK)
- net V4p9: now also UV4.9 (Qc)
Other:
- moved on the sheet: UV4
Changed lines of the file:
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@@
     (effects (font (size 1.27 1.27)) (justify right bottom))
   )
-  (label "GND" (at 553.085 1157.605 180)
+  (label "GND" (at 553.085 1157.605 180) (fields_autoplaced)
     (effects (font (size 1.27 1.27)) (justify right bottom))
   )
@@
     (effects (font (size 1.27 1.27)) (justify right bottom))
   )
-  (label "GND" (at 218.44 162.56 180)
+  (label "GND" (at 218.44 162.56 180) (fields_autoplaced)
     (effects (font (size 1.27 1.27)) (justify right bottom))
   )
@@
     (effects (font (size 1.27 1.27)) (justify right bottom))
   )
-  (label "GND" (at 201.93 236.22 0)
+  (label "GND" (at 201.93 236.22 0) (fields_autoplaced)
     (effects (font (size 1.27 1.27)) (justify left bottom))
   )
@@
     (effects (font (size 1.27 1.27)) (justify right bottom))
   )
-  (label "unconnected-(UV4-D-Pad14)" (at 657.225 1207.135 180) (fields_autoplaced)
-    (effects (font (size 1.27 1.27)) (justify right bottom))
-  )
   (label "Net-(UG4A-Q)" (at 757.555 372.11 0) (fields_autoplaced)
     (effects (font (size 1.27 1.27)) (justify left bottom))
@@
     (effects (font (size 1.27 1.27)) (justify right bottom))
   )
-  (label "unconnected-(UV4-GND-Pad7)" (at 672.465 1186.815 90)
-    (effects (font (size 1.27 1.27)) (justify left bottom))
-  )
   (label "+5V" (at -127 207.01 90) (fields_autoplaced)
     (effects (font (size 1.27 1.27)) (justify left bottom))
@@
     (effects (font (size 1.27 1.27)) (justify right bottom))
   )
-  (label "+5V" (at 565.785 1157.605 0)
+  (label "+5V" (at 565.785 1157.605 0) (fields_autoplaced)
     (effects (font (size 1.27 1.27)) (justify left bottom))
   )
@@
     )
   )
-  (global_label "V4p4" (shape input) (at 703.58 1228.09 270) (fields_autoplaced)
+  (global_label "V4p4" (shape input) (at 703.58 1226.82 270) (fields_autoplaced)
     (effects (font (size 1.27 1.27)) (justify right))
-    (property "Intersheetrefs" "${INTERSHEET_REFS}" (at 703.58 1235.7318 90)
+    (property "Intersheetrefs" "${INTERSHEET_REFS}" (at 703.58 1234.4618 90)
       (effects (font (size 1.27 1.27)) (justify right) hide)
     )
@@
     )
   )
-  (global_label "V4p14" (shape input) (at 656.59 1206.5 180) (fields_autoplaced)
+  (global_label "V4p14" (shape input) (at 657.86 1206.5 180) (fields_autoplaced)
     (effects (font (size 1.27 1.27)) (justify right))
-    (property "Intersheetrefs" "${INTERSHEET_REFS}" (at 647.7387 1206.5 0)
+    (property "Intersheetrefs" "${INTERSHEET_REFS}" (at 649.0087 1206.5 0)
       (effects (font (size 1.27 1.27)) (justify right) hide)
     )
@@
     )
   )
-  (global_label "V4p13" (shape input) (at 709.93 1228.09 270) (fields_autoplaced)
+  (global_label "V4p13" (shape input) (at 709.93 1226.82 270) (fields_autoplaced)
     (effects (font (size 1.27 1.27)) (justify right))
-    (property "Intersheetrefs" "${INTERSHEET_REFS}" (at 709.93 1236.9413 90)
+    (property "Intersheetrefs" "${INTERSHEET_REFS}" (at 709.93 1235.6713 90)
       (effects (font (size 1.27 1.27)) (justify right) hide)
     )
@@
     )
   )
-  (global_label "V4p3" (shape input) (at 668.02 1228.09 270) (fields_autoplaced)
+  (global_label "V4p3" (shape input) (at 668.02 1226.82 270) (fields_autoplaced)
     (effects (font (size 1.27 1.27)) (justify right))
-    (property "Intersheetrefs" "${INTERSHEET_REFS}" (at 668.02 1235.7318 90)
+    (property "Intersheetrefs" "${INTERSHEET_REFS}" (at 668.02 1234.4618 90)
       (effects (font (size 1.27 1.27)) (justify right) hide)
     )
@@
     )
   )
-  (global_label "V4p7" (shape input) (at 723.9 1207.77 0) (fields_autoplaced)
+  (global_label "V4p7" (shape input) (at 723.9 1206.5 0) (fields_autoplaced)
     (effects (font (size 1.27 1.27)) (justify left))
-    (property "Intersheetrefs" "${INTERSHEET_REFS}" (at 731.5418 1207.77 0)
+    (property "Intersheetrefs" "${INTERSHEET_REFS}" (at 731.5418 1206.5 0)
       (effects (font (size 1.27 1.27)) (justify left) hide)
     )
@@
     )
   )
-  (global_label "V4p1" (shape input) (at 697.23 1228.09 270) (fields_autoplaced)
+  (global_label "V4p1" (shape input) (at 697.23 1226.82 270) (fields_autoplaced)
     (effects (font (size 1.27 1.27)) (justify right))
-    (property "Intersheetrefs" "${INTERSHEET_REFS}" (at 697.23 1235.7318 90)
+    (property "Intersheetrefs" "${INTERSHEET_REFS}" (at 697.23 1234.4618 90)
       (effects (font (size 1.27 1.27)) (justify right) hide)
     )
@@
     )
   )
-  (global_label "V4p14" (shape input) (at 683.26 1228.09 270) (fields_autoplaced)
+  (global_label "V4p14" (shape input) (at 683.26 1226.82 270) (fields_autoplaced)
     (effects (font (size 1.27 1.27)) (justify right))
-    (property "Intersheetrefs" "${INTERSHEET_REFS}" (at 683.26 1236.9413 90)
+    (property "Intersheetrefs" "${INTERSHEET_REFS}" (at 683.26 1235.6713 90)
       (effects (font (size 1.27 1.27)) (justify right) hide)
     )
@@
     )
   )
-  (global_label "V4p10" (shape input) (at 716.28 1228.09 270) (fields_autoplaced)
+  (global_label "V4p10" (shape input) (at 716.28 1226.82 270) (fields_autoplaced)
     (effects (font (size 1.27 1.27)) (justify right))
-    (property "Intersheetrefs" "${INTERSHEET_REFS}" (at 716.28 1236.9413 90)
+    (property "Intersheetrefs" "${INTERSHEET_REFS}" (at 716.28 1235.6713 90)
       (effects (font (size 1.27 1.27)) (justify right) hide)
     )
@@
     )
   )
-  (global_label "V4p2" (shape input) (at 673.1 1228.09 270) (fields_autoplaced)
+  (global_label "V4p2" (shape input) (at 673.1 1226.82 270) (fields_autoplaced)
     (effects (font (size 1.27 1.27)) (justify right))
-    (property "Intersheetrefs" "${INTERSHEET_REFS}" (at 673.1 1235.7318 90)
+    (property "Intersheetrefs" "${INTERSHEET_REFS}" (at 673.1 1234.4618 90)
       (effects (font (size 1.27 1.27)) (justify right) hide)
     )
@@
     )
   )
-  (global_label "V4p11" (shape input) (at 683.26 1187.45 90) (fields_autoplaced)
+  (global_label "V4p11" (shape input) (at 683.26 1186.18 90) (fields_autoplaced)
     (effects (font (size 1.27 1.27)) (justify left))
-    (property "Intersheetrefs" "${INTERSHEET_REFS}" (at 683.26 1178.5987 90)
+    (property "Intersheetrefs" "${INTERSHEET_REFS}" (at 683.26 1177.3287 90)
       (effects (font (size 1.27 1.27)) (justify left) hide)
     )
@@
     )
   )
-  (global_label "V4p6" (shape input) (at 690.88 1228.09 270) (fields_autoplaced)
+  (global_label "V4p6" (shape input) (at 690.88 1226.82 270) (fields_autoplaced)
     (effects (font (size 1.27 1.27)) (justify right))
-    (property "Intersheetrefs" "${INTERSHEET_REFS}" (at 690.88 1235.7318 90)
+    (property "Intersheetrefs" "${INTERSHEET_REFS}" (at 690.88 1234.4618 90)
       (effects (font (size 1.27 1.27)) (justify right) hide)
     )
@@
       (effects (font (size 1.27 1.27)))
     )
-    (property "Footprint" "Package_DIP:DIP-16_W7.62mm" (at 699.77 1115.06 0)
+    (property "Footprint" "Package_DIP:DIP-14_W7.62mm" (at 699.77 1115.06 0)
       (effects (font (size 1.27 1.27)) hide)
     )
@@
     )
   )
-  (symbol (lib_id "ForgottenMachines:74179") (at 690.245 1207.135 90) (unit 1)
+  (symbol (lib_id "ForgottenMachines:74179") (at 690.88 1206.5 90) (unit 1)
     (in_bom yes) (on_board yes) (dnp no)
-    (property "Reference" "UV4" (at 701.04 1202.055 90)
+    (property "Reference" "UV4" (at 701.675 1201.42 90)
       (effects (font (size 1.27 1.27)))
     )
-    (property "Value" "74179\n or\n8271" (at 692.15 1208.405 90)
+    (property "Value" "74179\n or\n8271" (at 692.785 1207.77 90)
       (effects (font (size 1.27 1.27)))
     )
-    (property "Footprint" "Package_DIP:DIP-16_W7.62mm" (at 706.755 1170.305 0)
+    (property "Footprint" "Package_DIP:DIP-14_W7.62mm" (at 707.39 1169.67 0)
       (effects (font (size 1.27 1.27)) hide)
     )
-    (property "Datasheet" "" (at 685.165 1207.135 0)
+    (property "Datasheet" "" (at 685.8 1206.5 0)
       (effects (font (size 1.27 1.27)) hide)
     )
