File: Mystery Test Board/AMLDC-2044B.kicad_sch (KiCad schematic)
At the start: 331 parts, among them J1 Port A, J2 Port B, Q1 PNP MPS6533, Y1 Crystal

Commit message: Ready for Top p4
Parts:
- removed UU5: 74LS21, Package_DIP:DIP-14_W7.62mm, symbol 74xx:74LS21
- removed UV4: 74179 or 8271, Package_DIP:DIP-14_W7.62mm, symbol ForgottenMachines:74179
- added SW1: ~{RESET} RESET, Button_Switch_THT:SW_Lever_1P2T_NKK_GW12LxH, symbol Switch:SW_SPDT
- added UU5: 9321, Package_DIP:DIP-16_W7.62mm, symbol ForgottenMachines:9321
- added UV4: 74LS197, Package_DIP:DIP-14_W7.62mm, symbol 74xx:74LS197
Connections:
- net B5p5 is gone; now on net B5p10: UB5.5
- net B6p2 is gone; now on net B6p11: UB6.2
- net B8p1 is gone; now on net B8p12: UB8.1 (CP1..3)
- net B8p10 is gone; now on net GND: UB8.10 (GND)
- net B8p5 is gone; now on net +5V: UB8.5 (VCC)
- net C5p13 is gone; now on net B5p2: UC5.13
- net C7p3 is gone; now on net C7p12: UC7.3 (C)
- net D5p1 is gone; now on net B5p1: UD5.1 (A)
- net D5p10 is gone; now on net C5p4: UD5.10 (B)
- net D5p2 is gone; now on net C5p4: UD5.2 (B)
- net D5p5 is gone; now on net C5p3: UD5.5 (Q)
- net D7p2 is gone; now on net C7p5: UD7.2 (D)
- net D7p3 is gone; now on net C7p11: UD7.3 (C)
- net D8p11 is gone; now on net C8p8: UD8.11 (C)
- net D8p2 is gone; now on net D8p9: UD8.2 (D)
- net D8p5 is gone; now on net C8p5: UD8.5 (Q)
- net E6p5 is gone; now on net E6p11: UE6.5
- net E7p14 is gone; now on net +5V: UE7.14 (VCC)
- net E7p7 is gone; now on net GND: UE7.7 (GND)
- net E7p8 is gone; now on net D7p10: UE7.8
- net E7p9 is gone; now on net D7p5: UE7.9
- net F5p1 is gone; now on net F5p13: UF5.1 (~{R})
- net F5p12 is gone; now on net E5p10: UF5.12 (D)
- net F5p2 is gone; now on net E5p9: UF5.2 (D)
- net F5p3 is gone; now on net F5p11: UF5.3 (C)
- net F5p5 is gone; now on net E5p10: UF5.5 (Q)
- net F5p6 is gone; now on net E5p4: UF5.6 (~{Q})
- net F5p8 is gone; now on net E5p9: UF5.8 (~{Q})
- net F6p13 is gone; now on net E6p13: UF6.13
- net F6p2 is gone; now on net E6p2: UF6.2
- net F6p5 is gone; now on net F6p11: UF6.5
- net F8p12 is gone; now on net E8p4: UF8.12
- net F8p9 is gone; now on net E8p5: UF8.9
- net G7p2 is gone; now on net F7p3: UG7.2
- net H5p13 is gone; now on net E5p11: UH5.13 (~{R})
- net H5p9 is gone; now on net F5p13: UH5.9 (Q)
- net H6p1 is gone; now on net G6p1: UH6.1
- net H6p12 is gone; now on net G6p3: UH6.12
- net H6p2 is gone; now on net G6p2: UH6.2
- net H6p9 is gone; now on net G6p6: UH6.9
- net H7p2 is gone; now on net F7p2: UH7.2 (D)
- net H7p5 is gone; now on net H7p12: UH7.5 (Q)
- net H7p8 is gone; now on net F7p3: UH7.8 (~{Q})
- net J6p11 is gone; now on net G6p2: UJ6.11
- net J7p12 is gone; now on net H7p3: UJ7.12 (~{Q})
- net K6p9 is gone; now on net GND: UK6.9 (A)
- net K7p3 is gone; now on net L7p12: UK7.3
- net K7p4 is gone; now on net K7p13: UK7.4
- net K8p3 is gone; now on net GND: UK8.3
- net L5p4 is gone; now on net K5p1: UL5.4 (00)
- net L5p5 is gone; now on net K5p13: UL5.5 (01)
- net L5p6 is gone; now on net K5p3: UL5.6 (02)
- net L5p7 is gone; now on net K5p5: UL5.7 (03)
- net L6p2 is gone; now on net L6p12: UL6.2
- net L6p5 is gone; now on net L6p12: UL6.5
- net L6p9 is gone; now on net L6p12: UL6.9
- net L7p3 is gone; now on net M7p3: UL7.3 (C)
- net L7p8 is gone; now on net K7p9: UL7.8 (~{Q})
- net M7p1 is gone; now on net L7p1: UM7.1 (~{R})
- net M7p11 is gone; now on net M7p3: UM7.11 (C)
- net M7p13 is gone; now on net L7p1: UM7.13 (~{R})
- net M8p12 is gone; now on net K8p1: UM8.12 (K)
- net M8p6 is gone; now on net K8p4: UM8.6 (C)
- net M8p9 is gone; now on net K8p1: UM8.9 (J)
- net N5p16 is gone; now on net +5V: UN5.16 (VCC)
- net N5p8 is gone; now on net GND: UN5.8 (GND)
- net N5p9 is gone; now on net M5p5: UN5.9 (Q7)
- net N6p13 is gone; now on net M6p8: UN6.13
- net N6p2 is gone; now on net N6p10: UN6.2
- net N7p10 is gone; now on net M7p6: UN7.10
- net N7p9 is gone; now on net M7p8: UN7.9
- net P6p2 is gone; now on net GND: UP6.2 (D)
- net P6p5 is gone; now on net P6p12: UP6.5 (Q)
- net P7p1 is gone; now on net P7p12: UP7.1 (CP1..3)
- net P7p10 is gone; now on net GND: UP7.10 (GND)
- net R5p14 is gone; now on net +5V: UR5.14 (VDD)
- net R5p7 is gone; now on net GND: UR5.7 (VSS)
- net R5p8 is gone; now on net N5p2: UR5.8 (CK)
- net R6p1 is gone; now on net P6p1: UR6.1 (~{R})
- net R6p2 is gone; now on net GND: UR6.2 (D)
- net R6p5 is gone; now on net R6p12: UR6.5 (Q)
- net R7p1 is gone; now on net R7p12: UR7.1 (CP1..3)
- net R7p10 is gone; now on net GND: UR7.10 (GND)
- net R7p14 is gone; now on net P7p11: UR7.14 (CP0)
- net R7p3 is gone; now on net P7p3: UR7.3 (R0(2))
- net S6p1 is gone; now on net P6p1: US6.1 (~{R})
- net S6p2 is gone; now on net GND: US6.2 (D)
- net S6p5 is gone; now on net S6p12: US6.5 (Q)
- net S7p1 is gone; now on net S7p12: US7.1 (CP1..3)
- net S7p10 is gone; now on net GND: US7.10 (GND)
- net S7p14 is gone; now on net R7p11: US7.14 (CP0)
- net S7p3 is gone; now on net P7p3: US7.3 (R0(2))
- net T0p11 is gone; now on net S0p11: UT0.11
- net T0p2 is gone; now on net T0p13: UT0.2
- net T0p3 is gone; now on net S0p3: UT0.3
- net T0p5 is gone; now on net T0p10: UT0.5
- net T0p6 is gone; now on net S0p6: UT0.6
- net T0p8 is gone; now on net S0p8: UT0.8
- net T1p1 is gone; now on net P1p13: UT1.1
- net T1p12 is gone; now on net P1p12: UT1.12
- net T1p13 is gone; now on net P1p13: UT1.13
- net T1p2 is gone; now on net P1p12: UT1.2
- net T3p11 is gone; now on net S3p11: UT3.11
- net T3p13 is gone; now on net P3p13: UT3.13
- net T3p2 is gone; now on net P3p13: UT3.2
- net T3p3 is gone; now on net S3p3: UT3.3
- net T3p5 is gone; now on net T3p10: UT3.5
- net T3p6 is gone; now on net S3p6: UT3.6
- net T3p8 is gone; now on net S3p8: UT3.8
- net U0p3 is gone; now on net S0p3: UU0.3
- net U0p5 is gone; now on net U0p10: UU0.5
- net U0p6 is gone; now on net S0p6: UU0.6
- net U0p8 is gone; now on net S0p8: UU0.8
- net U1p14 is gone; now on net +5V: UU1.14 (VCC)
- net U1p7 is gone; now on net GND: UU1.7 (GND)
- net U2p11 is gone; now on net T2p2: UU2.11
- net U2p3 is gone; now on net T2p1: UU2.3
- net U2p6 is gone; now on net T2p4: UU2.6
- net U2p8 is gone; now on net T2p5: UU2.8
- net U3p11 is gone; now on net S3p11: UU3.11
- net U3p2 is gone; now on net U3p13: UU3.2
- net U3p3 is gone; now on net S3p3: UU3.3
- net U3p5 is gone; now on net U3p10: UU3.5
- net U3p6 is gone; now on net S3p6: UU3.6
- net U3p8 is gone; now on net S3p8: UU3.8
- net U4p14 is gone; now on net +5V: UU4.14 (VCC)
- net U4p7 is gone; now on net GND: UU4.7 (GND)
- net V0p11 is gone; now on net S0p11: UV0.11
- net V0p2 is gone; now on net V0p13: UV0.2
- net V0p3 is gone; now on net S0p3: UV0.3
- net V0p5 is gone; now on net V0p10: UV0.5
- net V0p6 is gone; now on net S0p6: UV0.6
- net V0p8 is gone; now on net S0p8: UV0.8
- net V1p10 is gone; now on net U1p10: UV1.10 (P1)
- net V1p11 is gone; now on net U1p11: UV1.11 (P3)
- net V1p14 is gone; now on net +5V: UV1.14 (VCC)
- net V1p3 is gone; now on net U1p3: UV1.3 (P2)
- net V1p4 is gone; now on net U1p4: UV1.4 (P0)
- net V1p7 is gone; now on net GND: UV1.7 (GND)
- net V2p12 is gone; now on net U2p2: UV2.12
- net V2p2 is gone; now on net U2p13: UV2.2
- net V2p8 is gone; now on net U2p9: UV2.8
- net V3p11 is gone; now on net S3p11: UV3.11
- net V3p2 is gone; now on net V3p13: UV3.2
- net V3p3 is gone; now on net S3p3: UV3.3
- net V3p5 is gone; now on net V3p10: UV3.5
- net V3p6 is gone; now on net S3p6: UV3.6
- net V3p8 is gone; now on net S3p8: UV3.8
- net W0p11 is gone; now on net S0p11: UW0.11
- net W0p13 is gone; now on net S0p3: UW0.13
- net W0p5 is gone; now on net S0p6: UW0.5
- net W0p9 is gone; now on net S0p8: UW0.9
- net W1p12 is gone; now on net GND: UW1.12 (GND)
- net W1p2 is gone; now on net U1p3: UW1.2 (D0)
- net W1p3 is gone; now on net U1p11: UW1.3 (D1)
- net W1p4 is gone; now on net W1p13: UW1.4 (E23)
- net W1p5 is gone; now on net +5V: UW1.5 (VCC)
- net W1p6 is gone; now on net U1p10: UW1.6 (D2)
- net W1p7 is gone; now on net U1p4: UW1.7 (D3)
- net W2p12 is gone; now on net GND: UW2.12 (GND)
- net W2p2 is gone; now on net W2p10: UW2.2 (D0)
- net W2p3 is gone; now on net W2p9: UW2.3 (D1)
- net W2p5 is gone; now on net +5V: UW2.5 (VCC)
- net W3p13 is gone; now on net S3p3: UW3.13
- net W3p5 is gone; now on net S3p6: UW3.5
- net W3p9 is gone; now on net S3p8: UW3.9
- net W4p12 is gone; now on net GND: UW4.12 (GND)
- net W4p2 is gone; now on net U4p3: UW4.2 (D0)
- net W4p3 is gone; now on net U4p11: UW4.3 (D1)
- net W4p4 is gone; now on net W4p13: UW4.4 (E23)
- net W4p5 is gone; now on net +5V: UW4.5 (VCC)
- net W4p6 is gone; now on net U4p10: UW4.6 (D2)
- net W4p7 is gone; now on net U4p4: UW4.7 (D3)
- net +5V: now also C17.2, C18.2, C32.2, C33.2, C34.2, C35.2, C37.2, C5.2, C51.2, C52.2, C53.2, C54.2, C7.1, R21.1, R23.2, R24.1, R31.2, R40.1, R44.1, R60.2, R64.2, R65.2, R66.2, R80.2, R81.1, R82.1, UB5.14 (VCC), UB6.14 (VCC), UB7.14 (VCC), UC5.14 (VCC), UC6.14 (VCC), UC7.14 (VCC), UC8.14 (VCC), UD5.16 (VCC), UD6.14 (VCC), UD7.14 (VCC), UD8.14 (VCC), UE5.14 (VCC), UE6.14 (VCC), UE8.14 (VCC), UF5.14 (VCC), UF6.14 (VCC), UF8.14 (VCC), UG5.14 (VCC), UG6.14 (VCC), UG7.14 (VCC), UG8.14 (VCC), UH5.14 (VCC), UH6.14 (VCC), UH7.14 (VCC), UJ6.14 (VCC), UJ7.16 (VCC), UK5.14 (VCC), UK6.16 (VCC), UK7.14 (VCC), UK8.14 (VCC), UL5.16 (VCC), UL6.14 (VCC), UL7.14 (VCC), UM5.14 (VCC), UM6.14 (VCC), UM7.14 (VCC), UM8.5 (VCC), UN6.14 (VCC), UN7.14 (VCC), UP5.14 (VCC), UP6.14 (VCC), UR6.14 (VCC), US6.14 (VCC), UT0.14 (VCC), UT1.14 (VCC), UT2.14 (VCC), UT3.14 (VCC), UU0.14 (VCC), UU2.14 (VCC), UU3.14 (VCC), UV0.14 (VCC), UV2.14 (VCC), UV3.14 (VCC), UW0.14 (VCC), UW3.14 (VCC), UV4.14 (VCC)
- net B6p12: now also R81.2
- net B6p6: now also R80.1, UB6.9
- net D5p14: now also C40.1
- net D5p6: now also C24.2
- net D5p7: now also C24.1
- net F5p9: now also UE5.5
- net G8p9: now also UG8.13
- net GND: now also C17.1, C18.1, C36.1, C37.1, C38.1, C51.1, C52.1, C53.1, R20.2, UB5.7 (GND), UB6.7 (GND), UB7.7 (GND), UC5.7 (GND), UC6.7 (GND), UC7.7 (GND), UC8.7 (GND), UD5.8 (GND), UD6.7 (GND), UD7.7 (GND), UD8.7 (GND), UE5.7 (GND), UE6.7 (GND), UE8.7 (GND), UF5.7 (GND), UF6.7 (GND), UF7.7 (GND), UF8.7 (GND), UG5.7 (GND), UG6.7 (GND), UG7.7 (GND), UG8.7 (GND), UH5.7 (GND), UH6.7 (GND), UH7.7 (GND), UJ6.7 (GND), UJ7.8 (GND), UK5.7 (GND), UK6.8 (GND), UK7.7 (GND), UL5.8 (GND), UL6.7 (GND), UL7.7 (GND), UM5.7 (GND), UM6.7 (GND), UM7.7 (GND), UN6.7 (GND), UN7.7 (GND), UP5.7 (GND), UP6.7 (GND), US6.7 (GND), UT0.7 (GND), UT1.7 (GND), UT2.7 (GND), UT3.7 (GND), UU0.7 (GND), UU2.7 (GND), UU3.7 (GND), UV0.7 (GND), UV2.7 (GND), UV3.7 (GND), UW0.7 (GND), UW3.7 (GND), Y1.2, UV4.7 (GND)
- net J7p6: now also C47.2
- net K6p14: now also C50.1
- net K6p15: now also C50.2
- net K6p6: now also C49.2
- net K6p7: now also C49.1
- net Q1p1: now also C8.2, C9.1, R23.1, R24.2; no longer Q1.2 (B)
- net Q1p3: now also C9.2, R25.1, Y1.1
- net S0p11: now also UU0.11
- net S2p1: now also US2.1 (A), US2.2 (B)
- net S2p13: now also US2.13 (Qh)
- net S3p11: now also UW3.11
- net S6p4: now also US6.4 (~{S})
- net U0p2: now also UU0.13
- net U2p5: now also UV2.10
- net U4p10: now also UV4.10 (P1)
- net U4p11: now also UV4.11 (P3)
- net U4p13: now also UV4.13 (Mr)
- net U4p3: now also UV4.3 (P2)
- net U4p4: now also UV4.4 (P0)
- net U5p1: now also UU5.1 (E)
- net U5p10: now also UU5.10 (02)
- net U5p12: now also UU5.12 (00)
- net U5p13: now also UU5.13 (A0)
- net U5p2: now also UU5.2 (A0)
- net U5p4: now also UU5.4 (00)
- net U5p5: now also UU5.5 (01)
- net U5p6: now also UU5.6 (02)
- net U5p9: now also UU5.9 (03)
- net V4p1: now also UV4.1 (Pl)
- net V4p12: now also UV4.12 (Q3)
- net V4p2: now also UV4.2 (Q2)
- net V4p5: now also UV4.5 (Q0)
- net V4p6: now also UV4.6 (Cp1)
- net V4p9: now also UV4.9 (Q1)
- net W0p2: now also UW0.2
- net R39p1: now reaches R39.1
- net R39p1: now also R69.2
- net R39p2: now reaches R39.2
- net D8p13: now reaches UD8.13 (~{R})
- net R64p1: now reaches R63.1
- net R64p1: now also R64.1
- net B51: now reaches J2.51 (Pin_51)
- net B67: now reaches J2.67 (Pin_67)
- net B69: now reaches J2.69 (Pin_69)
- net Q1p2: now reaches R21.2
- net Q1p2: now also Q1.2 (B), R20.1
- net R42p2: now reaches R42.2
- net R82p2: now reaches R82.2
- net R60p1: now reaches R61.1
- net R60p1: now also R60.1
- net R78p1: now reaches R78.1
- net R66p1: now reaches R66.1
- net R66p1: now also R62.1
- net G8p11: now reaches UG8.11
- net G8p12: now reaches UG8.12
- net R79p2: now reaches R79.2
- new net U5p11: UU5.11 (01)
- new net U5p14: UU5.14 (A0)
- new net U5p15: UU5.15 (E)
- new net U5p3: UU5.3 (A0)
- new net U5p7: UU5.7 (03)
- new net V4p8: UV4.8 (Cp0)
- no-connect marks 95 -> 91

Commit message: Start Backside AMLDC
Connections:
- net T6p1 is gone; now on net P6p1: UT6.1 (~{R})
- net T6p2 is gone; now on net GND: UT6.2 (D)
- net T6p5 is gone; now on net T6p12: UT6.5 (Q)
- net T7p1 is gone; now on net T7p12: UT7.1 (CP1..3)
- net T7p10 is gone; now on net GND: UT7.10 (GND)
- net T7p14 is gone; now on net S7p11: UT7.14 (CP0)
- net T7p5 is gone; now on net +5V: UT7.5 (VCC)
- net V5p10 is gone; now on net U5p3: UV5.10 (Q2)
- net V5p15 is gone; now on net U5p2: UV5.15 (Q3)
- net V5p16 is gone; now on net +5V: UV5.16 (VCC)
- net V5p8 is gone; now on net GND: UV5.8 (GND)
- net V6p1 is gone; now on net V6p13: UV6.1 (~{R})
- net V6p5 is gone; now on net V6p12: UV6.5 (Q)
- net W5p1 is gone; now on net V5p1: UW5.1 (~{Mr})
- net W5p10 is gone; now on net V5p12: UW5.10 (Q2)
- net W5p15 is gone; now on net V5p13: UW5.15 (Q3)
- net W5p16 is gone; now on net +5V: UW5.16 (VCC)
- net W5p2 is gone; now on net V5p4: UW5.2 (Q0)
- net W5p7 is gone; now on net V5p5: UW5.7 (Q1)
- net W5p8 is gone; now on net GND: UW5.8 (GND)
- net W6p1 is gone; now on net +5V: UW6.1
- net W6p9 is gone; now on net V6p9: UW6.9
- net +5V: now also C22.2, C23.2, R26.1, UT6.14 (VCC), UU5.16 (VCC), UV6.14 (VCC), UV7.14 (VCC), UW6.14 (VCC)
- net GND: now also C21.2, C22.1, C23.1, UT6.7 (GND), UU5.8 (GND), UV6.7 (GND), UV7.7 (GND), UW6.7 (GND)
- net SW1p2: now reaches SW1.2 (B)
- net SW1p2: now also C21.1
- net R22p1: now reaches R22.1
- net R22p2: now reaches R22.2
