File: Mystery Test Board/AMLDC-2044B.kicad_sch (KiCad schematic)
At the start: 332 parts, among them J1 Port A, J2 Port B, Q1 PNP MPS6533, SW1 ~{RESET} RESET, Y1 Crystal

Commit message: Note on MPS6533-Motorola
Other:
- note added: "According to the markings on this TO-92 casing, the pinout I've chosen for this is backwards"

Commit message: Wow
Other:
- note added: "Net D0p9 might be two separate nets, connected by a bad trace/pad on the bottom side at UD0p8. Check a fabricated board to see if these touching traces on that pad have been cut."

Commit message: backside p2
Connections:
- net B1p1 is gone; now on net ~{DCHA}: UB1.1
- net B1p10 is gone; now on net IO RST: R77.1, UB1.10
- net B1p8 is gone; now on net J1p13: UB1.8
- net B2p1 is gone; now on net DATOB: UB2.1
- net B2p11 is gone; now on net DATIC: R91.1, UB2.11
- net B2p4 is gone; now on net DATIB: R70.1, UB2.4
- net B3p1 is gone; now on net E2p8: UB3.1
- net B3p2 is gone; now on net E2p8: UB3.2
- net B4p2 is gone; now on net C2p10: UB4.2 (B)
- net C0p5 is gone; now on net DISK1: R19.1, UC0.5
- net C0p9 is gone; now on net TRK3: CR1.1 (K), R49.1, UC0.9
- net C1p1 is gone; now on net R10p2: UC1.1
- net C1p12 is gone; now on net C0p8: UC1.12
- net C1p2 is gone; now on net C0p6: UC1.2
- net C2p1 is gone; now on net GND: UC2.1 (A)
- net C2p2 is gone; now on net C1p6: UC2.2 (B)
- net C31p2 is gone; now on net C1p13: C31.2, R94.2
- net C3p10 is gone; now on net C1p11: UC3.10 (~{S})
- net C3p13 is gone; now on net C2p4: UC3.13 (~{R})
- net C3p3 is gone; now on net C1p6: UC3.3 (C)
- net C4p10 is gone; now on net C4p11: UC4.10
- net C4p12 is gone; now on net C4p13: UC4.12
- net C4p4 is gone; now on net C4p3: UC4.4
- net C4p5 is gone; now on net H2p4: UC4.5, UD4.11 (C)
- net C58p1 is gone; now on net D0p4: C58.1, R71.1
- net C58p2 is gone; now on net GND: C58.2, C59.2, C60.2, C61.2
- net C59p1 is gone; now on net E0p10: C59.1, R51.1
- net C60p1 is gone; now on net E0p4: C60.1, R53.1
- net C61p1 is gone; now on net E0p2: C61.1, R33.1
- net D0p1 is gone; now on net DATIA: UD0.1
- net D0p11 is gone; now on net DATOA: UD0.11
- net D0p3 is gone; now on net CLR: R71.2, UD0.3
- net D1p1 is gone; now on net DCHI: UD1.1
- net D1p11 is gone; now on net DCHO: UD1.11
- net D1p6 is gone; now on net H2p9: UD1.6
- net D1p9 is gone; now on net D1p13: UD1.5, UD1.9, UE1.5 (Q), UG1.4
- net D2p1 is gone; now on net DATOC: UD2.1
- net D2p3 is gone; now on net F1p12: UD2.3
- net D2p4 is gone; now on net F1p10: UD2.4
- net D3p1 is gone; now on net GND: UD3.1 (A)
- net D3p2 is gone; now on net F2p11: UD3.2 (B)
- net D3p5 is gone; now on net D2p5: UD3.5 (Q)
- net D4p5 is gone; now on net F2p11: UD4.5 (Q)
- net E0p1 is gone; now on net IO PLS: UE0.1
- net E0p11 is gone; now on net STRT: R51.2, UE0.11
- net E0p3 is gone; now on net INTA: R53.2, UE0.3
- net E1p11 is gone; now on net F0p6: UE1.11 (C)
- net E2p10 is gone; now on net E0p12: UE2.10 (~{S})
- net E2p11 is gone; now on net E0p8: UE2.11 (C)
- net E2p12 is gone; now on net C2p10: UE2.12 (D)
- net E4p1 is gone; now on net E3p3: UE4.1
- net E4p10 is gone; now on net E3p11: UE4.10
- net E4p11 is gone; now on net J3p4: UE4.11
- net E4p12 is gone; now on net F1p10: UE4.12
- net E4p13 is gone; now on net E3p13: UE4.13
- net E4p2 is gone; now on net E3p5: UE4.2
- net E4p5 is gone; now on net E3p9: UE4.5
- net E4p8 is gone; now on net H3p3: UE4.8
- net E4p9 is gone; now on net H3p3: UE4.9
- net F0p1 is gone; now on net ~{DS1}: UF0.1
- net F0p11 is gone; now on net DISK NEW REQ: UF0.11
- net F0p13 is gone; now on net DISK PRES REQ: UF0.13
- net F0p3 is gone; now on net ~{DS2}: UF0.3
- net F0p5 is gone; now on net ~{RQENB}: UF0.5
- net F1p1 is gone; now on net ~{DCHP IN}: UF1.1
- net F1p11 is gone; now on net J1p13: UF1.11
- net F1p13 is gone; now on net DISK0 ACT: UF1.13
- net F1p9 is gone; now on net B1p11: UF1.9
- net F2p10 is gone; now on net TRK2: UF2.10
- net F2p13 is gone; now on net C4p1: UF2.13
- net F2p2 is gone; now on net DSK SEL: UF2.2
- net F2p4 is gone; now on net DISK WR DATA: UF2.4
- net F2p5 is gone; now on net WALLOUT: UF2.5
- net F2p8 is gone; now on net TRK4: UF2.8
- net F4p12 is gone; now on net F1p6: UF4.12 (D), UF4.2 (D)
- net F4p5 is gone; now on net F2p1: UF4.5 (Q)
- net F4p9 is gone; now on net H3p2: UF4.9 (Q)
- net G0p1 is gone; now on net ~{DS3}: UG0.1
- net G1p2 is gone; now on net E1p9: UG1.13, UG1.2
- net G1p3 is gone; now on net ~{DCHR}: UG1.3
- net G1p6 is gone; now on net ~{DCHM0}: UG1.6
- net G1p8 is gone; now on net ~{DCHP OUT}: UG1.8
- net G2p12 is gone; now on net B1p11: UG2.12
- net G3p10 is gone; now on net J3p3: UG3.10
- net G3p2 is gone; now on net C3p5: UG3.2, UH3.13
- net H0p1 is gone; now on net ~{INTP IN}: UH0.1
- net H0p11 is gone; now on net ~{DS5}: JP4.2 (B), UH0.11
- net H0p13 is gone; now on net ~{DS4}: JP6.2 (B), UH0.13
- net H0p2 is gone; now on net E0p5: UH0.2, UJ0.1
- net H0p3 is gone; now on net ~{MSKO}: UH0.3
- net H0p9 is gone; now on net ~{DS0}: JP2.2 (B), UH0.9
- net H1p1 is gone; now on net G0p8: UH1.1
- net H1p10 is gone; now on net G0p8: UH1.10, UH1.2
- net H1p3 is gone; now on net J0p10: UH1.3
- net H1p6 is gone; now on net H0p5: UH1.6
- net H1p8 is gone; now on net D0p9: UH1.8
- net H1p9 is gone; now on net G0p8: UH1.9
- net H2p10 is gone; now on net E1p13: UH2.10
- net H2p11 is gone; now on net E1p13: UH2.11
- net H2p6 is gone; now on net K1p10: UH2.6
- net H3p1 is gone; now on net C2p12: UH3.1
- net H3p10 is gone; now on net H3p11: UH3.10
- net H3p12 is gone; now on net F1p6: UH3.12, UJ3.13
- net H3p4 is gone; now on net H2p12: UH3.4
- net H4p1 is gone; now on net TRK6: UH4.1 (A)
- net H4p11 is gone; now on net J1p13: UH4.11 (Clr)
- net J0p3 is gone; now on net ~{INTP OUT}: UJ0.3
- net J0p5 is gone; now on net J0p4: UJ0.5
- net J0p6 is gone; now on net ~{INTR}: UJ0.6
- net J0p8 is gone; now on net ~{SELB}: UJ0.8
- net J1p11 is gone; now on net H0p4: UJ1.11 (C)
- net J1p2 is gone; now on net H0p6: UJ1.2 (D)
- net J1p3 is gone; now on net F0p6: UJ1.3 (C)
- net J1p5 is gone; now on net J0p4: UJ1.5 (Q)
- net J1p6 is gone; now on net J0p2: UJ1.6 (~{Q})
- net J2p12 is gone; now on net J0p9: UJ2.12 (D), UJ2.5 (Q)
- net J2p2 is gone; now on net GND: UJ2.2 (D)
- net J2p3 is gone; now on net J2p9: UJ2.3 (C)
- net J2p4 is gone; now on net E0p8: UJ2.4 (~{S}), UK2.12
- net J2p8 is gone; now on net H1p13: UJ2.8 (~{Q})
- net J3p10 is gone; now on net L0p9: UJ3.10
- net J3p11 is gone; now on net L0p9: UJ3.11
- net J3p2 is gone; now on net C1p6: UJ3.2
- net J3p9 is gone; now on net L0p9: UJ3.9
- net K0p12 is gone; now on net SPARE: UK0.12
- net K0p2 is gone; now on net DISK2: UK0.2
- net K0p4 is gone; now on net DSK ~{RST}: UK0.4
- net K0p9 is gone; now on net A77: UK0.9
- net K1p12 is gone; now on net J0p9: UK1.12 (D)
- net K1p13 is gone; now on net G2p4: UK1.13 (~{R})
- net K1p9 is gone; now on net E1p12: UK1.2 (D), UK1.9 (Q)
- net K2p1 is gone; now on net K1p11: UK2.1
- net K2p10 is gone; now on net D0p6: UK2.10
- net K2p2 is gone; now on net K1p6: UK2.2
- net K2p6 is gone; now on net K1p3: UK2.6
- net K2p9 is gone; now on net J1p13: UK2.9
- net L0p10 is gone; now on net L0p13: UL0.10, UL0.5
- net L0p11 is gone; now on net ~{DATA14}: UL0.11, UM0.11, UN0.11, UP0.11, UR0.11
- net L0p8 is gone; now on net ~{DATA12}: UL0.8, UM0.8, UN0.9, UP0.8, UR0.8
- net L1p1 is gone; now on net D2p12: UL1.1 (Pl)
- net L1p10 is gone; now on net N0p10: UL1.10 (P1), UM1.10 (P1), UN1.6 (D2)
- net L1p11 is gone; now on net N0p8: UL1.11 (P3), UN1.3 (D1)
- net L1p12 is gone; now on net L0p9: UL1.12 (Q3)
- net L1p2 is gone; now on net L0p4: UL1.2 (Q2)
- net L1p3 is gone; now on net N0p6: UL1.3 (P2), UM1.3 (P2), UN1.2 (D0)
- net L1p4 is gone; now on net N0p8: UM1.11 (P3)
- net L1p5 is gone; now on net L0p1: UL1.5 (Q0)
- net L1p6 is gone; now on net L0p1: UL1.6 (Cp1)
- net L1p9 is gone; now on net L0p12: UL1.9 (Q1)
- net L2p1 is gone; now on net L2p2: UL2.1
- net L2p11 is gone; now on net J1p1: UL2.11
- net L2p3 is gone; now on net K1p11: UL2.3, UM2.1 (~{PL})
- net L2p4 is gone; now on net B2p8: UL2.4
- net L2p5 is gone; now on net B2p8: UL2.5
- net L2p9 is gone; now on net D0p8: UL2.9
- net L3p10 is gone; now on net L0p13: UL3.10, UL3.5
- net L3p13 is gone; now on net L0p13: UL3.13, UL3.2
- net L3p3 is gone; now on net ~{DATA3}: UL3.3, UM3.3, UN3.13, UP3.3, UR3.3
- net L3p6 is gone; now on net ~{DATA1}: UL3.6, UM3.6, UN3.5, UP3.6, UR3.6
- net L4p1 is gone; now on net D2p12: UL4.1 (Pl)
- net L4p12 is gone; now on net L3p9: UL4.12 (Q3)
- net L4p13 is gone; now on net J1p13: UL4.13 (Mr), UM4.13 (Mr)
- net L4p2 is gone; now on net L3p4: UL4.2 (Q2)
- net L4p5 is gone; now on net L3p1: UL4.5 (Q0)
- net L4p6 is gone; now on net L3p1: UL4.6 (Cp1)
- net L4p9 is gone; now on net L3p12: UL4.9 (Q1)
- net M0p10 is gone; now on net M0p13: UM0.10, UM0.5
- net M1p1 is gone; now on net B2p12: UM1.1 (Pl)
- net M1p12 is gone; now on net M0p9: UM1.12 (Q3)
- net M1p2 is gone; now on net M0p4: UM1.2 (Q2)
- net M1p5 is gone; now on net M0p1: UM1.5 (Q0)
- net M1p6 is gone; now on net M0p1: UM1.6 (Cp1)
- net M1p8 is gone; now on net F1p8: UM1.8 (Cp0)
- net M1p9 is gone; now on net M0p12: UM1.9 (Q1)
- net M2p11 is gone; now on net N1p9: UM2.11 (D0)
- net M2p12 is gone; now on net N1p10: UM2.12 (D1)
- net M2p13 is gone; now on net N1p16: UM2.13 (D2)
- net M2p14 is gone; now on net N1p15: UM2.14 (D3)
- net M3p10 is gone; now on net M3p13: UM3.10, UM3.5
- net M4p1 is gone; now on net B2p12: UM4.1 (Pl)
- net M4p12 is gone; now on net M3p9: UM4.12 (Q3)
- net M4p2 is gone; now on net M3p4: UM4.2 (Q2)
- net M4p5 is gone; now on net M3p1: UM4.5 (Q0)
- net M4p6 is gone; now on net M3p1: UM4.6 (Cp1)
- net M4p9 is gone; now on net M3p12: UM4.9 (Q1)
- net N0p1 is gone; now on net F0p12: UN0.1
- net N0p3 is gone; now on net D0p12: UN0.3
- net N0p4 is gone; now on net T0p13: UN0.4, UP0.10, UP0.5
- net N1p12 is gone; now on net GND: UN1.12 (GND)
- net N1p7 is gone; now on net N0p12: UL1.4 (P0), UM1.4 (P0), UN1.7 (D3)
- net N2p13 is gone; now on net L2p8: UN2.13 (E01), UN2.4 (E23)
- net N2p2 is gone; now on net N0p6: UN2.2 (D0)
- net N2p3 is gone; now on net N0p8: UN2.3 (D1)
- net N2p5 is gone; now on net +5V: C69.1, UN2.5 (VCC), UP2.14 (VCC)
- net N2p6 is gone; now on net N0p10: UN2.6 (D2)
- net N2p7 is gone; now on net N0p12: UN2.7 (D3)
- net N3p1 is gone; now on net K1p11: UN3.1
- net N3p10 is gone; now on net L4p10: UN3.10
- net N3p12 is gone; now on net L4p4: UN3.12
- net N3p6 is gone; now on net L4p3: UN3.6
- net N3p8 is gone; now on net L4p11: UN3.8
- net N4p12 is gone; now on net GND: C55.2, UN4.12 (GND), UP4.11 (B2), UP4.14 (D3), UP4.2 (B0), UP4.5 (B1)
- net N4p5 is gone; now on net +5V: UN4.5 (VCC)
- net P0p12 is gone; now on net K1p5: UP0.12
- net P0p13 is gone; now on net T0p13: UP0.13, UP0.2
- net P1p10 is gone; now on net B1p13: UP1.10
- net P1p11 is gone; now on net ~{DATA12}: UP1.11
- net P1p12 is gone; now on net J0p4: UP1.12, UP1.2, UP1.4, UT1.12, UT1.2
- net P1p13 is gone; now on net F0p8: UP1.1, UP1.13, UT1.1, UT1.13
- net P1p5 is gone; now on net F0p8: UP1.5
- net P1p8 is gone; now on net R0p13: UP1.8
- net P1p9 is gone; now on net B1p13: UP1.9
- net P2p10 is gone; now on net B25: UP2.10
- net P2p12 is gone; now on net B27: UP2.12
- net P2p6 is gone; now on net B23: UP2.6
- net P2p8 is gone; now on net B19: UP2.8
- net P2p9 is gone; now on net R2p9: UP2.9
- net P3p10 is gone; now on net P3p13: UP3.10, UP3.5
- net P3p9 is gone; now on net J2p9: UP3.9
- net Pad77 is gone; now on net A77: R35.2
- net R13p2 is gone; now on net C2p7: C15.1, R13.2
- net R1p10 is gone; now on net R0p1: UR1.10 (Q2)
- net R1p15 is gone; now on net R0p12: UR1.15 (Q1)
- net R1p16 is gone; now on net R0p9: UR1.16 (Q0)
- net R1p5 is gone; now on net +5V: UR1.5 (VCC), US1.5 (VCC)
- net R1p9 is gone; now on net R0p4: UR1.9 (Q3)
- net R2p12 is gone; now on net GND: UR2.12 (GND)
- net R2p15 is gone; now on net P2p11: UR2.15 (Q1)
- net R2p16 is gone; now on net P2p13: UR2.16 (Q0)
- net R2p4 is gone; now on net E2p9: UR2.4 (E23)
- net R34P1 is gone; now on net GND: R15.1, R16.1, R34.1, R35.1
- net R3p10 is gone; now on net R0p13: UR3.10, UR3.5, US3.10, US3.5
- net R3p13 is gone; now on net R0p13: UR3.13, UR3.2, US3.13, US3.2
- net R4p10 is gone; now on net R3p1: UR4.10 (Q2)
- net R4p13 is gone; now on net N3p2: UR4.13 (E01), UR4.4 (E23), US4.13 (E01), US4.4 (E23)
- net R4p15 is gone; now on net R3p12: UR4.15 (Q1)
- net R4p16 is gone; now on net R3p9: UR4.16 (Q0)
- net R4p5 is gone; now on net +5V: UR4.5 (VCC)
- net R4p9 is gone; now on net R3p4: UR4.9 (Q3)
- net R56P2 is gone; now on net +5V: R17.2, R36.2, R56.2, R92.2
- net R78p1 is gone; now on net N1p4: R78.1
- net R82p2 is gone; now on net M3p13: R82.2
- net R9p2 is gone; now on net D1p2: C43.1, R9.2
- net S1p10 is gone; now on net S0p1: US1.10 (Q2)
- net S1p15 is gone; now on net S0p12: US1.15 (Q1)
- net S1p16 is gone; now on net S0p9: US1.16 (Q0)
- net S1p9 is gone; now on net S0p4: US1.9 (Q3)
- net S2p1 is gone; now on net C3p5: US2.1 (A), US2.2 (B)
- net S2p13 is gone; now on net S1p2: US2.13 (Qh)
- net S4p10 is gone; now on net S3p1: US4.10 (Q2)
- net S4p15 is gone; now on net S3p12: US4.15 (Q1)
- net S4p16 is gone; now on net S3p9: US4.16 (Q0)
- net S4p5 is gone; now on net +5V: US4.5 (VCC)
- net S4p9 is gone; now on net S3p4: US4.9 (Q3)
- net T0p12 is gone; now on net F0p12: UT0.12
- net T1p10 is gone; now on net B1p12: UT1.10
- net T1p8 is gone; now on net N1p4: UT1.8
- net T1p9 is gone; now on net B1p12: UT1.9
- net +5V: now also C19.2, C63.1, R48.2, R6.2, R8.1, R89.1
- net A77: now also R4.1
- net B2p13: no longer UD2.13
- net B2p2: now also R58.2
- net B3p10: now also CR4.2 (A), R3.2
- net B3p4: now also R2.2
- net B3p6: now also R29.1
- net B4p15: now also R1.2
- net B4p7: now also R87.1
- net C0p6: now also R10.1
- net C0p8: now also R94.1
- net C14p2: no longer R29.1
- net C2p10: now also R30.1
- net D0p10: now also C20.2, R83.2
- net D0p2: now also C1.1, R46.2
- net D0p8: now also UP4.7 (S1)
- net D0p9: now also UD2.13
- net D1p10: now also R11.2
- net D2p2: now also R14.2
- net D3p15: now also R27.1
- net D3p7: now also R89.2
- net D4p12: now also R88.1
- net DATIA: now also R46.1
- net DATOA: now also R83.1
- net DATOB: now also R58.1
- net DATOC: now also R14.1
- net DCHI: now also R9.1
- net DCHO: now also R11.1
- net DISK NEW REQ: now also R72.1
- net DISK PRES REQ: now also R32.1
- net DISK WR DATA: now also R3.1
- net DISK0 ACT: now also R73.2
- net DISK1: now also CR5.1 (K), R18.1
- net DISK2: now also R57.1, R92.1
- net DSK ~{RST}: now also R15.2, R76.1
- net E2p8: now also C14.1
- net G2p1: now also UP4.9 (S0)
- net GND: now also C1.2, C10.1, C19.1, C20.1, C28.1, C44.2, C46.2, C63.2, C69.2, C70.2, CR5.2 (A), R5.1, UG4.1 (A), UP2.7 (GND)
- net H4p15: now also R47.2
- net H4p2: now also R48.1
- net IO PLS: now also R33.2
- net J2p9: now also UJ0.12
- net K0p1: now also R57.2
- net K0p10: now also R4.2
- net K0p13: now also C71.1, R75.2
- net K0p5: now also R76.2
- net L0p13: now also UL2.6
- net L0p3: now also JP8.1 (A)
- net M2p2: now also US2.8 (CK)
- net P0p9: now also UP0.9
- net P1p3: now also JP8.2 (B)
- net P1p6: now also JP7.2 (B)
- net Pad15p15: now also R68.2
- net R0p13: now also R85.1
- net R1p2: now also US2.6 (Qd)
- net R1p3: now also US2.4 (Qb)
- net R1p6: now also US2.3 (Qa)
- net R1p7: now also US2.5 (Qc)
- net R50P2: now also CR4.1 (K), R12.1
- net S1p3: now also US2.11 (Qf)
- net S1p6: now also US2.10 (Qe)
- net S1p7: now also US2.12 (Qg)
- net SPARE: now also R34.2, R75.1
- net T0p10: no longer UT0.10
- net T0p13: now also UT0.10
- net TRK3: now also R37.1
- net TRK6: now also R6.1, R7.1
- net ~{DATA14}: now also JP7.1 (A)
- net ~{DCHA}: now also R38.1
- net ~{DCHM0}: now also C62.1
- net ~{DCHP OUT}: now also R5.2, R54.2, R74.1
- net ~{DS2}: now also R74.2
- net ~{INTP OUT}: now also R55.1
- net ~{SELD}: now also UJ0.11
- net unconnected-(UP5-Pad3): now reaches UP5.3
- net unconnected-(UP5-Pad11): now reaches UP5.11
- net unconnected-(US2-~{R}-Pad9): now reaches US2.9 (~{R})
- net C29p1: now reaches R50.2
- net C29p1: now also C29.1
- net unconnected-(UT2-Pad11): now reaches UT2.11
- net unconnected-(UP4-A0-Pad1): now reaches UP4.1 (A0)
- net unconnected-(UP4-F2-Pad12): now reaches UP4.12 (F2)
- net unconnected-(UP4-F3-Pad13): now reaches UP4.13 (F3)
- net unconnected-(UP4-F0-Pad3): now reaches UP4.3 (F0)
- net unconnected-(UP4-F1-Pad4): now reaches UP4.4 (F1)
- net unconnected-(UT2-Pad3): now reaches UT2.3
Other:
- note added: "Error: Cannot find UT7 pin '13'. Error: Cannot find UT7 pin '4'. Error: Cannot find UT7 pin '6'. Error: Cannot find UT7 pin '7'. BUT UT7p7 is actually USED to V7p13"
- moved on the sheet: C65

Commit message: AMLDC - Right before switching card-edge from Disk to Tape
Parts:
- added J1 (x2): Slot_02x50_Odd_Even, Forgotten Machines:DG NOVA Backplane Connector - Frontside, symbol NovaMem-rescue:Slot_02x50_Odd_Even-_local
Connections:
- net 2G5p2 is gone; now on net GND: UG5.2 (D)
- net B5p11 is gone; now on net G2p2: UB5.11
- net B5p12 is gone; now on net B4p13: UB5.12
- net B5p13 is gone; now on net D4p13: UB5.13
- net B5p4 is gone; now on net B5p3: UB5.4
- net B5p6 is gone; now on net C4p1: UB5.6
- net B5p8 is gone; now on net B4p10: UB5.8
- net B6p1 is gone; now on net B6p11: UB6.1
- net B6p12 is gone; now on net E3p1: R81.2, UB6.12
- net B6p13 is gone; now on net E3p1: UB6.13
- net B6p3 is gone; now on net F4p1: UB6.3
- net B6p5 is gone; now on net B6p4: UB6.5
- net B6p8 is gone; now on net E3p1: UB6.8
- net C5p1 is gone; now on net E2p13: UC5.1
- net C5p10 is gone; now on net B3p8: UC5.10
- net C5p11 is gone; now on net C4p8: UC5.11
- net C5p12 is gone; now on net C4p8: UC5.12
- net C5p2 is gone; now on net F1p10: UC5.2
- net C5p3 is gone; now on net H2p4: UC5.3, UD5.5 (Q)
- net C5p5 is gone; now on net GND: UC5.5
- net C5p6 is gone; now on net GND: UC5.6
- net C5p8 is gone; now on net G2p10: UC5.8
- net C5p9 is gone; now on net G2p10: UC5.9
- net C6p11 is gone; now on net B4p10: UC6.11 (C)
- net D5p4 is gone; now on net D4p3: UD5.4 (~{Q})
- net D5p9 is gone; now on net B3p4: UD5.9 (A)
- net D6p11 is gone; now on net E4p6: UD6.11
- net E5p1 is gone; now on net H3p5: UE5.1
- net E5p2 is gone; now on net J3p5: UE5.2
- net E5p3 is gone; now on net G2p8: UE5.3
- net E5p6 is gone; now on net J3p5: UE5.6
- net E5p8 is gone; now on net G2p9: UE5.8
- net E6p1 is gone; now on net J3p5: UE6.1
- net E6p10 is gone; now on net G2p9: UE6.10
- net E6p12 is gone; now on net C1p6: UE6.12
- net E6p13 is gone; now on net E3p9: UE6.13, UF6.13
- net E6p4 is gone; now on net E6p3: UE6.4
- net F5p13 is gone; now on net WALLOUT: UF5.1 (~{R}), UF5.13 (~{R}), UH5.9 (Q)
- net F6p1 is gone; now on net G2p9: UF6.1
- net F6p12 is gone; now on net C2p5: UF6.12
- net F6p4 is gone; now on net F6p3: UF6.4
- net F6p6 is gone; now on net M2p2: UF6.6
- net G5p3 is gone; now on net F4p3: UG5.3 (C)
- net G6p13 is gone; now on net H5p8: UG6.13
- net G6p2 is gone; now on net G5p6: UG6.2, UH6.2, UJ6.11
- net G6p4 is gone; now on net E4p6: UG6.4
- net H5p11 is gone; now on net H4p12: UH5.11 (C)
- net H5p12 is gone; now on net H2p12: UH5.12 (D)
- net H5p6 is gone; now on net F3p1: UH5.6 (~{Q})
- net H6p10 is gone; now on net G6p6: UH6.10
- net H6p11 is gone; now on net H4p10: UH6.11
- net H6p13 is gone; now on net F3p1: UH6.13
- net H6p4 is gone; now on net H6p3: UH6.4
- net H6p5 is gone; now on net H6p3: UH6.5
- net H6p6 is gone; now on net H5p3: UH6.6
- net H6p8 is gone; now on net H5p1: UH6.8
- net J6p1 is gone; now on net J3p6: UJ6.1
- net J6p10 is gone; now on net H2p12: UJ6.10
- net J6p12 is gone; now on net H3p5: UJ6.12
- net J6p2 is gone; now on net G6p8: UJ6.2
- net J6p9 is gone; now on net E4p6: UJ6.9
- net K5p10 is gone; now on net DATA RDR: UK5.10
- net K5p12 is gone; now on net +V TERM: UK5.12
- net K5p2 is gone; now on net B15: UK5.2
- net K5p4 is gone; now on net B34: UK5.4
- net K5p6 is gone; now on net +V TERM: UK5.6
- net K6p5 is gone; now on net H2p13: UK6.5 (Q)
- net L5p1 is gone; now on net GND: UL5.1 (E)
- net L5p2 is gone; now on net L3p4: UL5.2 (A0)
- net L5p3 is gone; now on net L3p9: UL5.3 (A0)
- net L6p1 is gone; now on net K5p1: UL6.1
- net L6p10 is gone; now on net K5p3: UL6.10
- net L6p12 is gone; now on net C4p6: UL6.12, UL6.2, UL6.5, UL6.9
- net L6p13 is gone; now on net K5p5: UL6.13
- net L6p4 is gone; now on net K5p13: UL6.4
- net M5p6 is gone; now on net G6p10: UM5.6
- net M5p8 is gone; now on net L1p8: UM5.8
- net M6p1 is gone; now on net P0p1: UM6.1
- net M6p10 is gone; now on net M6p11: UM6.10
- net M6p12 is gone; now on net K2p11: UM6.12
- net M6p13 is gone; now on net J2p13: UM6.13
- net M6p3 is gone; now on net M6p2: UM6.3
- net M6p4 is gone; now on net M6p2: UM6.4
- net M6p5 is gone; now on net K1p5: UM6.5
- net M6p9 is gone; now on net D0p8: UM6.9
- net N5p1 is gone; now on net K1p11: UN5.1 (~{PL})
- net N5p10 is gone; now on net M2p9: UN5.10 (DS)
- net N5p15 is gone; now on net GND: UN5.15 (~{CE})
- net N5p2 is gone; now on net M2p2: UN5.2 (CP), UR5.8 (CK)
- net N5p3 is gone; now on net N4p9: UN5.3 (D4)
- net N5p4 is gone; now on net N4p10: UN5.4 (D5)
- net N5p5 is gone; now on net N4p16: UN5.5 (D6)
- net N5p6 is gone; now on net N4p15: UN5.6 (D7)
- net N6p1 is gone; now on net L2p2: UN6.1
- net N6p11 is gone; now on net L4p11: UN6.11
- net N6p12 is gone; now on net L4p11: UN6.12
- net N6p4 is gone; now on net N6p3: UN6.4
- net N6p6 is gone; now on net N6p5: UN6.6
- net N6p8 is gone; now on net M2p2: UN6.8
- net N6p9 is gone; now on net M2p2: UN6.9
- net P5p1 is gone; now on net T3p9: UP5.1
- net P5p2 is gone; now on net P3p4: UP5.2
- net P5p4 is gone; now on net P3p1: UP5.4
- net P5p5 is gone; now on net P3p12: UP5.5
- net P5p6 is gone; now on net H1p12: UP5.6
- net P6p1 is gone; now on net G2p1: UP6.1 (~{R}), UR6.1 (~{R}), US6.1 (~{R}), UT6.1 (~{R})
- net P6p11 is gone; now on net K0p11: UP6.11 (C)
- net P6p3 is gone; now on net P3p4: UP6.3 (C)
- net P6p4 is gone; now on net L6p3: UP6.4 (~{S})
- net P6p9 is gone; now on net P3p4: UP6.9 (Q)
- net R5p1 is gone; now on net S1p2: UR5.1 (A)
- net R5p10 is gone; now on net R4p6: UR5.10 (Qe)
- net R5p11 is gone; now on net R4p3: UR5.11 (Qf)
- net R5p12 is gone; now on net R4p7: UR5.12 (Qg)
- net R5p13 is gone; now on net R4p2: UR5.13 (Qh)
- net R5p3 is gone; now on net S4p6: UR5.3 (Qa)
- net R5p4 is gone; now on net S4p3: UR5.4 (Qb)
- net R5p5 is gone; now on net S4p7: UR5.5 (Qc)
- net R5p6 is gone; now on net S4p2: UR5.6 (Qd)
- net R6p11 is gone; now on net K0p8: UR6.11 (C)
- net R6p3 is gone; now on net P3p12: UR6.3 (C)
- net R6p4 is gone; now on net L6p6: UR6.4 (~{S})
- net R6p9 is gone; now on net P3p12: UR6.9 (Q)
- net R79p2 is gone; now on net F4p1: R79.2
- net S6p11 is gone; now on net K0p6: US6.11 (C)
- net S6p3 is gone; now on net P3p1: US6.3 (C)
- net S6p4 is gone; now on net L6p8: US6.4 (~{S})
- net S6p9 is gone; now on net P3p1: US6.9 (Q)
- net unconnected-(UP4-F1-Pad4) is gone; now on net S6p13: UP4.4 (F1)
- net unconnected-(UP4-F2-Pad12) is gone; now on net R6p13: UP4.12 (F2)
- net unconnected-(UP4-F3-Pad13) is gone; now on net P6p13: UP4.13 (F3)
- net unconnected-(US2-~{R}-Pad9) is gone; now on net M2p9: US2.9 (~{R})
- net +5V: now also R41.2, R45.2, R67.2, J1.3 (Pin_3), J1.3 (Pin_3), J1.4 (Pin_4), J1.4 (Pin_4), J1.97 (Pin_69), J1.97 (Pin_69), J1.98 (Pin_98), J1.98 (Pin_98)
- net +VINH: now also J1.10 (Pin_10), J1.84 (Pin_84)
- net -5V: now also J1.6 (Pin_6), J1.81 (Pin_81)
- net B6p6: now also C7.2, UB6.10
- net CLR: now also J1.50 (Pin_50)
- net D5p15: now also C40.2, R44.2
- net D5p7: now also R45.1
- net DATIA: now also J1.44 (Pin_44)
- net DATIB: now also J1.42 (Pin_42)
- net DATIC: now also J1.54 (Pin_54)
- net DATOA: now also J1.58 (Pin_58)
- net DATOB: now also J1.56 (Pin_56)
- net DATOC: now also J1.48 (Pin_48)
- net DCHI: now also J1.37 (Pin_37)
- net DCHO: now also J1.33 (Pin_33)
- net E3p1: now also C5.1
- net G6p1: no longer UG6.1
- net GND: now also J1.1 (Pin_1), J1.1 (Pin_1), J1.100 (Pin_100), J1.100 (Pin_100), J1.2 (Pin_2), J1.2 (Pin_2), J1.33 (Pin_33), J1.34 (Pin_34), J1.50 (Pin_50), J1.99 (Pin_99), J1.99 (Pin_99)
- net H4p4: now also UG6.1
- net INTA: now also J1.40 (Pin_40)
- net IO PLS: now also J1.74 (Pin_74)
- net IO RST: now also J1.70 (Pin_70)
- net K6p12: now also C48.2
- net K6p15: now also R41.1
- net K6p7: now also R40.2
- net OVFLO: now also J1.39 (Pin_39)
- net STRT: now also J1.52 (Pin_52)
- net ~{DATA0}: now also J1.62 (Pin_62)
- net ~{DATA10}: now also J1.75 (Pin_75)
- net ~{DATA11}: now also J1.58 (Pin_58)
- net ~{DATA12}: now also J1.59 (Pin_59)
- net ~{DATA13}: now also J1.64 (Pin_64)
- net ~{DATA14}: now also J1.56 (Pin_56)
- net ~{DATA15}: now also J1.66 (Pin_66)
- net ~{DATA1}: now also J1.65 (Pin_65)
- net ~{DATA2}: now also J1.82 (Pin_82)
- net ~{DATA3}: now also J1.73 (Pin_73)
- net ~{DATA4}: now also J1.61 (Pin_61)
- net ~{DATA5}: now also J1.57 (Pin_57)
- net ~{DATA6}: now also J1.95 (Pin_95)
- net ~{DATA7}: now also J1.55 (Pin_55)
- net ~{DATA8}: now also J1.60 (Pin_60)
- net ~{DATA9}: now also J1.63 (Pin_63)
- net ~{DCHA}: now also J1.60 (Pin_60)
- net ~{DCHM0}: now also J1.17 (Pin_17)
- net ~{DCHM1}: now also J1.21 (Pin_21)
- net ~{DCHP IN}: now also J1.94 (Pin_94)
- net ~{DCHP OUT}: now also J1.93 (Pin_93)
- net ~{DCHR}: now also J1.35 (Pin_35)
- net ~{DS0}: now also J1.72 (Pin_72)
- net ~{DS1}: now also J1.68 (Pin_68)
- net ~{DS2}: now also J1.66 (Pin_66)
- net ~{DS3}: now also J1.46 (Pin_46)
- net ~{DS4}: now also J1.62 (Pin_62)
- net ~{DS5}: now also J1.64 (Pin_64)
- net ~{INTP IN}: now also J1.96 (Pin_96)
- net ~{INTP OUT}: now also J1.95 (Pin_95)
- net ~{INTR}: now also J1.29 (Pin_29)
- net ~{MSKO}: now also J1.38 (Pin_38)
- net ~{RQENB}: now also J1.41 (Pin_41)
- net ~{SELB}: now also J1.82 (Pin_82)
- net ~{SELD}: now also J1.80 (Pin_80)
- net B34: now reaches J2.34 (Pin_34)
- net B40: now reaches J2.40 (Pin_40)
- net B48: now reaches J2.48 (Pin_48)
- net B52: now reaches J2.52 (Pin_52)
- net B54: now reaches J2.54 (Pin_54)
- net unconnected-(UP4-A0-Pad1) renamed P4p1
- net unconnected-(UP4-F0-Pad3) renamed P4p3
- net unconnected-(UP5-Pad11) renamed P5p11
- net unconnected-(UP5-Pad3) renamed P5p3
- net unconnected-(UT2-Pad11) renamed T2p11
- net unconnected-(UT2-Pad3) renamed T2p3
- new net 9 CH: J1.71 (Pin_71)
- new net BOT: J1.53 (Pin_53)
- new net DLY CNT: J1.47 (Pin_47)
- new net DLY1: J1.81 (Pin_81)
- new net EOT: J1.48 (Pin_48)
- new net HI DENS: J1.49 (Pin_49)
- new net RB0: J1.31 (Pin_31)
- new net RB1: J1.40 (Pin_40)
- new net RB2: J1.25 (Pin_25)
- new net RB3: J1.27 (Pin_27)
- new net RB4: J1.13 (Pin_13)
- new net RB5: J1.15 (Pin_15)
- new net RB6: J1.19 (Pin_19)
- new net RB7: J1.23 (Pin_23)
- new net RBP: J1.38 (Pin_38)
- new net RD EN: J1.76 (Pin_76)
- new net RPO: J1.49 (Pin_49)
- new net RWND T: J1.69 (Pin_69)
- new net RWNDG: J1.11 (Pin_11)
- new net SEL 2 (1): J1.78 (Pin_78)
- new net SEL 2 (2): J1.79 (Pin_79)
- new net SEL2: J1.75 (Pin_75)
- new net SND CLK: J1.63 (Pin_63)
- new net SPC BKD: J1.67 (Pin_67)
- new net TUR: J1.54 (Pin_54)
- new net WB0: J1.87 (Pin_87)
- new net WB1: J1.85 (Pin_85)
- new net WB2: J1.89 (Pin_89)
- new net WB3: J1.84 (Pin_84)
- new net WB4: J1.91 (Pin_91)
- new net WB5: J1.86 (Pin_86)
- new net WB6: J1.34 (Pin_34)
- new net WB7: J1.83 (Pin_83)
- new net WBP: J1.59 (Pin_59)
- new net WL: J1.36 (Pin_36)
- new net WRT STROBE: J1.77 (Pin_77)
- new net WRT ~{RST}: J1.57 (Pin_57)
- new net WRT7: J1.61 (Pin_61)
- new net ~{RUN}: J1.73 (Pin_73)
- no-connect marks 91 -> 180
Other:
- note added: "SLOT 16 MAG TAPE OR IO"
- note removed: "SLOT 15 DISK OR IO"
