File: Mystery Test Board/AMLDC-2044B.kicad_sch (KiCad schematic)
At the start: 334 parts, among them J1 Port A, J1 Slot_02x50_Odd_Even, J2 Port B, Q1 PNP MPS6533, SW1 ~{RESET} RESET, Y1 Crystal

Commit message: AMLDC Ready for part 6
Parts:
- removed J1 (x2): Slot_02x50_Odd_Even, Forgotten Machines:DG NOVA Backplane Connector - Frontside, symbol NovaMem-rescue:Slot_02x50_Odd_Even-_local
Connections:
- net +V TERM: no longer J2.11 (Pin_11), J2.13 (Pin_13), UK5.12, UK5.6
- net B15: no longer J2.15 (Pin_15), UK5.2
- net B19: no longer J2.19 (Pin_19), UP2.8
- net B23: no longer J2.23 (Pin_23), UP2.6
- net B25: no longer J2.25 (Pin_25), UP2.10
- net B27: no longer J2.27 (Pin_27), UP2.12
- net B34: no longer J2.34 (Pin_34), UK5.4
- net B40: no longer J2.40 (Pin_40)
- net B48: no longer J2.48 (Pin_48)
- net B49: no longer J2.49 (Pin_49)
- net B54: no longer J2.54 (Pin_54)
- net B67: no longer J2.67 (Pin_67)
- net B69: no longer J2.69 (Pin_69)
- net BOT: now also J2.53 (Pin_53)
- net CLK RDR: no longer J2.38 (Pin_38)
- net DATA RDR: no longer J2.36 (Pin_36), UK5.10
- net EOT: now also J2.48 (Pin_48)
- net Entrex Backplane S01B53 to S13B53: no longer J2.53 (Pin_53)
- net HI DENS: now also J2.49 (Pin_49)
- net RB0: now also J2.31 (Pin_31)
- net RB1: now also J2.40 (Pin_40)
- net RB2: now also J2.25 (Pin_25), UP2.10
- net RB3: now also J2.27 (Pin_27), UP2.12
- net RB4: now also J2.13 (Pin_13), UK5.12
- net RB5: now also J2.15 (Pin_15), UK5.2
- net RB6: now also J2.19 (Pin_19), UP2.8
- net RB7: now also J2.23 (Pin_23), UP2.6
- net RBP: now also J2.38 (Pin_38)
- net RWND T: now also J2.69 (Pin_69)
- net RWNDG: now also J2.11 (Pin_11), UK5.6
- net SPC BKD: now also J2.67 (Pin_67)
- net TUR: now also J2.54 (Pin_54)
- net WB6: now also J2.34 (Pin_34), UK5.4
- net WL: now also J2.36 (Pin_36), UK5.10
- no-connect marks 180 -> 92
Other:
- note added: "SLOT 15 DISK OR IO"
- moved on the sheet: UK5C

Commit message: Ready for AMLDC p8
Connections:
- net B7p10 is gone; now on net L1p8: UB7.10
- net B7p4 is gone; now on net C2p5: UB7.4
- net B7p5 is gone; now on net G2p9: UB7.5
- net B8p14 is gone; now on net E8p6: UB8.14 (CP0)
- net B8p2 is gone; now on net H5p5: UB8.2 (R0(1))
- net B8p3 is gone; now on net H5p5: UB8.3 (R0(2))
- net C6p8 is gone; now on net B7p9: UC6.8 (~{Q})
- net C7p12 is gone; now on net C6p9: UC7.12 (D), UC7.3 (C)
- net C7p13 is gone; now on net B6p4: UC7.13 (~{R})
- net C7p4 is gone; now on net D6p8: UC7.4 (~{S})
- net C7p5 is gone; now on net F2p9: UC7.5 (Q), UD7.2 (D)
- net C7p6 is gone; now on net D6p9: UC7.6 (~{Q})
- net C7p9 is gone; now on net D6p10: UC7.9 (Q)
- net C8p1 is gone; now on net G5p5: UC8.1
- net C8p2 is gone; now on net F4p3: UC8.2
- net C8p3 is gone; now on net E5p13: UC8.3
- net C8p4 is gone; now on net C2p5: UC8.4
- net C8p5 is gone; now on net E6p9: UC8.5, UD8.5 (Q)
- net C8p6 is gone; now on net E4p3: UC8.6
- net C8p9 is gone; now on net C8p10: UC8.9
- net D7p1 is gone; now on net E3p1: UD7.1 (~{R})
- net D7p10 is gone; now on net E5p12: UD7.10 (~{S}), UE7.8
- net D7p11 is gone; now on net F4p3: UD7.11 (C)
- net D7p12 is gone; now on net G5p5: UD7.12 (D)
- net D7p13 is gone; now on net F4p1: UD7.13 (~{R})
- net D7p8 is gone; now on net B6p4: UD7.8 (~{Q})
- net D8p1 is gone; now on net J3p4: UD8.1 (~{R})
- net D8p10 is gone; now on net B7p8: UD8.10 (~{S})
- net D8p12 is gone; now on net GND: UD8.12 (D)
- net D8p13 is gone; now on net E3p1: UD8.13 (~{R})
- net D8p3 is gone; now on net B7p6: UD8.3 (C)
- net D8p9 is gone; now on net J3p4: UD8.2 (D), UD8.9 (Q)
- net E7p12 is gone; now on net F1p10: UE7.12
- net E7p13 is gone; now on net E3p5: UE7.13
- net E8p1 is gone; now on net G5p6: UE8.1
- net E8p11 is gone; now on net E7p10: UE8.11
- net E8p12 is gone; now on net B4p10: UE8.12
- net E8p13 is gone; now on net F0p10: UE8.13
- net E8p2 is gone; now on net E5p12: UE8.2
- net E8p3 is gone; now on net C6p13: UE8.3
- net E8p4 is gone; now on net E6p8: UE8.4, UF8.12
- net E8p5 is gone; now on net J3p12: UE8.5, UF8.9
- net F7p2 is gone; now on net H2p12: UF7.2 (D), UH7.2 (D)
- net F7p5 is gone; now on net E6p2: UF7.5 (Q)
- net F7p6 is gone; now on net G6p9: UF7.6 (~{Q})
- net F8p10 is gone; now on net F6p11: UF8.10
- net F8p13 is gone; now on net E6p3: UF8.13
- net F8p8 is gone; now on net F3p10: UF8.8
- net G5p1 is gone; now on net B6p4: UG5.1 (~{R})
- net G6p5 is gone; now on net B7p9: UG6.5
- net G7p1 is gone; now on net F4p1: UG7.1
- net G7p11 is gone; now on net F5p11: UG7.11
- net G7p12 is gone; now on net G6p11: UG7.12
- net G7p13 is gone; now on net G6p11: UG7.13
- net G7p4 is gone; now on net G7p3: UG7.4
- net G7p5 is gone; now on net G7p3: UG7.5
- net G7p6 is gone; now on net H7p1: UG7.6
- net G8p1 is gone; now on net F7p1: UG8.1
- net G8p10 is gone; now on net G5p4: UG8.10
- net G8p11 is gone; now on net G7p8: UG8.11
- net G8p12 is gone; now on net B7p9: UG8.12
- net G8p2 is gone; now on net B6p11: UG8.2
- net G8p4 is gone; now on net G8p3: UG8.4
- net G8p5 is gone; now on net L1p8: UG8.5
- net G8p6 is gone; now on net L1p8: UG8.6
- net G8p8 is gone; now on net G8p9: UG8.8
- net H7p11 is gone; now on net G2p9: UH7.11 (C)
- net J2p11 is gone; now on net D7p9: UJ2.11 (C)
- net J3p1 is gone; now on net E6p9: UJ3.1
- net J7p9 is gone; now on net J6p8: UJ7.9 (A)
- net K7p1 is gone; now on net F1p5: UK7.1
- net K7p10 is gone; now on net G7p9: UK7.10
- net K7p11 is gone; now on net K6p10: UK7.11
- net K7p12 is gone; now on net L1p8: UK7.12
- net K7p13 is gone; now on net J1p13: UK7.13, UK7.4
- net K7p2 is gone; now on net H2p1: UK7.2
- net K7p6 is gone; now on net K6p2: UK7.6
- net K8p10 is gone; now on net C7p11: UK8.10
- net K8p11 is gone; now on net C7p11: UK8.11
- net K8p12 is gone; now on net C7p11: UK8.12
- net K8p13 is gone; now on net K7p5: UK8.13
- net K8p2 is gone; now on net GND: UK8.2
- net K8p6 is gone; now on net K8p5: UK8.6
- net K8p9 is gone; now on net K7p8: UK8.9
- net L7p10 is gone; now on net K1p6: UL7.10 (~{S})
- net L7p11 is gone; now on net J3p8: UL7.11 (C)
- net L7p12 is gone; now on net C6p12: UK7.3, UL7.12 (D)
- net L7p13 is gone; now on net J1p1: UL7.13 (~{R})
- net L7p2 is gone; now on net F0p10: UL7.2 (D)
- net L7p5 is gone; now on net P0p9: UL7.5 (Q)
- net L7p6 is gone; now on net N7p12: UL7.6 (~{Q})
- net L7p9 is gone; now on net G7p10: UL7.9 (Q)
- net M7p12 is gone; now on net E3p5: UM7.12 (D)
- net M7p2 is gone; now on net D7p5: UM7.2 (D)
- net M7p3 is gone; now on net H1p11: UL7.3 (C), UM7.11 (C), UM7.3 (C)
- net M7p8 is gone; now on net J2p10: UM7.8 (~{Q}), UN7.9
- net M7p9 is gone; now on net P0p4: UM7.9 (Q)
- net N7p13 is gone; now on net N0p2: UN7.13
- net N7p8 is gone; now on net M6p6: UN7.8
- net P7p11 is gone; now on net P5p10: UP7.11 (Q3), UR7.14 (CP0)
- net P7p12 is gone; now on net P5p9: UP7.1 (CP1..3), UP7.12 (Q0)
- net P7p14 is gone; now on net E6p6: UP7.14 (CP0)
- net P7p2 is gone; now on net H2p13: UP7.2 (R0(1))
- net P7p5 is gone; now on net +5V: UP7.5 (VCC)
- net P7p8 is gone; now on net P5p13: UP7.8 (Q2)
- net P7p9 is gone; now on net P5p12: UP7.9 (Q1)
- net R22p1 is gone; now on net Q1p3: R22.1
- net R39p1 is gone; now on net +5V: R39.1, R69.2
- net R39p2 is gone; now on net B6p11: R39.2
- net R42p2 is gone; now on net G7p9: R42.2
- net R7p2 is gone; now on net P7p3: UR7.2 (R0(1))
- net R7p5 is gone; now on net +5V: UR7.5 (VCC)
- net S7p2 is gone; now on net P7p3: US7.2 (R0(1))
- net +5V: now also C38.2, R43.1, R79.1
- net F7p3: no longer UG7.2
- net G7p9: now also C48.1
- net GND: now also C54.1, R42.1, UM8.13 (GND)
- net H2p13: now also UP7.3 (R0(2))
- net J6p13: now also UG7.2
- net J7p10: now also R69.1
- net J7p7: now also CR2.1 (K)
- net P7p3: no longer UP7.3 (R0(2))
- net U1p2: now also UU1.2 (Q2)
- net C47p1: now reaches R43.2
- net C47p1: now also C47.1, CR2.2 (A)

Commit message: Draw 9
Connections:
- net D0p12 is gone; now on net W0p1: UD0.12, UN0.3
- net J1p13 is gone; now on net V1p13: UB1.8, UF1.11, UH4.11 (Clr), UJ1.13 (~{R}), UK2.9, UK7.13, UK7.4, UL1.13 (Mr), UL4.13 (Mr), UM1.13 (Mr), UM4.13 (Mr)
- net K5p11 is gone; now on net U3p12: UK5.11
- net L0p3 is gone; now on net ~{DATA15}: JP8.1 (A), UL0.3, UM0.3, UN0.13, UP0.3, UR0.3
- net L0p6 is gone; now on net ~{DATA13}: UL0.6, UM0.6, UN0.5, UP0.6, UR0.6
- net L3p11 is gone; now on net ~{DATA2}: UL3.11, UM3.11, UN3.11, UP3.11, UR3.11
- net L3p8 is gone; now on net ~{DATA0}: UL3.8, UM3.8, UN3.9, UP3.8, UR3.8
- net L4p8 is gone; now on net U3p9: UL4.8 (Cp0)
- net M2p5 is gone; now on net W1p16: UM2.5 (D6)
- net M3p13 is gone; now on net M0p13: R82.2, UM3.10, UM3.13, UM3.2, UM3.5
- net M4p8 is gone; now on net V3p9: UM4.8 (Cp0)
- net N3p2 is gone; now on net R1p4: UN3.2, UR4.13 (E01), UR4.4 (E23), US4.13 (E01), US4.4 (E23)
- net N4p13 is gone; now on net N1p4: UN4.13 (E01), UN4.4 (E23)
- net P2p2 is gone; now on net B51: UP2.2
- net P2p4 is gone; now on net HI DENS: UP2.4
- net P3p13 is gone; now on net W0p2: UP3.10, UP3.13, UP3.2, UP3.5, UT3.13, UT3.2
- net P4p1 is gone; now on net W3p8: UP4.1 (A0)
- net R60p1 is gone; now on net EOT: R60.1, R61.1
- net R64p1 is gone; now on net BOT: R63.1, R64.1
- net R66p1 is gone; now on net RB1: R62.1, R66.1
- net S0p11 is gone; now on net ~{DATA10}: US0.11, UT0.11, UU0.11, UV0.11, UW0.11
- net S0p3 is gone; now on net ~{DATA11}: US0.3, UT0.3, UU0.3, UV0.3, UW0.13
- net S0p6 is gone; now on net ~{DATA9}: US0.6, UT0.6, UU0.6, UV0.6, UW0.5
- net S0p8 is gone; now on net ~{DATA8}: US0.8, UT0.8, UU0.8, UV0.8, UW0.9
- net S3p11 is gone; now on net ~{DATA6}: US3.11, UT3.11, UU3.11, UV3.11, UW3.11
- net S3p3 is gone; now on net ~{DATA7}: US3.3, UT3.3, UU3.3, UV3.3, UW3.13
- net S3p6 is gone; now on net ~{DATA5}: US3.6, UT3.6, UU3.6, UV3.6, UW3.5
- net S3p8 is gone; now on net ~{DATA4}: US3.8, UT3.8, UU3.8, UV3.8, UW3.9
- net T0p4 is gone; now on net W0p4: UT0.4
- net T1p3 is gone; now on net ~{DATA11}: UT1.3
- net T1p4 is gone; now on net B2p6: UT1.4
- net T1p5 is gone; now on net H2p9: UT1.5
- net T1p6 is gone; now on net M0p13: UT1.6
- net T2p6 is gone; now on net H5p2: UT2.6
- net T3p10 is gone; now on net W0p2: UT3.10, UT3.5
- net U0p10 is gone; now on net L0p13: UU0.10, UU0.5
- net U0p2 is gone; now on net L0p13: UU0.13, UU0.2
- net U1p1 is gone; now on net D2p12: UU1.1 (Pl)
- net U1p10 is gone; now on net W0p10: UU1.10 (P1), UV1.10 (P1), UW1.6 (D2)
- net U1p12 is gone; now on net U0p9: UU1.12 (Q3)
- net U1p13 is gone; now on net K6p4: UU1.13 (Mr)
- net U1p2 is gone; now on net U0p4: UU1.2 (Q2)
- net U1p3 is gone; now on net W0p6: UU1.3 (P2), UV1.3 (P2), UW1.2 (D0)
- net U1p4 is gone; now on net W0p12: UU1.4 (P0), UV1.4 (P0), UW1.7 (D3)
- net U1p5 is gone; now on net U0p1: UU1.5 (Q0)
- net U1p6 is gone; now on net U0p1: UU1.6 (Cp1)
- net U1p8 is gone; now on net L1p8: UU1.8 (Cp0)
- net U2p1 is gone; now on net BOT: UU2.1
- net U2p10 is gone; now on net EOT: UU2.10
- net U2p12 is gone; now on net RB1: UU2.12
- net U2p4 is gone; now on net RBP: UU2.4
- net U3p10 is gone; now on net L0p13: UU3.10, UU3.5
- net U3p13 is gone; now on net L0p13: UU3.13, UU3.2
- net U4p1 is gone; now on net D2p12: UU4.1 (Pl)
- net U4p11 is gone; now on net W3p8: UU4.11 (P3), UV4.11 (P3), UW4.3 (D1)
- net U4p12 is gone; now on net U3p9: UU4.12 (Q3)
- net U4p13 is gone; now on net V1p13: UU4.13 (Mr), UV4.13 (Mr)
- net U4p2 is gone; now on net U3p4: UU4.2 (Q2)
- net U4p3 is gone; now on net W3p6: UU4.3 (P2), UV4.3 (P2), UW4.2 (D0)
- net U4p4 is gone; now on net J1p12: UU4.4 (P0), UV4.4 (P0), UW4.7 (D3)
- net U4p5 is gone; now on net U3p1: UU4.5 (Q0)
- net U4p6 is gone; now on net U3p1: UU4.6 (Cp1)
- net U4p9 is gone; now on net U3p12: UU4.9 (Q1)
- net V0p10 is gone; now on net M0p13: UV0.10, UV0.5
- net V0p13 is gone; now on net M0p13: UV0.13, UV0.2
- net V1p1 is gone; now on net B2p12: UV1.1 (Pl)
- net V1p12 is gone; now on net V0p9: UV1.12 (Q3)
- net V1p2 is gone; now on net V0p4: UV1.2 (Q2)
- net V1p5 is gone; now on net V0p1: UV1.5 (Q0)
- net V1p6 is gone; now on net V0p1: UV1.6 (Cp1)
- net V1p8 is gone; now on net M0p9: UV1.8 (Cp0)
- net V1p9 is gone; now on net V0p12: UV1.9 (Q1)
- net V2p1 is gone; now on net U0p9: UV2.1
- net V2p13 is gone; now on net U0p4: UV2.13
- net V2p9 is gone; now on net U1p9: UV2.9
- net V3p10 is gone; now on net M0p13: UV3.10, UV3.5
- net V3p13 is gone; now on net M0p13: UV3.13, UV3.2
- net V4p1 is gone; now on net B2p12: UV4.1 (Pl)
- net V4p12 is gone; now on net V3p9: UV4.12 (Q3)
- net V4p2 is gone; now on net V3p4: UV4.2 (Q2)
- net V4p5 is gone; now on net V3p1: UV4.5 (Q0)
- net V4p6 is gone; now on net V3p1: UV4.6 (Cp1)
- net V4p8 is gone; now on net V0p9: UV4.8 (Cp0)
- net V4p9 is gone; now on net V3p12: UV4.9 (Q1)
- net W0p3 is gone; now on net TUR: UW0.3
- net W1p10 is gone; now on net M2p4: UW1.10 (Q2)
- net W1p13 is gone; now on net N1p4: UW1.13 (E01), UW1.4 (E23)
- net W1p15 is gone; now on net M2p6: UW1.15 (Q1)
- net W1p9 is gone; now on net M2p3: UW1.9 (Q3)
- net W2p13 is gone; now on net E2p9: UW2.13 (E01)
- net W2p15 is gone; now on net P2p3: UW2.15 (Q1)
- net W2p16 is gone; now on net P2p1: UW2.16 (Q0)
- net W2p4 is gone; now on net L2p8: UW2.4 (E23)
- net W2p6 is gone; now on net W0p10: UW2.6 (D2)
- net W2p7 is gone; now on net W0p12: UW2.7 (D3)
- net W3p12 is gone; now on net J1p12: UW3.12
- net W4p10 is gone; now on net N5p12: UW4.10 (Q2)
- net W4p13 is gone; now on net N1p4: UW4.13 (E01), UW4.4 (E23)
- net W4p15 is gone; now on net N5p14: UW4.15 (Q1)
- net W4p16 is gone; now on net N5p13: UW4.16 (Q0)
- net +5V: now also R86.1
- net GND: now also C32.1, C33.1, C34.1, C35.1, R28.2, R59.2, R61.2, R62.2, R63.2
- net RBP: now also R59.1, R65.1
- net TUR: now also R28.1, R86.2
- net U0p1: now also UV2.11
- net U1p11: no longer UW1.3 (D1)
- net U1p9: now also UU0.12
- net U4p10: now also UW3.10
- net W0p8: now also UW1.3 (D1)
- net R78p2: now reaches R78.2
Other:
- note added: "UN7p11 is used...but it doesn't exist"
