File: Trapezoid_Terminal/Arduino Controller/Arduino Controller - Entrex Trapezoid.kicad_sch (KiCad schematic)
At the start: 11 parts, among them J2 Conn_01x04, J3 Conn_01x08, J4 Conn_01x08, J5 Conn_01x06, J6 Conn_01x04, J7 Conn_01x02, J8 Conn_01x19, SW1 SW_Push, U1 74LS04, U2 74LS04

Commit message: build
Parts:
- added H1 (x4): MountingHole, MountingHole:MountingHole_3mm, symbol Mechanical:MountingHole
- added J1: Conn_01x19, Connector_PinHeader_2.54mm:PinHeader_1x19_P2.54mm_Vertical, symbol Connector_Generic:Conn_01x19
- added J9: Logic 8 CH, Forgotten Machines:PinHeader_2x05_P2.54mm_Vertical - Backside, symbol Connector_Generic:Conn_02x05_Odd_Even
- added W1, W2: Winchester_MRE-14, Forgotten Machines:Winchester MRE14 @ 2.54mm pitch, symbol ForgottenMachines:Winchester_MRE-14
- SW1: value SW_Push -> Reset
- U1, U2: footprint (none) -> Package_DIP:DIP-14_W7.62mm
Connections:
- net +5V: now also U2.14 (VCC)
- net Clock Input: now also J9.7 (Pin_7), W1.J (Pin_2), W2.J (Pin_2)
- net D0: now also J6.1 (Pin_1)
- net D1: now also J6.2 (Pin_2)
- net D10: now also J8.3 (Pin_3)
- net D11: now also J8.4 (Pin_4)
- net D12: now also J8.5 (Pin_5)
- net D13: now also J8.6 (Pin_6)
- net D14: now also J8.7 (Pin_7)
- net D15: now also J8.8 (Pin_8)
- net D16: now also J8.9 (Pin_9)
- net D17: now also J8.10 (Pin_10)
- net D18: now also J8.11 (Pin_11)
- net D19: now also J8.12 (Pin_12)
- net D2: now also J6.3 (Pin_3)
- net D20: now also J8.13 (Pin_13)
- net D21: now also J8.14 (Pin_14)
- net D22: now also J8.15 (Pin_15)
- net D23: now also J8.16 (Pin_16)
- net D24: now also J8.17 (Pin_17)
- net D25: now also J8.18 (Pin_18)
- net D26: now also J8.19 (Pin_19)
- net D27: now also J1.1 (Pin_1)
- net D28: now also J1.2 (Pin_2)
- net D29: now also J1.3 (Pin_3)
- net D3: now also J6.4 (Pin_4)
- net D30: now also J1.4 (Pin_4)
- net D31: now also J1.5 (Pin_5)
- net D32: now also J1.6 (Pin_6)
- net D33: now also J1.7 (Pin_7)
- net D34: now also J1.8 (Pin_8)
- net D35: now also J1.9 (Pin_9)
- net D36: now also J1.10 (Pin_10)
- net D37: now also J1.11 (Pin_11)
- net D38: now also J1.12 (Pin_12)
- net D39: now also J1.13 (Pin_13)
- net D40: now also J1.14 (Pin_14)
- net D41: now also J1.15 (Pin_15)
- net D42: now also J1.16 (Pin_16)
- net D43: now also J1.17 (Pin_17)
- net D44: now also J1.18 (Pin_18)
- net D45: now also J1.19 (Pin_19)
- net D46: now also J5.6 (Pin_6)
- net D47: now also J5.5 (Pin_5)
- net D48: now also J5.4 (Pin_4)
- net D53: now also J5.3 (Pin_3)
- net D8: now also J8.1 (Pin_1)
- net D9: now also J8.2 (Pin_2)
- net Data Input: now also W1.D (Pin_2), W2.D (Pin_2)
- net Data Transmit: now also J9.1 (Pin_1), W1.B (Pin_4), W2.B (Pin_4)
- net GND: now also U2.7 (GND), J9.10 (Pin_10), J9.9 (Pin_9)
- net Other Transmit: now also J9.3 (Pin_3), W1.C (Pin_5), W2.C (Pin_5)
- net Port Select Switch: now also W1.E (Pin_3), W2.E (Pin_3)
- net SCL: now also J5.1 (Pin_1)
- net SDA: now also J5.2 (Pin_2)
- net Strobe Input: now also J9.5 (Pin_5), W1.N (Pin_2), W2.N (Pin_2)
- net ~{Clock Input}: now also J9.8 (Pin_8), W1.P (Pin_5), W2.P (Pin_5)
- net ~{Data Input}: now also W1.H (Pin_3), W2.H (Pin_3)
- net ~{Data Transmit}: now also J9.2 (Pin_2), W1.F (Pin_4), W2.F (Pin_4)
- net ~{Other Transmit}: now also J9.4 (Pin_4), W1.A (Pin_1), W2.A (Pin_1)
- net ~{Strobe Input}: now also J9.6 (Pin_6), W1.R (Pin_1), W2.R (Pin_1)
- no-connect marks 10 -> 16
Other:
- moved on the sheet: J2, J3, J4, J5, J6, J7, J8, SW1, U1A, U1B, U1C, U1D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

Commit message: Trapezoid Interface
Parts:
- removed U2: 74LS04, Package_DIP:DIP-14_W7.62mm, symbol 74xx:74LS04
- added J10: Conn_01x04, Connector_PinHeader_2.54mm:PinHeader_1x04_P2.54mm_Vertical, symbol Connector_Generic:Conn_01x04
- renumbered SW1 to Reset1
Connections:
- net +5V: now also W1.L (Pin_4), W2.L (Pin_4), J10.3 (Pin_3), J10.4 (Pin_4)
- net GND: now also W1.K (Pin_3), W1.M (Pin_1), W2.K (Pin_3), W2.M (Pin_1), J10.1 (Pin_1), J10.2 (Pin_2)
- no-connect marks 16 -> 10
