File: Trapezoid_Terminal/Arduino Controller/Arduino Controller - Entrex Trapezoid.kicad_pcb (KiCad board)
At the start: 2 copper layers, 114 x 87 mm, 9 parts, among them J2 Conn_01x04, J3 Conn_01x08, J4 Conn_01x08, J5 Conn_01x06, J6 Conn_01x04, J7 Conn_01x02, J8 Conn_01x19

Commit message: build
Parts:
- added H1: MountingHole, MountingHole:MountingHole_3mm, F.Cu at (152.4, 99.8)
- added H2: MountingHole, MountingHole:MountingHole_3mm, F.Cu at (152.4, 107.3)
- added H3: MountingHole, MountingHole:MountingHole_3mm, F.Cu at (139.1, 99.7)
- added H4: MountingHole, MountingHole:MountingHole_3mm, F.Cu at (139.1, 107.2)
- added J1: Conn_01x19, Connector_PinHeader_2.54mm:PinHeader_1x19_P2.54mm_Vertical, F.Cu at (48.9, 123.2)
- added J9: Logic 8 CH, Forgotten Machines:PinHeader_2x05_P2.54mm_Vertical - Backside, F.Cu at (79.4, 80.0)
- added U1: 74LS04, Package_DIP:DIP-14_W7.62mm, F.Cu at (98.4, 74.9)
- added U2: 74LS04, Package_DIP:DIP-14_W7.62mm, F.Cu at (78.1, 108.6)
- added W1: Winchester_MRE-14, Forgotten Machines:Winchester MRE14 @ 2.54mm pitch, F.Cu at (120.6, 103.7)
- added W2: Winchester_MRE-14, Forgotten Machines:Winchester MRE14 @ 2.54mm pitch, F.Cu at (132.8, 79.6)
- SW1: renamed from Reset; value SW_Push -> Reset
- moved XA1 2.29 mm to (150.4, 65.5)
- moved J5 0.36 mm to (95.9, 47.0)
- moved J6 0.36 mm to (111.1, 47.0)
Connections:
- net A0 renamed Net-(J4-Pin_1)
- net A1 renamed Net-(J4-Pin_2)
- net A10 renamed Net-(J3-Pin_3)
- net A11 renamed Net-(J3-Pin_4)
- net A12 renamed Net-(J3-Pin_5)
- net A13 renamed Net-(J3-Pin_6)
- net A14 renamed Net-(J3-Pin_7)
- net A15 renamed Net-(J3-Pin_8)
- net A8 renamed Net-(J3-Pin_1)
- net A9 renamed Net-(J3-Pin_2)
- J4 pad 3: ~{ISTP} -> Net-(J4-Pin_3)
- J4 pad 4: ~{PL} -> Net-(J4-Pin_4)
- J4 pad 5: ~{CON INST} -> Net-(J4-Pin_5)
- J4 pad 6: ~{CON RQ} -> Net-(J4-Pin_6)
- J4 pad 7: ~{RST} -> Net-(J4-Pin_7)
- J4 pad 8: RESTART ENABLE -> Net-(J4-Pin_8)
- J5 pad 1: ~{ISTP} -> SCL
- J5 pad 2: ~{PL} -> SDA
- J5 pad 3: ~{CON INST} -> D53
- J5 pad 4: ~{CON RQ} -> D48
- J5 pad 5: ~{RST} -> D47
- J5 pad 6: RESTART ENABLE -> D46
- J6 pad 1: D2 -> D0
- J6 pad 2: ~{CONT+ISTP+MSTP} -> D1
- J6 pad 3: ~{CON DATA} -> D2
- J6 pad 4: ~{STOP} -> D3
- J7 pad 1: 53 -> unconnected-(J7-Pin_1-Pad1)
- J7 pad 2: 52 -> unconnected-(J7-Pin_2-Pad2)
- J8 pad 1: ~{STOP} -> D8
- J8 pad 10: D8 -> D17
- J8 pad 11: D9 -> D18
- J8 pad 12: D10 -> D19
- J8 pad 13: D11 -> D20
- J8 pad 14: D12 -> D21
- J8 pad 15: D13 -> D22
- J8 pad 16: GND -> D23
- J8 pad 17: AREF -> D24
- J8 pad 18: SDA -> D25
- J8 pad 19: SCL -> D26
- J8 pad 2: ~{CON DATA} -> D9
- J8 pad 3: ~{CONT+ISTP+MSTP} -> D10
- J8 pad 4: D2 -> D11
- J8 pad 5: D3 -> D12
- J8 pad 6: D4 -> D13
- J8 pad 7: D5 -> D14
- J8 pad 8: D6 -> D15
- J8 pad 9: D7 -> D16
- XA1 pad 3V3: Net-(XA1-Pad3V3) -> unconnected-(XA1-3.3V-Pad3V3)
- XA1 pad 5V2: Net-(XA1-Pad5V2) -> unconnected-(XA1-SPI_5V-Pad5V2)
- XA1 pad A2: ~{ISTP} -> Net-(J4-Pin_3)
- XA1 pad A3: ~{PL} -> Net-(J4-Pin_4)
- XA1 pad A4: ~{CON INST} -> Net-(J4-Pin_5)
- XA1 pad A5: ~{CON RQ} -> Net-(J4-Pin_6)
- XA1 pad A6: ~{RST} -> Net-(J4-Pin_7)
- XA1 pad A7: RESTART ENABLE -> Net-(J4-Pin_8)
- XA1 pad D0: ~{CON DATA} -> D0
- XA1 pad D1: ~{CONT+ISTP+MSTP} -> D1
- XA1 pad D14: ~{STOP} -> D14
- XA1 pad D4: D4 -> Port Select Switch
- XA1 pad D49: D49 -> ~{Data Transmit}
- XA1 pad D5: D5 -> ~{Other Transmit}
- XA1 pad D50: D50 -> Data Transmit
- XA1 pad D51: D51 -> Data Input
- XA1 pad D52: 53 -> Clock Input
- XA1 pad D53: 52 -> D53
- XA1 pad D6: D6 -> Other Transmit
- XA1 pad D7: D7 -> Strobe Input
- XA1 pad GND4: Net-(XA1-PadGND4) -> unconnected-(XA1-SPI_GND-PadGND4)
- XA1 pad IORF: Net-(XA1-PadIORF) -> unconnected-(XA1-IOREF-PadIORF)
- XA1 pad MISO: Net-(XA1-PadMISO) -> unconnected-(XA1-SPI_MISO-PadMISO)
- XA1 pad MOSI: Net-(XA1-PadMOSI) -> unconnected-(XA1-SPI_MOSI-PadMOSI)
- XA1 pad RST2: Net-(XA1-PadRST2) -> unconnected-(XA1-SPI_RESET-PadRST2)
- XA1 pad SCK: Net-(XA1-PadSCK) -> unconnected-(XA1-SPI_SCK-PadSCK)
Routing:
- removed copper zone on F.Cu, net GND
Other:
- outline, holes or cut-outs redrawn
- board text added: "74LS04"
- board text added: "BDIR"
- board text added: "BSYNC TERMINAL"
- board text added: "CLK"
- board text added: "Clock Input"
- board text added: "Data Input"
- board text added: "Data Transmit"
- board text added: "Logic 8"
- board text added: "Other Transmit"
- board text added: "Port Select Switch"
- board text added: "RX"
- board text added: "Strobe Input"
- board text added: "TX"
- board text added: "~{BDIR}"
- board text added: "~{BDIR} ~{BSYNC TERMINAL} ~{CLK} ~{Clock Input} ~{Data Input} ~{Data Transmit} ~{Other Transmit} ~{RX} ~{Strobe Input} ~{TX} BDIR BSYNC TERMINAL CLK Clock Input Data Input Data Transmit Other Transmit Port Select Switch RX Strobe Input TX"
- board text added: "~{BSYNC TERMINAL}"
- board text added: "~{CLK}"
- board text added: "~{Clock Input}"
- board text added: "~{Data Input}"
- board text added: "~{Data Transmit}"
- board text added: "~{Other Transmit}"
- board text added: "~{RX}"
- board text added: "~{Strobe Input}"
- board text added: "~{TX}"
- board text removed: "AREF"
- board text removed: "Front Panel"

Commit message: Trapezoid Interface
Parts:
- removed J7: Conn_01x02, port_nova:PinHeader_1x02_P2.54mm_Vertical
- removed U2: 74LS04, Package_DIP:DIP-14_W7.62mm
- added J10: Conn_01x04, Connector_PinHeader_2.54mm:PinHeader_1x04_P2.54mm_Vertical, F.Cu at (128.3, 44.5)
- XA1: footprint Arduino:Arduino_Mega2560_Shield -> Forgotten Machines:Arduino_Mega2560_Shield
- moved J5 2.54 mm to (95.9, 44.5)
- moved J6 2.54 mm to (111.1, 44.5)
- moved J9 1.35 mm to (79.2, 78.7)
- renumbered SW1 to Reset1
Routing:
- net Other Transmit: track 0.00 -> 151.0 mm, vias 0 -> 2
- net Strobe Input: track 0.00 -> 149.0 mm, vias 0 -> 4
- net D25: track 0.00 -> 148.3 mm, vias 0 -> 1
- net D23: track 0.00 -> 147.3 mm, vias 0 -> 1
- net D24: track 0.00 -> 146.4 mm, vias 0 -> 1
- net D22: track 0.00 -> 146.3 mm, vias 0 -> 1
- net ~{Other Transmit}: track 0.00 -> 144.6 mm, vias 0 -> 3
- net Clock Input: track 0.00 -> 141.3 mm, vias 0 -> 5
- net Port Select Switch: track 0.00 -> 134.7 mm, vias 0 -> 3
- net D26: track 0.00 -> 134.2 mm, vias 0 -> 1
- net D21: track 0.00 -> 133.8 mm, vias 0 -> 1
- net ~{Data Transmit}: track 0.00 -> 129.3 mm, vias 0 -> 1
- net D20: track 0.00 -> 129.0 mm, vias 0 -> 1
- net D19: track 0.00 -> 124.5 mm, vias 0 -> 1
- net D18: track 0.00 -> 120.3 mm, vias 0 -> 1
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- added copper zone on F.Cu, net +5V
Other:
- board text added: "(Nixdorf)"
- board text added: "+5v"
- board text added: "15"
- board text added: "16"
- board text added: "17"
- board text added: "18"
- board text added: "25"
- board text added: "26"
- board text added: "27"
- board text added: "28"
- board text added: "29"
- board text added: "30"
- board text added: "31"
- board text added: "32"
- board text added: "33"
- board text added: "34"
- board text added: "35"
- board text added: "36"
- board text added: "37"
- board text added: "38"
- board text added: "39"
- board text added: "40"
- board text added: "41"
- board text added: "42"
- board text added: "43"
- board text added: "44"
- board text added: "BSYNC"
- board text added: "Entrex {dblquote}Trapezoid{dblquote} Data/Terminal Interface"
- board text added: "Reset"
- board text removed: "52"
- board text removed: "BSYNC TERMINAL"

Commit message: same
Connections:
- W1 pad K: unconnected-(W1-Pin_3-PadK) -> GND
- W1 pad L: unconnected-(W1-Pin_4-PadL) -> +5V
- W1 pad M: unconnected-(W1-Pin_1-PadM) -> GND
- W2 pad K: unconnected-(W2-Pin_3-PadK) -> GND
- W2 pad L: unconnected-(W2-Pin_4-PadL) -> +5V
- W2 pad M: unconnected-(W2-Pin_1-PadM) -> GND
Routing:
- net GND: track 29.3 -> 44.2 mm, vias 3 -> 6
- net +5V: track 5.59 -> 17.6 mm, vias 2 -> 4
Other:
- board text removed: "4"
- board text removed: "5"
- board text removed: "6"
- board text removed: "7"
Changed lines of the file:
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@@
   (net 93 "unconnected-(XA1-SPI_RESET-PadRST2)")
   (net 94 "unconnected-(XA1-SPI_SCK-PadSCK)")
-  (net 95 "unconnected-(W1-Pin_3-PadK)")
-  (net 96 "unconnected-(W1-Pin_4-PadL)")
-  (net 97 "unconnected-(W1-Pin_1-PadM)")
-  (net 98 "unconnected-(W2-Pin_3-PadK)")
-  (net 99 "unconnected-(W2-Pin_4-PadL)")
-  (net 100 "unconnected-(W2-Pin_1-PadM)")
   (footprint "port_nova:PinHeader_1x04_P2.54mm_Vertical" (layer "F.Cu")
     (at 153.568 80.346)
@@
       (net 78 "Clock Input") (pinfunction "Pin_2") (pintype "passive"))
     (pad "K" thru_hole oval (at 2.54 0 270) (size 1.7 1.7) (drill 1) (layers "*.Cu" "*.Mask")
-      (net 95 "unconnected-(W1-Pin_3-PadK)") (pinfunction "Pin_3") (pintype "passive+no_connect"))
+      (net 45 "GND") (pinfunction "Pin_3") (pintype "passive"))
     (pad "L" thru_hole oval (at -2.54 2.54 270) (size 1.7 1.7) (drill 1) (layers "*.Cu" "*.Mask")
-      (net 96 "unconnected-(W1-Pin_4-PadL)") (pinfunction "Pin_4") (pintype "passive+no_connect"))
+      (net 44 "+5V") (pinfunction "Pin_4") (pintype "passive"))
     (pad "M" thru_hole oval (at 0 3.81 270) (size 1.7 1.7) (drill 1) (layers "*.Cu" "*.Mask")
-      (net 97 "unconnected-(W1-Pin_1-PadM)") (pinfunction "Pin_1") (pintype "passive+no_connect"))
+      (net 45 "GND") (pinfunction "Pin_1") (pintype "passive"))
     (pad "N" thru_hole oval (at 2.54 2.54 270) (size 1.7 1.7) (drill 1) (layers "*.Cu" "*.Mask")
       (net 75 "Strobe Input") (pinfunction "Pin_2") (pintype "passive"))
@@
       (net 78 "Clock Input") (pinfunction "Pin_2") (pintype "passive"))
     (pad "K" thru_hole oval (at 2.54 0 270) (size 1.7 1.7) (drill 1) (layers "*.Cu" "*.Mask")
-      (net 98 "unconnected-(W2-Pin_3-PadK)") (pinfunction "Pin_3") (pintype "passive+no_connect"))
+      (net 45 "GND") (pinfunction "Pin_3") (pintype "passive"))
     (pad "L" thru_hole oval (at -2.54 2.54 270) (size 1.7 1.7) (drill 1) (layers "*.Cu" "*.Mask")
-      (net 99 "unconnected-(W2-Pin_4-PadL)") (pinfunction "Pin_4") (pintype "passive+no_connect"))
+      (net 44 "+5V") (pinfunction "Pin_4") (pintype "passive"))
     (pad "M" thru_hole oval (at 0 3.81 270) (size 1.7 1.7) (drill 1) (layers "*.Cu" "*.Mask")
-      (net 100 "unconnected-(W2-Pin_1-PadM)") (pinfunction "Pin_1") (pintype "passive+no_connect"))
+      (net 45 "GND") (pinfunction "Pin_1") (pintype "passive"))
     (pad "N" thru_hole oval (at 2.54 2.54 270) (size 1.7 1.7) (drill 1) (layers "*.Cu" "*.Mask")
       (net 75 "Strobe Input") (pinfunction "Pin_2") (pintype "passive"))
@@
     (effects (font (size 1 1) (thickness 0.15)))
   )
-  (gr_text "6" (at 127.775 36.195 -90) (layer "F.SilkS")
-    (effects (font (size 1 1) (thickness 0.15)))
-  )
-  (gr_text "7" (at 130.175 36.195 -90) (layer "F.SilkS")
-    (effects (font (size 1 1) (thickness 0.15)))
-  )
   (gr_text "8" (at 103.505 57.285 -90) (layer "F.SilkS")
     (effects (font (size 1 1) (thickness 0.15)))
@@
     (effects (font (size 1 1) (thickness 0.15)))
   )
-  (gr_text "4" (at 122.675 36.195 -90) (layer "F.SilkS")
-    (effects (font (size 1 1) (thickness 0.15)))
-  )
   (gr_text "1" (at 108.525 46.99 -90) (layer "F.SilkS")
     (effects (font (size 1 1) (thickness 0.15)))
   )
-  (gr_text "5" (at 125.175 36.195 -90) (layer "F.SilkS")
-    (effects (font (size 1 1) (thickness 0.15)))
-  )
   (gr_text "SDA" (at 93.385 47.625 -90) (layer "F.SilkS")
     (effects (font (size 1 1) (thickness 0.15)))
@@
     (effects (font (size 0.7 0.7) (thickness 0.15)) (justify left bottom))
   )
-  (gr_text "~{BDIR}\n~{BSYNC TERMINAL}\n~{CLK}\n~{Clock Input}\n~{Data Input}\n~{Data Transmit}\n~{Other Transmit}\n~{RX}\n~{Strobe Input}\n~{TX}\nBDIR\nBSYNC TERMINAL\nCLK\nClock Input\nData Input\nData Transmit\nOther Transmit\nPort Select Switch\nRX\nStrobe Input\nTX" (at 167.19 -21.51) (layer "F.SilkS")
-    (effects (font (size 0.7 0.7) (thickness 0.15)) (justify left bottom))
-  )
   (gr_text "53" (at 90.805 46.99) (layer "F.SilkS")
     (effects (font (size 1 1) (thickness 0.15)))
@@
   (segment (start 74.168 93.472) (end 74.295 93.345) (width 0.25) (layer "B.Cu") (net 43))
   (segment (start 56.388 93.472) (end 74.168 93.472) (width 0.25) (layer "B.Cu") (net 43))
-  (via (at 106.553 111.506) (size 0.6) (drill 0.3) (layers "F.Cu" "B.Cu") (free) (net 44))
-  (via (at 112.141 111.506) (size 0.6) (drill 0.3) (layers "F.Cu" "B.Cu") (free) (net 44))
-  (segment (start 106.553 111.506) (end 112.141 111.506) (width 1) (layer "B.Cu") (net 44))
+  (via (at 145.034 69.977) (size 0.6) (drill 0.3) (layers "F.Cu" "B.Cu") (net 44))
+  (via (at 106.68 106.172) (size 0.6) (drill 0.3) (layers "F.Cu" "B.Cu") (net 44))
+  (via (at 138.811 69.977) (size 0.6) (drill 0.3) (layers "F.Cu" "B.Cu") (free) (net 44))
+  (via (at 112.268 106.172) (size 0.6) (drill 0.3) (layers "F.Cu" "B.Cu") (net 44))
+  (segment (start 112.268 106.172) (end 117.927 106.172) (width 1) (layer "B.Cu") (net 44))
+  (segment (start 106.68 106.172) (end 112.268 106.172) (width 1) (layer "B.Cu") (net 44))
+  (segment (start 138.811 69.977) (end 145.034 69.977) (width 0.7) (layer "B.Cu") (net 44))
+  (segment (start 117.927 106.172) (end 118.015 106.26) (width 1) (layer "B.Cu") (net 44))
+  (segment (start 120.523 111.76) (end 120.555 111.792) (width 0.25) (layer "F.Cu") (net 45))
   (segment (start 107.188 68.072) (end 107.188 61.976) (width 0.5) (layer "F.Cu") (net 45))
+  (segment (start 120.523 111.125) (end 120.555 111.157) (width 0.5) (layer "F.Cu") (net 45))
+  (segment (start 120.555 111.157) (end 120.555 111.728) (width 0.5) (layer "F.Cu") (net 45))
   (segment (start 107.188 61.976) (end 104.394 59.182) (width 0.5) (layer "F.Cu") (net 45))
   (segment (start 89.38 78.66) (end 89.38 81.2) (width 0.5) (layer "F.Cu") (net 45))
+  (segment (start 120.555 111.728) (end 120.523 111.76) (width 0.25) (layer "F.Cu") (net 45))
+  (segment (start 132.842 86.233) (end 132.775 86.166) (width 0.25) (layer "F.Cu") (net 45))
   (segment (start 97.155 90.17) (end 95.25 88.265) (width 0.5) (layer "F.Cu") (net 45))
   (segment (start 89.38 75.466) (end 89.408 75.438) (width 0.5) (layer "F.Cu") (net 45))
   (segment (start 95.25 88.265) (end 95.25 81.28) (width 0.5) (layer "F.Cu") (net 45))
+  (segment (start 120.555 111.093) (end 120.523 111.125) (width 0.5) (layer "F.Cu") (net 45))
+  (segment (start 120.555 111.792) (end 120.555 111.982) (width 0.25) (layer "F.Cu") (net 45))
+  (segment (start 132.842 86.106) (end 132.775 86.166) (width 0.25) (layer "F.Cu") (net 45))
   (segment (start 98.425 90.17) (end 97.155 90.17) (width 0.5) (layer "F.Cu") (net 45))
   (segment (start 89.38 81.2) (end 89.38 75.466) (width 0.5) (layer "F.Cu") (net 45))
+  (segment (start 120.555 107.53) (end 120.555 111.093) (width 0.5) (layer "F.Cu") (net 45))
+  (segment (start 132.775 83.41) (end 132.842 86.106) (width 0.5) (layer "F.Cu") (net 45))
+  (via (at 120.523 111.125) (size 0.6) (drill 0.3) (layers "F.Cu" "B.Cu") (net 45))
   (via (at 95.25 81.28) (size 0.6) (drill 0.3) (layers "F.Cu" "B.Cu") (net 45))
   (via (at 89.408 75.438) (size 0.6) (drill 0.3) (layers "F.Cu" "B.Cu") (net 45))
+  (via (at 120.523 111.76) (size 0.6) (drill 0.3) (layers "F.Cu" "B.Cu") (net 45))
   (via (at 104.394 59.182) (size 0.6) (drill 0.3) (layers "F.Cu" "B.Cu") (net 45))
+  (via (at 132.842 86.106) (size 0.6) (drill 0.3) (layers "F.Cu" "B.Cu") (net 45))
+  (segment (start 119.38 104.503299) (end 119.38 106.355) (width 0.25) (layer "B.Cu") (net 45))
+  (segment (start 123.095 103.72) (end 120.163299 103.72) (width 0.25) (layer "B.Cu") (net 45))
+  (segment (start 120.163299 103.72) (end 119.38 104.503299) (width 0.25) (layer "B.Cu") (net 45))
+  (segment (start 119.38 106.355) (end 120.555 107.53) (width 0.25) (layer "B.Cu") (net 45))
   (segment (start 98.416 66.684) (end 97.028 68.072) (width 0.25) (layer "F.Cu") (net 47))
   (segment (start 98.416 55.256) (end 98.416 66.684) (width 0.25) (layer "F.Cu") (net 47))

Commit message: DRC Checks p1
Routing:
- net Other Transmit: track 151.0 -> 145.6 mm
- net ~{Data Input}: track 72.8 -> 71.5 mm
- net D43: track 86.4 -> 85.6 mm
- net ~{Strobe Input}: track 117.8 -> 117.0 mm
- net Data Transmit: track 118.2 -> 117.5 mm
- net D18: track 120.3 -> 119.7 mm
- net Net-(XA1-RESET): track 61.4 -> 60.9 mm
- net D22: track 146.3 -> 145.8 mm
Other:
- outline, holes or cut-outs redrawn

Commit message: mmm
Other:
- board text added: "Unused"
- board text removed: "+12V"
Changed lines of the file:
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@@
     (solder_mask_min_width 0.25)
     (pcbplotparams
-      (layerselection 0x00010fc_ffffffff)
+      (layerselection 0x00310fc_ffffffff)
       (plot_on_all_layers_selection 0x0000000_00000000)
       (disableapertmacros false)
@@
       (psa4output false)
       (plotreference true)
-      (plotvalue true)
+      (plotvalue false)
       (plotinvisibletext false)
       (sketchpadsonfab false)
@@
     (effects (font (size 1 1) (thickness 0.15)))
   )
-  (gr_text "+12V" (at 156.568 87.966) (layer "F.SilkS")
-    (effects (font (size 0.85 0.85) (thickness 0.15)))
+  (gr_text "Unused" (at 156.568 87.966) (layer "F.SilkS")
+    (effects (font (size 0.5 0.5) (thickness 0.1)))
   )
   (gr_text "~{Clock Input}\n" (at 122.675 85.4) (layer "F.SilkS")
@@
     (effects (font (size 1 1) (thickness 0.15)))
   )
-  (gr_text "(Nixdorf)" (at 47.625 70.104) (layer "F.SilkS")
+  (gr_text "(Nixdorf)" (at 48.895 72.39) (layer "F.SilkS")
     (effects (font (size 3 3) (thickness 0.5) bold) (justify left bottom))
   )
@@
     (effects (font (size 1 1) (thickness 0.15)))
   )
+  (dimension (type aligned) (layer "Dwgs.User")
+    (pts (xy 44.57 41.3) (xy 44.45 128.41))
+    (height 9.799289)
+    (gr_text "87.1101 mm" (at 33.560721 84.839917 89.92107118) (layer "Dwgs.User")
+      (effects (font (size 1 1) (thickness 0.15)))
+    )
+    (format (prefix "") (suffix "") (units 3) (units_format 1) (precision 4))
+    (style (thickness 0.1) (arrow_length 1.27) (text_position_mode 0) (extension_height 0.58642) (extension_offset 0.5) keep_text_aligned)
+  )
+  (dimension (type aligned) (layer "Dwgs.User")
+    (pts (xy 44.568 41.346) (xy 158.568 41.346))
+    (height -9.596)
+    (gr_text "114.0000 mm" (at 101.568 30.6) (layer "Dwgs.User")
+      (effects (font (size 1 1) (thickness 0.15)))
+    )
+    (format (prefix "") (suffix "") (units 3) (units_format 1) (precision 4))
+    (style (thickness 0.1) (arrow_length 1.27) (text_position_mode 0) (extension_height 0.58642) (extension_offset 0.5) keep_text_aligned)
+  )
   (segment (start 78.096 66.666) (end 78.096 55.246) (width 0.25) (layer "F.Cu") (net 1))
