File: DataScope/Original DataScope Boards/CRT Term Board No 1A+1B/CRT Term Board No 1A+1B.kicad_sch (KiCad schematic)
At the start: 10 parts

Commit message: X
Parts:
- added UB5: 74LS40, symbol 74xx:74LS40
- added UC3: 74LS04, symbol 74xx:74LS04
Connections:
- net ~{RC*}: now also UB5.13
- net ~{TC01-DLSa}: now also UB5.9
- net at UA7.3 (C), UB6.11 (C), UB6.3 (C)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: now also UC3.8
- new net: UB5.8, UC3.9
- new net CLKR: UB5.12
- new net CLKW: UB5.10
Other:
- note added: "(SH4&7) (B01618 SH7)"
- note added: "NOTE* BOTH CLKR & CLKW CAN BE ON DURING INSERT"
- note added: "TP3"
