File: DataScope/Original DataScope Boards/CRT Term Board No 1A+B/3 of 16.kicad_sch (KiCad schematic)
At the start: 0 parts

Commit message: Upgrades 3
Parts:
- added JTP3: Conn_01x01_Pin, symbol Connector:Conn_01x01_Pin
- added R7C4: 1.5K, symbol Device:R_US
- added R8C4: 1K, symbol Device:R_US
- added UA4: 74LS51, symbol 74xx:74LS51
- added UA6: 74LS10, symbol 74xx:74LS10
- added UA7, UB6, UB7, UC6, UC7, UD7: 74LS74, symbol 74xx:74LS74
- added UA8, UB5: 74LS40, symbol 74xx:74LS40
- added UB8, UD8: 74LS00, symbol 74xx:74LS00
- added UC3, UC9: 74LS04, symbol 74xx:74LS04
Connections:
- new net: UA4.1, UC7.6 (~{Q})
- new net: UA7.1 (~{R}), UB6.1 (~{R}), UB6.13 (~{R}), UC6.1 (~{R}), UC6.13 (~{R}), UD7.13 (~{R})
- new net: UA4.6, UA7.2 (D)
- new net: UA7.3 (C), UB6.11 (C), UB6.3 (C), UC3.8, UC6.11 (C), UC6.3 (C), UD7.11 (C)
- new net: UA8.1, UA8.2, UB8.3
- new net: UA4.5, UA4.8
- new net: UB7.5 (Q), UC7.12 (D)
- new net: UC9.11, UD8.11
- new net: UB5.8, UC3.9
- new net: UA8.4, UB8.8
- new net: UA8.5, UB8.11
- new net (SHOULD NEVER GO LO): JTP3.1 (Pin_1), UD8.8
- new net 01: UA6.11
- new net AS1: UA7.6 (~{Q}), UB6.12 (D)
- new net AS2: UB6.2 (D), UB6.9 (Q)
- new net AS3: UB6.5 (Q), UC6.2 (D)
- new net AS4: UC6.12 (D), UC6.5 (Q)
- new net AS5: UC6.9 (Q), UD7.12 (D)
- new net AS6: UD7.9 (Q)
- new net CLKR: UB5.12
- new net CLKW: UB5.10
- new net COPY: UB8.13
- new net DATA GONE: UB8.12
- new net DATA RDY: UB8.2, UB8.9
- new net DATA READY: UA6.10
- new net DL OUT SHIFT: UB7.3 (C), UC7.11 (C), UC7.3 (C), UC9.10
- new net DL WRITE: UA8.6, UB8.5
- new net DLCODE: UB7.2 (D)
- new net FR1: UD8.4
- new net FR2: UD8.5
- new net FRAMED: UA4.10, UC9.4
- new net FRZ: UD8.9
- new net GND: R7C4.2
- new net INSERT: UB8.1
- new net LINE: UC7.2 (D), UC7.9 (Q)
- new net OUT: UA4.2
- new net RC: UA6.1
- new net RC*: UC9.12, UD8.10
- new net RE: UA4.3, UA6.9
- new net VCC: R8C4.1, UA7.4 (~{S}), UB6.10 (~{S}), UB6.4 (~{S}), UB7.4 (~{S}), UC7.10 (~{S}), UC7.4 (~{S}), UD7.10 (~{S}), UD7.4 (~{S})
- new net WE: UB8.10
- new net ~{02}: UB8.4
- new net ~{AS3}: UB6.6 (~{Q})
- new net ~{AS6}: UA4.9
- new net ~{CLKR}: UA6.8
- new net ~{CLKW}: UB8.6
- new net ~{DLSEL+DLNXT}: UA6.2
- new net ~{DONE}: UB7.1 (~{R}), UC7.1 (~{R}), UD7.1 (~{R})
- new net ~{FRAMED}: UA4.13, UA6.13, UC9.3, UD8.6
- new net ~{RC*}: UA6.12, UB5.13, UC9.13, UD8.13
- new net ~{RE}: UA4.4
- new net ~{SRS * LINE MSM}: UC7.13 (~{R})
- new net ~{TC01*DLSEL}: UD8.12
- new net ~{TC01-DLSa}: R7C4.1, R8C4.2, UB5.9
- no-connect marks 0 -> 10
Other:
- note added: "(SH4&7) (B01618 SH7)"
- note added: "4 BIT LINE CNTR"
- note added: "6 BIT COL CNTR"
- note added: "AS1 INSERT"
- note added: "AS2 COPY"
- note added: "AS3 ROLL DOWN"
- note added: "AS4 ROLL UP"
- note added: "AS5 ERROR BEEP"
- note added: "AS6 READ REG"
- note added: "B01618"
- note added: "CRT Term Bd 1A+B Command Buffer Part 2 - Drawing No. 01617"
- note added: "DATA RDY (3)"
- note added: "LONG SR SH6"
- note added: "NOTE* BOTH CLKR & CLKW CAN BE ON DURING INSERT"
- note added: "SH10"
- note added: "SH16"
- note added: "SH4"
- note added: "SH4&7"
- note added: "SH4,5&6"
- note added: "SH5"
- note added: "SH6"
- note added: "SH7"
- note added: "SH8"
- note added: "SH8,16"
- note added: "TP3"
