File: DataScope/Original DataScope Boards/CRT Term Board No 1A+B/CRT Term Board No 1A+B.kicad_sch (KiCad schematic)
At the start: 12 parts

Commit message: done 1
Parts:
- added JTP3: Conn_01x01_Pin, symbol Connector:Conn_01x01_Pin
- added U1, UB8, UD8: 74LS00, symbol 74xx:74LS00
- added UA8: 74LS40, symbol 74xx:74LS40
- added UC9: 74LS04, symbol 74xx:74LS04
Connections:
- net (SHOULD NEVER GO LO): now also JTP3.1 (Pin_1), UD8.8
- net 01: now also UA6.11
- net DL OUT SHIFT: now also UC9.10
- net FRAMED: now also UC9.4
- net FRZ: now also UD8.9
- net RC*: now also UC9.12, UD8.10
- net RE: now also UA6.9
- net WE: now also U1.10
- net ~{FRAMED}: now also UC9.3, UD8.6
- net ~{RC*}: now also UC9.13, UD8.13
- net DATA READY: now reaches UA6.10
- net ~{CLKR}: now reaches UA6.8
- new net: U1.3, UA8.1, UA8.2
- new net: UC9.11, UD8.11
- new net: U1.8, UA8.4
- new net: U1.11, UA8.5
- new net COPY: U1.13
- new net DATA GONE: U1.12
- new net DATA RDY: U1.2, U1.9
- new net DL WRITE: UA8.6, UB8.5
- new net FR1: UD8.4
- new net FR2: UD8.5
- new net INSERT: U1.1
- new net ~{02}: UB8.4
- new net ~{CLKW}: UB8.6
- new net ~{TC01*DLSEL}: UD8.12
Other:
- note added: "CRT Term Bd 1A+B Command Buffer Part 2 - Drawing No. 01617"
- note added: "DATA RDY (3)"
- note added: "SH16"

Commit message: Upgrades 3
Parts:
- removed JTP3: Conn_01x01_Pin, symbol Connector:Conn_01x01_Pin
- removed R7C4: 1.5K, symbol Device:R_US
- removed R8C4: 1K, symbol Device:R_US
- removed U1, UB8, UD8: 74LS00, symbol 74xx:74LS00
- removed UA4: 74LS51, symbol 74xx:74LS51
- removed UA6: 74LS10, symbol 74xx:74LS10
- removed UA7, UB6, UB7, UC6, UC7, UD7: 74LS74, symbol 74xx:74LS74
- removed UA8, UB5: 74LS40, symbol 74xx:74LS40
- removed UC3, UC9: 74LS04, symbol 74xx:74LS04
Connections:
- no-connect marks 10 -> 0
Other:
- added sheet Command Buffer Part 2 (3 of 16.kicad_sch)
- added sheet Control Flops (4 of 16.kicad_sch)
- note removed: "(SH4&7) (B01618 SH7)"
- note removed: "4 BIT LINE CNTR"
- note removed: "6 BIT COL CNTR"
- note removed: "AS1 INSERT"
- note removed: "AS2 COPY"
- note removed: "AS3 ROLL DOWN"
- note removed: "AS4 ROLL UP"
- note removed: "AS5 ERROR BEEP"
- note removed: "AS6 READ REG"
- note removed: "B01618"
- note removed: "CRT Term Bd 1A+B Command Buffer Part 2 - Drawing No. 01617"
- note removed: "DATA RDY (3)"
- note removed: "LONG SR SH6"
- note removed: "NOTE* BOTH CLKR & CLKW CAN BE ON DURING INSERT"
- note removed: "SH10"
- note removed: "SH16"
- note removed: "SH4"
- note removed: "SH4&7"
- note removed: "SH4,5&6"
- note removed: "SH5"
- note removed: "SH6"
- note removed: "SH7"
- note removed: "SH8"
- note removed: "SH8,16"
- note removed: "TP3"
