File: DataScope/Original DataScope Boards/CRT Term Board No 1A+B/4 of 16.kicad_sch (KiCad schematic)
At the start: 7 parts

Commit message: n
Connections:
- net FRAMED: now also UE10.10
- net TI: now reaches UE10.11
- net ~{INT}: now reaches UE10.9
Other:
- note added: "+5V"
- note added: "38-6"
- note added: "B19-9"
- note added: "R6D18"
- note added: "SH12"
- note added: "SH13"
- note added: "SH5"
- moved on the sheet: UE10C
